File: MotherBoard/BenchyMotherBoard-PCB/display.kicad_sch (KiCad schematic)
At the start: 39 parts, among them J2 LVDS-DISPLAY, J6 HDMI_A_1.4, Q3 RQ5A030AP, U15 LM317L, U16 AS321, U25 TPD12S016RKTR, U34 74HCT2G08, U4 AM6254ATCGGAALW, U5 SiI9022ACNU

Commit message: Start PCB layout
Parts:
- J19: renamed from J2; footprint Daxxn_Connectors:0541324033 -> Daxxn_Connectors:5019514000
- U5: footprint Package_DFN_QFN:QFN-72-1EP_10x10mm_P0.5mm_EP6x6mm -> Daxxn_Packages:QFN-72-1EP_10x10mm_P0.5mm_EP6x6mm
- renumbered J6 to J20, U25 to U37, U34 to U40
Connections:
- net VOUT0-DATA18: now reaches U5.10 (D18)
- net VOUT0-DATA17: now reaches U5.11 (D17)
- net VOUT0-DATA16: now reaches U5.13 (D16)
- net VOUT0-DATA23: now reaches U5.4 (D23)
- net VOUT0-DATA22: now reaches U5.6 (D22)
- net VOUT0-DATA21: now reaches U5.7 (D21)
- net VOUT0-DATA20: now reaches U5.8 (D20)
- net VOUT0-DATA19: now reaches U5.9 (D19)
- no-connect marks 31 -> 23

Commit message: Fix power net names and increase PCB size
Parts:
- J19: footprint Daxxn_Connectors:5019514000 -> Daxxn_Connectors:0541324033
Changed lines of the file:
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@@
       (effects (font (size 1.27 1.27)) (justify left))
     )
-    (property "Footprint" "Daxxn_Connectors:5019514000" (at 88.9 83.82 0)
+    (property "Footprint" "Daxxn_Connectors:0541324033" (at 88.9 83.82 0)
       (effects (font (size 1.27 1.27)) hide)
     )

Commit message: Replacing motherboard and more - SAVE
Parts:
- renumbered C158 to C379, C158 to C380, C159 to C381, C158 to C382, C158 to C383, C158 to C384, C158 to C385, C158 to C386, C156 to C387, C157 to C388, C158 to C389, C159 to C390, C160 to C391, C161 to C392, C158 to C393, FB10 to FB20, Q3 to Q6, R102 to R173, R102 to R174, R102 to R175, R101 to R176, R102 to R177, R103 to R178, R104 to R179, R102 to R180, R102 to R181, R102 to R182, R102 to R183, R102 to R184, R102 to R185, R102 to R186, U4 to U1, U15 to U38, U16 to U39
