File: MotherBoard/BenchyMotherBoard-PCB/BenchyMotherBoard-PCB.kicad_pcb (KiCad board)
At the start: 2 copper layers, 335 parts, among them J1 PWR-CONN, J10 USB3_A, J11 USB3_A, J12 USB3_A, J13 USB_A, J14 USB_A, J15 DISPLAY-FPC, J2 SWD-TAG, J3 Micro_SD_Card_Det, J4 BOOT0-CONN, J5 BOOT1-CONN, J6 BOOT2-CONN, J7 USB3_A, J8 USB3_B, J9 USB3_A, Q1 RQ5A030AP, U1 TPS65400RGZT, U10 AP2127K-3.3, U11 IS43TR16256B-125KBLI, U12 UCS2114, U13 UCS2114, U14 UCS2114, U15 24LC08, U16 USB2412, U17 LM317L, U18 AS321, U2 STM32MP157FAB1, U3 MAX15027, U4 TPS7A94, U5 ATTINY416-MNR, U6 MAX15027, U7 74HCT2G08, U8 MAX15027, Y1 24MHz, Y2 32.7KHz, Y3 25MHz, Y4 25MHz

Commit message: (WIP) Start layout
Parts:
- added C172: 100nF, Capacitor_SMD:C_0402_1005Metric, F.Cu at (-154.1, 251.8)
- added C173: 15pF, Capacitor_SMD:C_0402_1005Metric, F.Cu at (-151.2, 249.9)
- added C174: 10uF, Capacitor_SMD:C_1210_3225Metric, F.Cu at (-109.8, 217.0)
- added C175: 10uF, Capacitor_SMD:C_1210_3225Metric, F.Cu at (-85.2, 193.1)
- added C176: 10uF, Capacitor_SMD:C_1210_3225Metric, F.Cu at (-70.7, 176.2)
- added C177: 10uF, Capacitor_SMD:C_1210_3225Metric, F.Cu at (-70.7, 180.5)
- added D10: GP DIODE, Diode_SMD:D_SOD-123, F.Cu at (-8.17, -3.45)
- added D11: GP DIODE, Diode_SMD:D_SOD-123, F.Cu at (-25.8, 5.00)
- added D12: GP DIODE, Diode_SMD:D_SOD-123, F.Cu at (-10.0, 5.00)
- added D13: GP DIODE, Diode_SMD:D_SOD-123, F.Cu at (-25.8, 8.35)
- added D14: GP DIODE, Diode_SMD:D_SOD-123, F.Cu at (-20.0, 5.00)
- added D9: GP DIODE, Diode_SMD:D_SOD-123, F.Cu at (-25.8, 11.7)
- added J16: TFT-DISPLAY, Daxxn_Connectors:FH12A-20S-0.5SH55, F.Cu at (160.0, 190.0)
- added J17: USB_A, Daxxn_Connectors:1002-014-01000, F.Cu at (125.0, 190.0)
- added J18: COMMS-PWR, Connector_JST:JST_XA_B04B-XASK-1_1x04_P2.50mm_Vertical, F.Cu at (-96.1, 178.3)
- added J19: COMMS-ELOAD, Connector_JST:JST_XA_B04B-XASK-1_1x04_P2.50mm_Vertical, F.Cu at (-96.1, 186.8)
- added J20: COMMS-RELAY, Connector_JST:JST_XA_B04B-XASK-1_1x04_P2.50mm_Vertical, F.Cu at (-111.8, 207.3)
- added J21: COMMS-LOGIC, Connector_JST:JST_XA_B04B-XASK-1_1x04_P2.50mm_Vertical, F.Cu at (-16.2, 213.4)
- added JP2: WP-JMP, Connector_PinSocket_2.54mm:PinSocket_1x03_P2.54mm_Vertical, F.Cu at (-157.8, 247.2)
- added K1: JW2SN, Relay_THT:Relay_DPDT_Panasonic_JW2, F.Cu at (22.8, -46.8)
- added K2: JW2SN, Relay_THT:Relay_DPDT_Panasonic_JW2, F.Cu at (22.8, -17.9)
- added K3: JW2SN, Relay_THT:Relay_DPDT_Panasonic_JW2, F.Cu at (53.1, -46.8)
- added K4: JW2SN, Relay_THT:Relay_DPDT_Panasonic_JW2, F.Cu at (53.1, -61.3)
- added K5: JW2SN, Relay_THT:Relay_DPDT_Panasonic_JW2, F.Cu at (22.8, -61.3)
- added K6: JW2SN, Relay_THT:Relay_DPDT_Panasonic_JW2, F.Cu at (22.8, -32.4)
- added Q10: SSM3K361R_SOT23F, Package_TO_SOT_SMD:SOT-23, F.Cu at (-65.4, 176.3)
- added Q11: MMBT2222A, Package_TO_SOT_SMD:SOT-23, F.Cu at (-92.6, 205.1)
- added Q12: SSM3K361R_SOT23F, Package_TO_SOT_SMD:SOT-23, F.Cu at (-98.3, 213.1)
- added Q13: MMBT2222A, Package_TO_SOT_SMD:SOT-23, F.Cu at (-85.6, 197.5)
- added Q14: SSM3K361R_SOT23F, Package_TO_SOT_SMD:SOT-23, F.Cu at (-12.4, 219.8)
- added Q15: MMBT2222A, Package_TO_SOT_SMD:SOT-23, F.Cu at (-17.3, 219.8)
- added Q2: MMBT2222A, Package_TO_SOT_SMD:SOT-23, F.Cu at (-98.3, 208.6)
- added Q3: RQ5A030AP, Package_TO_SOT_SMD:SOT-23, F.Cu at (-115.9, 228.2)
- added Q4: SSM3K361R_SOT23F, Package_TO_SOT_SMD:SOT-23, F.Cu at (-71.1, 184.8)
- added Q5: MMBT2222A, Package_TO_SOT_SMD:SOT-23, F.Cu at (-104.5, 218.2)
- added Q6: SSM3K361R_SOT23F, Package_TO_SOT_SMD:SOT-23, F.Cu at (-115.9, 223.8)
- added Q7: MMBT2222A, Package_TO_SOT_SMD:SOT-23, F.Cu at (-104.4, 213.7)
- added Q8: SSM3K361R_SOT23F, Package_TO_SOT_SMD:SOT-23, F.Cu at (-111.0, 223.8)
- added Q9: MMBT2222A, Package_TO_SOT_SMD:SOT-23, F.Cu at (-80.0, 191.5)
- added R113: 3K, Resistor_SMD:R_0402_1005Metric, F.Cu at (-151.2, 245.9)
- added R114: 10K, Resistor_SMD:R_0402_1005Metric, F.Cu at (-154.1, 245.9)
- added R115: 12K 1%, Resistor_SMD:R_0402_1005Metric, F.Cu at (-154.1, 247.9)
- added R116: 50K, Resistor_SMD:R_0402_1005Metric, F.Cu at (-136.9, 243.5)
- added R117: 50K, Resistor_SMD:R_0402_1005Metric, F.Cu at (-154.1, 249.9)
- added R118: 1K, Resistor_SMD:R_0402_1005Metric, F.Cu at (-151.2, 247.9)
- added R119: 1K, Resistor_SMD:R_0402_1005Metric, F.Cu at (-77.8, 186.9)
- added R120: 10K, Resistor_SMD:R_0402_1005Metric, F.Cu at (-94.4, 208.3)
- added R121: 200K, Resistor_SMD:R_0402_1005Metric, F.Cu at (-66.4, 179.5)
- added R122: 10K, Resistor_SMD:R_0402_1005Metric, F.Cu at (-94.4, 210.3)
- added R123: 100, Resistor_SMD:R_0402_1005Metric, F.Cu at (-61.5, 175.1)
- added R124: 1K, Resistor_SMD:R_0402_1005Metric, F.Cu at (-122.6, 230.2)
- added R125: 10K, Resistor_SMD:R_0402_1005Metric, F.Cu at (-73.2, 188.0)
- added R126: 100, Resistor_SMD:R_0402_1005Metric, F.Cu at (-88.7, 203.8)
- added R127: 1K, Resistor_SMD:R_0402_1005Metric, F.Cu at (-76.1, 190.9)
- added R128: 10K, Resistor_SMD:R_0402_1005Metric, F.Cu at (-107.1, 221.4)
- added R129: 100, Resistor_SMD:R_0402_1005Metric, F.Cu at (-66.4, 181.5)
- added R130: 1K, Resistor_SMD:R_0402_1005Metric, F.Cu at (-128.4, 230.2)
- added R131: 10K, Resistor_SMD:R_0402_1005Metric, F.Cu at (-111.1, 220.1)
- added R132: 100, Resistor_SMD:R_0402_1005Metric, F.Cu at (-125.5, 230.2)
- added R133: 1K, Resistor_SMD:R_0402_1005Metric, F.Cu at (-76.1, 188.9)
- added R134: 10K, Resistor_SMD:R_0402_1005Metric, F.Cu at (-86.6, 200.7)
- added R135: 100, Resistor_SMD:R_0402_1005Metric, F.Cu at (-112.0, 227.0)
- added R136: 1K, Resistor_SMD:R_0402_1005Metric, F.Cu at (-81.0, 194.7)
- added R137: 10K, Resistor_SMD:R_0402_1005Metric, F.Cu at (-3.72, 210.2)
- added R138: 100, Resistor_SMD:R_0402_1005Metric, F.Cu at (-15.4, 223.1)
- added R139: 1K, Resistor_SMD:R_0402_1005Metric, F.Cu at (-18.3, 223.1)
- added U19: USB2412, Package_DFN_QFN:QFN-28-1EP_5x5mm_P0.5mm_EP3.35x3.35mm, F.Cu at (-111.8, 243.4)
- added U20: MAINS-OUT-1, Daxxn_Connectors:AC-EARTH-DIRECT-WIRE, F.Cu at (-9.55, -18.1)
- added U21: MAINS-IN, Daxxn_Connectors:AC-EARTH-DIRECT-WIRE, F.Cu at (-39.8, 14.2)
- added U22: MAINS-OUT-2, Daxxn_Connectors:AC-EARTH-DIRECT-WIRE, F.Cu at (-39.8, 8.31)
- added U23: MAINS-OUT-3, Daxxn_Connectors:AC-EARTH-DIRECT-WIRE, F.Cu at (-9.55, -12.2)
- added U24: MAINS-OUT-4, Daxxn_Connectors:AC-EARTH-DIRECT-WIRE, F.Cu at (5.00, -29.1)
- added U25: MAINS-OUT-5, Daxxn_Connectors:AC-EARTH-DIRECT-WIRE, F.Cu at (5.00, -35.0)
- added U26: MAINS-OUT-6, Daxxn_Connectors:AC-EARTH-DIRECT-WIRE, F.Cu at (-39.8, 2.39)
- added U9: MAX15027, Package_DFN_QFN:DFN-10-1EP_3x3mm_P0.5mm_EP1.65x2.38mm, F.Cu at (137.5, 47.5)
- C10, C143, C160, C25, C46: value 10uF -> 100nF; footprint Capacitor_SMD:C_1210_3225Metric -> Capacitor_SMD:C_0402_1005Metric
- C11: value 47pF -> 100nF
- C12: value 330pF -> 100nF; footprint Capacitor_SMD:C_0402_1005Metric -> Capacitor_SMD:C_0603_1608Metric
- C120: value 22uF -> 100nF; footprint Capacitor_SMD:C_1210_3225Metric -> Capacitor_SMD:C_0603_1608Metric
- C122: value 100nF -> 22uF; footprint Capacitor_SMD:C_0603_1608Metric -> Capacitor_SMD:C_1210_3225Metric
- C13, C40, C43, C44, C5, C7, C8: footprint Capacitor_SMD:C_0603_1608Metric -> Capacitor_SMD:C_0402_1005Metric
- C132: value 4.7uF -> 100nF; footprint Capacitor_SMD:C_0805_2012Metric -> Capacitor_SMD:C_0603_1608Metric
- C133, C138: value 15pF -> 4.7uF; footprint Capacitor_SMD:C_0402_1005Metric -> Capacitor_SMD:C_0805_2012Metric
- C135: value 1nF -> 15pF
- C136: value 10nF -> 1nF
- C137: value 15pF -> 10nF
- C139, C140, C166: value 10uF -> 15pF; footprint Capacitor_SMD:C_1210_3225Metric -> Capacitor_SMD:C_0402_1005Metric
- C14, C15, C51, C54, C55: footprint Capacitor_SMD:C_0402_1005Metric -> Capacitor_SMD:C_0603_1608Metric
- C141, C150, C151, C152, C155, C164, C17, C57: value 100nF -> 10uF; footprint Capacitor_SMD:C_0402_1005Metric -> Capacitor_SMD:C_1210_3225Metric
- C153, C154: value 100nF -> 1uF; footprint Capacitor_SMD:C_0402_1005Metric -> Capacitor_SMD:C_0805_2012Metric
- C156: value 10uF -> 1uF; footprint Capacitor_SMD:C_1210_3225Metric -> Capacitor_SMD:C_0805_2012Metric
- C157: value 1uF -> 100nF; footprint Capacitor_SMD:C_1210_3225Metric -> Capacitor_SMD:C_0805_2012Metric
- C158, C159, C162: value 15pF -> 100nF
- C16: value 100nF -> 1uF; footprint Capacitor_SMD:C_0402_1005Metric -> Capacitor_SMD:C_1210_3225Metric
- C161, C9: value 1uF -> 100nF; footprint Capacitor_SMD:C_1210_3225Metric -> Capacitor_SMD:C_0402_1005Metric
- C165: value 15pF -> 1uF; footprint Capacitor_SMD:C_0402_1005Metric -> Capacitor_SMD:C_1210_3225Metric
- C167, C170: value 1uF -> 15pF; footprint Capacitor_SMD:C_0805_2012Metric -> Capacitor_SMD:C_0402_1005Metric
- C168: value 1uF -> 10uF; footprint Capacitor_SMD:C_0805_2012Metric -> Capacitor_SMD:C_1210_3225Metric
- C169: value 10uF -> 1uF
- C171: footprint Capacitor_SMD:C_0805_2012Metric -> Capacitor_SMD:C_0402_1005Metric
- C18: value 100nF -> 47pF
- C19, C20, C21, C56: value 100nF -> 1uF; footprint Capacitor_SMD:C_0402_1005Metric -> Capacitor_SMD:C_0603_1608Metric
- C22, C28, C75, C80, C99: value 100nF -> 1uF
- C23: value 100nF -> 330pF; footprint Capacitor_SMD:C_0603_1608Metric -> Capacitor_SMD:C_0402_1005Metric
- C24, C32, C74, C79: value 1uF -> 100nF
- C26: value 117pF -> 100nF; footprint Capacitor_SMD:C_0402_1005Metric -> Capacitor_SMD:C_0603_1608Metric
- C27: value 1nF -> 100nF; footprint Capacitor_SMD:C_0402_1005Metric -> Capacitor_SMD:C_0603_1608Metric
- C29: value 1uF -> 10uF; footprint Capacitor_SMD:C_0603_1608Metric -> Capacitor_SMD:C_1210_3225Metric
- C30: value 1uF -> 117pF; footprint Capacitor_SMD:C_0603_1608Metric -> Capacitor_SMD:C_0402_1005Metric
- C31: value 1uF -> 1nF; footprint Capacitor_SMD:C_0603_1608Metric -> Capacitor_SMD:C_0402_1005Metric
- C41: value 150pF -> 100nF
- C45, C97: value 1uF -> 100nF; footprint Capacitor_SMD:C_0603_1608Metric -> Capacitor_SMD:C_0402_1005Metric
- C47: value 1.5nF -> 100nF
- C52: value 100nF -> 150pF
- C58: value 100nF -> 1.5nF
- C59: value 100nF -> 2.2uF
- C60: value 2.2uF -> 100nF
- C76, C81: value 4.7uF -> 100nF
- C77, C82: value 200nF -> 4.7uF
- C78: value 100nF -> 200nF
- C83: value 100nF -> 200nF; footprint Capacitor_SMD:C_0402_1005Metric -> Capacitor_SMD:C_0603_1608Metric
- J10: value USB3_A -> USB3_B; footprint Connector_USB:USB3_A_Molex_48393-001 -> Daxxn_Connectors:USB-GSB3211311WEU
- J11, J12, J9: footprint Connector_USB:USB3_A_Molex_48393-001 -> Daxxn_Connectors:GSB4116341HR
- J13, J14: value USB_A -> USB3_A; footprint Daxxn_Connectors:1002-014-01000 -> Daxxn_Connectors:GSB4116341HR
- J15: value DISPLAY-FPC -> USB_A; footprint Daxxn_Connectors:046841045100846+ -> Daxxn_Connectors:1002-014-01000
- J3: value Micro_SD_Card_Det -> FILES-SD-CARD; moved to B.Cu
- J7: value USB3_A -> BOOT-SD-CARD; footprint Connector_USB:USB3_A_Molex_48393-001 -> Daxxn_Connectors:microSD_HC_Molex_47219-2001; moved to B.Cu
- J8: value USB3_B -> FAN-CONN; footprint Daxxn_Connectors:USB-GSB3211311WEU -> Connector_JST:JST_NV_B02P-NV_1x02_P5.00mm_Vertical
- JP1: value WP-JMP -> PWR-ICSP-RST; footprint Connector_PinSocket_2.54mm:PinSocket_1x03_P2.54mm_Vertical -> Connector_PinHeader_2.54mm:PinHeader_1x02_P2.54mm_Vertical
- Q1: value RQ5A030AP -> SQ2310ES_SOT23
- R100: value 3K -> 18K
- R102: value 12K 1% -> 10K
- R103: value 50K -> 10K
- R104: value 50K -> 10 1%; footprint Resistor_SMD:R_0402_1005Metric -> Resistor_SMD:R_0805_2012Metric
- R105: value 1K -> 120; footprint Resistor_SMD:R_0402_1005Metric -> Resistor_SMD:R_0805_2012Metric
- R106: value 1K -> 330; footprint Resistor_SMD:R_0402_1005Metric -> Resistor_SMD:R_0805_2012Metric
- R107: footprint Resistor_SMD:R_0402_1005Metric -> Daxxn_Switches:Bourns_TC33X
- R108: value 200K -> 10K
- R109: value 10 1% -> 200K; footprint Resistor_SMD:R_0805_2012Metric -> Resistor_SMD:R_0402_1005Metric
- R110: value 120 -> 200K; footprint Resistor_SMD:R_0805_2012Metric -> Resistor_SMD:R_0402_1005Metric
- R111: value 330 -> 2.2K; footprint Resistor_SMD:R_0805_2012Metric -> Resistor_SMD:R_0402_1005Metric
- R112: value 10K -> 2.2K; footprint Daxxn_Switches:Bourns_TC33X -> Resistor_SMD:R_0402_1005Metric
- R26: value 5K -> 10K
- R27: value 72K -> 5K
- R28: value 10K -> 72K
- R31: value 33K -> 10K
- R32: value 5K -> 33K; footprint Daxxn_Switches:Bourns_TC33X -> Resistor_SMD:R_0402_1005Metric
- R33: value 10K -> 5K; footprint Resistor_SMD:R_0402_1005Metric -> Daxxn_Switches:Bourns_TC33X
- R85: value 2.2K -> 10K
- R86: value 2.2K -> 47K
- R87: value 43K -> 47K
- R88: value 50K -> 47K
- R89, R90: value 18K -> 47K
- R91: value 18K -> 10K
- R92: value 10K -> 100
- R93: value 10K -> 1K
- R94: value 10K -> 43K
- R95: value 10K -> 50K
- R96, R97: value 200K -> 2.2K
- R98, R99: value 2.2K -> 18K
- U10: value AP2127K-3.3 -> USB7206C; footprint Package_TO_SOT_SMD:SOT-23-5 -> Daxxn_Packages:100-VQFN-GND_12X12
- U11: value IS43TR16256B-125KBLI -> AP2127K-3.3; footprint Package_BGA:BGA-96_9.0x13.0mm_Layout2x3x16_P0.8mm -> Package_TO_SOT_SMD:SOT-23-5
- U12: value UCS2114 -> IS43TR16256B-125KBLI; footprint Daxxn_Packages:UCS2114T-1-V_LXVAO-Custom -> Package_BGA:BGA-96_9.0x13.0mm_Layout2x3x16_P0.8mm
- U15: value 24LC08 -> UCS2114; footprint Package_SO:SOIC-8_3.9x4.9mm_P1.27mm -> Daxxn_Packages:UCS2114T-1-V_LXVAO-Custom
- U16: value USB2412 -> LM317L; footprint Package_DFN_QFN:QFN-28-1EP_5x5mm_P0.5mm_EP3.35x3.35mm -> Package_TO_SOT_SMD:SOT-89-3
- U17: value LM317L -> AS321; footprint Package_TO_SOT_SMD:SOT-89-3 -> Package_TO_SOT_SMD:SOT-23-5
- U18: value AS321 -> 24LC08; footprint Package_TO_SOT_SMD:SOT-23-5 -> Package_SO:SOIC-8_3.9x4.9mm_P1.27mm
- U6: value MAX15027 -> SN74LVC1G32; footprint Package_DFN_QFN:DFN-10-1EP_3x3mm_P0.5mm_EP1.65x2.38mm -> Package_TO_SOT_SMD:SOT-23-5
- U7: value 74HCT2G08 -> MAX15027; footprint Package_SO:TSSOP-8_3x3mm_P0.65mm -> Package_DFN_QFN:DFN-10-1EP_3x3mm_P0.5mm_EP1.65x2.38mm
- U8: value MAX15027 -> 74HCT2G08; footprint Package_DFN_QFN:DFN-10-1EP_3x3mm_P0.5mm_EP1.65x2.38mm -> Package_SO:TSSOP-8_3x3mm_P0.65mm
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Connections:
- C100 pad 1: Net-(C100-Pad1) -> VDD
- C101 pad 1: VDD -> Net-(C101-Pad1)
- C102 pad 1: Net-(C102-Pad1) -> VDD
- C103 pad 1: VDD -> Net-(C103-Pad1)
- C104 pad 1: Net-(C104-Pad1) -> VDD
- C105 pad 1: VDD -> Net-(C105-Pad1)
- C108 pad 1: VTT-DDR -> VDD
- C11 pad 1: GND -> VDD
- C11 pad 2: /POWER/COMP1 -> GND
- C12 pad 1: GND -> Net-(C12-Pad1)
- C122 pad 1: VDD -> VTT-DDR
- C13 pad 1: Net-(C13-Pad1) -> GND
- C133 pad 1: GND -> VDD
- C133 pad 2: Net-(C133-Pad2) -> GND
- C134 pad 1: Net-(C134-Pad1) -> GND
- C134 pad 2: GND -> Net-(C134-Pad2)
- C135 pad 2: RESET -> GND
- C136 pad 1: GND -> Net-(C136-Pad1)
- C137 pad 2: Net-(C137-Pad2) -> RESET
- C138 pad 1: Net-(C138-Pad1) -> VDD
- C139 pad 2: VS -> Net-(C139-Pad2)
- C14 pad 1: VDD -> Net-(C14-Pad1)
- C14 pad 2: GND -> VDD
- C140 pad 1: GND -> Net-(C140-Pad1)
- C140 pad 2: Net-(C140-Pad2) -> GND
- C141 pad 2: Net-(C141-Pad2) -> VCC
- C142 pad 2: VS -> Net-(C142-Pad2)
- C144 pad 2: VS -> VCC
- C146 pad 2: VS -> VCC
- C148 pad 2: VS -> VCC
- C150 pad 2: VDD -> VCC
- C151 pad 2: VDD -> Net-(C151-Pad2)
- C152 pad 1: GND -> Net-(C152-Pad1)
- C152 pad 2: VDD -> GND
- C153 pad 1: GND -> Net-(C152-Pad1)
- C153 pad 2: VDD -> GND
- C154 pad 1: GND -> +30V
- C154 pad 2: VDD -> GND
- C155 pad 1: GND -> +30V
- C155 pad 2: VDD -> GND
- C156 pad 1: GND -> Net-(C156-Pad1)
- C156 pad 2: VS -> GND
- C157 pad 1: GND -> +30V
- C157 pad 2: VS -> GND
- C158 pad 1: Net-(C158-Pad1) -> GND
- C158 pad 2: GND -> VDD
- C159 pad 2: Net-(C159-Pad2) -> VDD
- C160 pad 2: VS -> VDD
- C161 pad 2: VS -> VDD
- C162 pad 1: Net-(C162-Pad1) -> GND
- C162 pad 2: GND -> VDD
- C163 pad 2: Net-(C163-Pad2) -> VDD
- C164 pad 2: Net-(C164-Pad2) -> VCC
- C165 pad 2: Net-(C165-Pad2) -> VCC
- C166 pad 1: +30V -> Net-(C166-Pad1)
- C167 pad 1: +30V -> GND
- C167 pad 2: GND -> Net-(C167-Pad2)
- C168 pad 1: Net-(C168-Pad1) -> GND
- C168 pad 2: GND -> VCC
- C169 pad 1: Net-(C168-Pad1) -> GND
- C169 pad 2: GND -> VCC
- C171 pad 1: +30V -> GND
- C171 pad 2: GND -> Net-(C171-Pad2)
- C18 pad 1: VDD -> GND
- C18 pad 2: GND -> /POWER/COMP1
- C21 pad 1: GND -> VDD
- C21 pad 2: Net-(C21-Pad2) -> GND
- C22 pad 1: Net-(C22-Pad1) -> VDD
- C22 pad 2: +30V -> GND
- C23 pad 1: +30V -> GND
- C23 pad 2: GND -> Net-(C23-Pad2)
- C24 pad 1: +30V -> Net-(C24-Pad1)
- C24 pad 2: GND -> Net-(C24-Pad2)
- C25 pad 1: +30V -> GND
- C25 pad 2: GND -> Net-(C25-Pad2)
- C26 pad 1: GND -> Net-(C26-Pad1)
- C26 pad 2: /POWER/COMP2 -> VDD-CORE
- C27 pad 1: GND -> VDD-CORE
- C27 pad 2: Net-(C27-Pad2) -> GND
- C28 pad 1: Net-(C28-Pad1) -> VDD-CORE
- C28 pad 2: Net-(C28-Pad2) -> GND
- C29 pad 1: VDD -> VDD-CORE
- C30 pad 1: VDD -> GND
- C30 pad 2: GND -> /POWER/COMP2
- C31 pad 1: VDD -> GND
- C31 pad 2: GND -> Net-(C31-Pad2)
- C32 pad 1: VDD -> Net-(C32-Pad1)
- C32 pad 2: GND -> Net-(C32-Pad2)
- C40 pad 1: Net-(C40-Pad1) -> VDD-CORE
- C40 pad 2: Net-(C40-Pad2) -> GND
- C41 pad 1: GND -> VDD-CORE
- C41 pad 2: /POWER/COMP4 -> GND
- C42 pad 1: GND -> VDD-CORE
- C42 pad 2: Net-(C42-Pad2) -> GND
- C43 pad 1: Net-(C43-Pad1) -> VDD-CORE
- C43 pad 2: USB-CORE -> GND
- C44 pad 1: USB-CORE -> VDD-CORE
- C45 pad 1: USB-CORE -> VDD-CORE
- C46 pad 1: USB-CORE -> VDD-CORE
- C47 pad 1: GND -> VDD-CORE
- C47 pad 2: Net-(C47-Pad2) -> GND
- C48 pad 1: +30V -> VDD-CORE
- C49 pad 1: +30V -> VDD-CORE
- C5 pad 1: Net-(C5-Pad1) -> VDD
- C5 pad 2: Net-(C5-Pad2) -> GND
- C50 pad 1: +30V -> VDD-CORE
- C51 pad 1: +30V -> Net-(C51-Pad1)
- C51 pad 2: GND -> Net-(C51-Pad2)
- C52 pad 1: +30V -> GND
- C52 pad 2: GND -> /POWER/COMP4
- C53 pad 1: +30V -> GND
- C53 pad 2: GND -> Net-(C53-Pad2)
- C54 pad 1: +30V -> Net-(C54-Pad1)
- C54 pad 2: GND -> USB-CORE
- C55 pad 1: +30V -> USB-CORE
- C56 pad 1: +30V -> USB-CORE
- C57 pad 1: +30V -> USB-CORE
- C58 pad 1: +30V -> GND
- C58 pad 2: GND -> Net-(C58-Pad2)
- C6 pad 1: GND -> VDD
- C6 pad 2: Net-(C6-Pad2) -> GND
- C7 pad 1: Net-(C7-Pad1) -> VDD
- C7 pad 2: VDD -> GND
- C76 pad 1: VDD-DISP -> VDD
- C77 pad 1: Net-(C77-Pad1) -> VDD-DISP
- C78 pad 1: VDD -> Net-(C78-Pad1)
- C81 pad 1: VDDA -> VDD
- C82 pad 1: Net-(C82-Pad1) -> VDDA
- C83 pad 1: USB-CORE -> Net-(C83-Pad1)
- C90 pad 1: VDD -> USB-CORE
- C97 pad 1: VS -> VDD
- C98 pad 1: VDD-USB -> VCC
- C99 pad 1: VDD -> VDD-USB
- D1 pad 2: /USB/USB1-D- -> /USB | DISPLAY/USB1-D-
- D1 pad 4: /USB/USB1-D+ -> /USB | DISPLAY/USB1-D+
- D1 pad 5: /USB/USB1-TX- -> /USB | DISPLAY/USB1-TX-
- D1 pad 6: /USB/USB1-TX+ -> /USB | DISPLAY/USB1-TX+
- D1 pad 7: /USB/USB1-RX- -> /USB | DISPLAY/USB1-RX-
- D1 pad 8: /USB/USB1-RX+ -> /USB | DISPLAY/USB1-RX+
- D2 pad 2: /USB/USB2-D- -> /USB | DISPLAY/USB2-D-
- D2 pad 4: /USB/USB2-D+ -> /USB | DISPLAY/USB2-D+
- D2 pad 5: /USB/USB2-TX- -> /USB | DISPLAY/USB2-TX-
- D2 pad 6: /USB/USB2-TX+ -> /USB | DISPLAY/USB2-TX+
- D2 pad 7: /USB/USB2-RX- -> /USB | DISPLAY/USB2-RX-
- D2 pad 8: /USB/USB2-RX+ -> /USB | DISPLAY/USB2-RX+
- D3 pad 2: /USB/USB3-D- -> /USB | DISPLAY/USB3-D-
- D3 pad 4: /USB/USB3-D+ -> /USB | DISPLAY/USB3-D+
- D3 pad 5: /USB/USB3-TX- -> /USB | DISPLAY/USB3-TX-
- D3 pad 6: /USB/USB3-TX+ -> /USB | DISPLAY/USB3-TX+
- D3 pad 7: /USB/USB3-RX- -> /USB | DISPLAY/USB3-RX-
- D3 pad 8: /USB/USB3-RX+ -> /USB | DISPLAY/USB3-RX+
- D4 pad 2: /USB/USB4-D- -> /USB | DISPLAY/USB4-D-
- D4 pad 4: /USB/USB4-D+ -> /USB | DISPLAY/USB4-D+
- D4 pad 5: /USB/USB4-TX- -> /USB | DISPLAY/USB4-TX-
- D4 pad 6: /USB/USB4-TX+ -> /USB | DISPLAY/USB4-TX+
- D4 pad 7: /USB/USB4-RX- -> /USB | DISPLAY/USB4-RX-
- D4 pad 8: /USB/USB4-RX+ -> /USB | DISPLAY/USB4-RX+
- D5 pad 2: /USB/USB5-D- -> /USB | DISPLAY/USB5-D-
- D5 pad 4: /USB/USB5-D+ -> /USB | DISPLAY/USB5-D+
- D5 pad 5: /USB/USB5-TX- -> /USB | DISPLAY/USB5-TX-
- D5 pad 6: /USB/USB5-TX+ -> /USB | DISPLAY/USB5-TX+
- D5 pad 7: /USB/USB5-RX- -> /USB | DISPLAY/USB5-RX-
- D5 pad 8: /USB/USB5-RX+ -> /USB | DISPLAY/USB5-RX+
- D6 pad 1: /USB/USB-IN1-D+ -> /USB | DISPLAY/USB-IN1-D+
- D6 pad 2: /USB/USB-IN1-D- -> /USB | DISPLAY/USB-IN1-D-
- D6 pad 4: /USB/USB-IN2-D+ -> /USB | DISPLAY/USB-IN2-D+
- D6 pad 5: /USB/USB-IN2-D- -> /USB | DISPLAY/USB-IN2-D-
- ICSP1 pad 5: SUP-RESET -> Net-(ICSP1-Pad5)
- J1 pad 1: VS -> VCC
- J10 pad 1: Net-(C145-Pad2) -> Net-(C143-Pad2)
- J10 pad 2: /USB/USB3-D- -> /USB | DISPLAY/USBU-D-
- J10 pad 3: /USB/USB3-D+ -> /USB | DISPLAY/USBU-D+
- J10 pad 5: /USB/USB3-TX- -> /USB | DISPLAY/USBU-TX-
- J10 pad 6: /USB/USB3-TX+ -> /USB | DISPLAY/USBU-TX+
- J10 pad 8: /USB/USB3-RX- -> /USB | DISPLAY/USBU-RX-
- J10 pad 9: /USB/USB3-RX+ -> /USB | DISPLAY/USBU-RX+
- J11 pad 1: Net-(C147-Pad2) -> Net-(C145-Pad2)
- J11 pad 2: /USB/USB4-D- -> /USB | DISPLAY/USB2-D-
- J11 pad 3: /USB/USB4-D+ -> /USB | DISPLAY/USB2-D+
- J11 pad 5: /USB/USB4-TX- -> /USB | DISPLAY/USB2-TX-
- J11 pad 6: /USB/USB4-TX+ -> /USB | DISPLAY/USB2-TX+
- J11 pad 8: /USB/USB4-RX- -> /USB | DISPLAY/USB2-RX-
- J11 pad 9: /USB/USB4-RX+ -> /USB | DISPLAY/USB2-RX+
- J12 pad 1: Net-(C149-Pad2) -> Net-(C147-Pad2)
- J12 pad 2: /USB/USB5-D- -> /USB | DISPLAY/USB3-D-
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Other:
- copper layers 2 -> 8

Commit message: (WIP) Replaced DDR VRef with reg and started layout
Parts:
- removed D10, D11, D12, D13, D14: GP DIODE, Diode_SMD:D_SOD-123
- removed K1, K2, K3, K4, K5, K6: JW2SN, Relay_THT:Relay_DPDT_Panasonic_JW2
- removed Q10, Q12, Q14, Q4, Q6, Q8: SSM3K361R_SOT23F, Package_TO_SOT_SMD:SOT-23
- removed Q11, Q13, Q15, Q5, Q7, Q9: MMBT2222A, Package_TO_SOT_SMD:SOT-23
- removed R119, R124, R127, R130, R133, R136, R139, R41, R42, R43: 1K, Resistor_SMD:R_0402_1005Metric
- removed R120, R122, R125, R128, R131, R134, R137, R26, R29, R38: 10K, Resistor_SMD:R_0402_1005Metric
- removed R121: 200K, Resistor_SMD:R_0402_1005Metric
- removed R123, R126, R129, R132, R135, R138: 100, Resistor_SMD:R_0402_1005Metric
- removed R27: 5K, Resistor_SMD:R_0402_1005Metric
- removed R28: 72K, Resistor_SMD:R_0402_1005Metric
- removed R39: 6.8K, Resistor_SMD:R_0402_1005Metric
- removed R40: 12K 1%, Resistor_SMD:R_0402_1005Metric
- removed U19: USB2412, Package_DFN_QFN:QFN-28-1EP_5x5mm_P0.5mm_EP3.35x3.35mm
- removed U20: MAINS-OUT-1, Daxxn_Connectors:AC-EARTH-DIRECT-WIRE
- removed U21: MAINS-IN, Daxxn_Connectors:AC-EARTH-DIRECT-WIRE
- removed U22: MAINS-OUT-2, Daxxn_Connectors:AC-EARTH-DIRECT-WIRE
- removed U23: MAINS-OUT-3, Daxxn_Connectors:AC-EARTH-DIRECT-WIRE
- removed U24: MAINS-OUT-4, Daxxn_Connectors:AC-EARTH-DIRECT-WIRE
- removed U25: MAINS-OUT-5, Daxxn_Connectors:AC-EARTH-DIRECT-WIRE
- removed U26: MAINS-OUT-6, Daxxn_Connectors:AC-EARTH-DIRECT-WIRE
- added C178: 10uF, Capacitor_SMD:C_1210_3225Metric, F.Cu at (164.0, 258.8)
- added C179: 10uF, Capacitor_SMD:C_1210_3225Metric, F.Cu at (164.0, 243.8)
- added C180: 10uF, Capacitor_SMD:C_1210_3225Metric, F.Cu at (164.0, 214.0)
- added C181: 10uF, Capacitor_SMD:C_1210_3225Metric, F.Cu at (164.0, 228.8)
- added C182: 100nF, Capacitor_SMD:C_0402_1005Metric, F.Cu at (148.0, 218.5)
- added C183: 100nF, Capacitor_SMD:C_0402_1005Metric, F.Cu at (148.5, 205.5)
- added C184: 10uF, Capacitor_SMD:C_1210_3225Metric, B.Cu at (148.0, 219.8)
- added G***: LOGO, Daxxn_Logos_Art:Daxxn_Logo_N, F.Cu at (224.0, 74.0)
- added J22: COMMS-LOGIC, Daxxn_Connectors:JST_XH_B4B-XH-A_Vertical, F.Cu at (170.0, 210.2)
- added kibuzzard-63F3F2E0: G***, kibuzzard-63F3F2E0, F.Cu at (224.0, 62.0)
- C1, C2, C4, D6, R77, R78: moved to B.Cu
- C100, C105, C111, C112, C113, C114, C115, C116, C117, C118, C119, C12, C120, C127, C128, C129, C130, C131, C132, C14, C15, C24, C26, C27, C32, C35, C36, C51, C54, C55, C60, C74, C76, C78: footprint Capacitor_SMD:C_0603_1608Metric -> Capacitor_SMD:C_0402_1005Metric
- C121, C122: value 22uF -> 100nF; footprint Capacitor_SMD:C_1210_3225Metric -> Capacitor_SMD:C_0402_1005Metric
- C123, C124, C157, C79: value 100nF -> 1uF
- C125, C126: value 100nF -> 22uF; footprint Capacitor_SMD:C_0603_1608Metric -> Capacitor_SMD:C_1210_3225Metric
- C133: value 4.7uF -> 100nF; footprint Capacitor_SMD:C_0805_2012Metric -> Capacitor_SMD:C_0402_1005Metric
- C134, C135, C166, C167: value 15pF -> 100nF
- C136: value 1nF -> 100nF
- C137: value 10nF -> 4.7uF; footprint Capacitor_SMD:C_0402_1005Metric -> Capacitor_SMD:C_0805_2012Metric
- C138: value 4.7uF -> 15pF; footprint Capacitor_SMD:C_0805_2012Metric -> Capacitor_SMD:C_0402_1005Metric
- C140: value 15pF -> 1nF
- C141: value 10uF -> 10nF; footprint Capacitor_SMD:C_1210_3225Metric -> Capacitor_SMD:C_0402_1005Metric
- C142: value 10uF -> 4.7uF; footprint Capacitor_SMD:C_1210_3225Metric -> Capacitor_SMD:C_0805_2012Metric
- C143, C171: value 100nF -> 15pF
- C144, C174, C177: value 10uF -> 15pF; footprint Capacitor_SMD:C_1210_3225Metric -> Capacitor_SMD:C_0402_1005Metric
- C147, C164, C175, C176: value 10uF -> 100nF; footprint Capacitor_SMD:C_1210_3225Metric -> Capacitor_SMD:C_0402_1005Metric
- C153, C154, C156: value 1uF -> 10uF; footprint Capacitor_SMD:C_0805_2012Metric -> Capacitor_SMD:C_1210_3225Metric
- C158, C160: value 100nF -> 1uF; footprint Capacitor_SMD:C_0402_1005Metric -> Capacitor_SMD:C_0805_2012Metric
- C159, C172: value 100nF -> 10uF; footprint Capacitor_SMD:C_0402_1005Metric -> Capacitor_SMD:C_1210_3225Metric
- C16: footprint Capacitor_SMD:C_1210_3225Metric -> Capacitor_SMD:C_0603_1608Metric
- C161: footprint Capacitor_SMD:C_0402_1005Metric -> Capacitor_SMD:C_0805_2012Metric
- C165: value 1uF -> 100nF; footprint Capacitor_SMD:C_1210_3225Metric -> Capacitor_SMD:C_0402_1005Metric
- C173: value 15pF -> 1uF; footprint Capacitor_SMD:C_0402_1005Metric -> Capacitor_SMD:C_1210_3225Metric
- C63: value 1uF -> 4.7uF
- C64: value 100nF -> 10uF; footprint Capacitor_SMD:C_0603_1608Metric -> Capacitor_SMD:C_0805_2012Metric
- C65: value 4.7uF -> 10uF; footprint Capacitor_SMD:C_0603_1608Metric -> Capacitor_SMD:C_0805_2012Metric
- C66: value 200nF -> 10uF; footprint Capacitor_SMD:C_0603_1608Metric -> Capacitor_SMD:C_0805_2012Metric
- C67: value 2.2uF -> 1uF
- C68, C99: value 1uF -> 100nF; footprint Capacitor_SMD:C_0603_1608Metric -> Capacitor_SMD:C_0402_1005Metric
- C69: value 10uF -> 4.7uF
- C73: value 2.2uF -> 200nF; footprint Capacitor_SMD:C_0603_1608Metric -> Capacitor_SMD:C_0402_1005Metric
- C81: footprint Capacitor_SMD:C_0603_1608Metric -> Capacitor_SMD:C_0402_1005Metric; moved to B.Cu
- C82: value 4.7uF -> 100nF; footprint Capacitor_SMD:C_0603_1608Metric -> Capacitor_SMD:C_0402_1005Metric
- C83: value 200nF -> 100nF; footprint Capacitor_SMD:C_0603_1608Metric -> Capacitor_SMD:C_0402_1005Metric
- C96, C97: value 100nF -> 10uF; footprint Capacitor_SMD:C_0402_1005Metric -> Capacitor_SMD:C_0805_2012Metric
- C98: value 1uF -> 1nF; footprint Capacitor_SMD:C_0603_1608Metric -> Capacitor_SMD:C_0402_1005Metric
- D9: value GP DIODE -> ESDLC5V0PB8; footprint Diode_SMD:D_SOD-123 -> Package_DFN_QFN:UDFN-9_1.0x3.8mm_P0.5mm
- J11: value USB3_A -> USB3-PORT2
- J12: value USB3_A -> USB3-PORT3
- J13: value USB3_A -> USB3-PORT4
- J14: value USB3_A -> USB3-PORT5
- J15: value USB_A -> USB-INTERNAL-PORT1
- J17: value USB_A -> USB-INTERNAL-PORT2
- J18, J19: footprint Connector_JST:JST_XA_B04B-XASK-1_1x04_P2.50mm_Vertical -> Daxxn_Connectors:JST_XH_B4B-XH-A_Vertical
- J20: value COMMS-RELAY -> COMMS-SWITCHER; footprint Connector_JST:JST_XA_B04B-XASK-1_1x04_P2.50mm_Vertical -> Daxxn_Connectors:JST_XH_B4B-XH-A_Vertical
- J21: value COMMS-LOGIC -> RELAYS-CONN; footprint Connector_JST:JST_XA_B04B-XASK-1_1x04_P2.50mm_Vertical -> Connector_JST:JST_XH_B8B-XH-A_1x08_P2.50mm_Vertical
- J8: footprint Connector_JST:JST_NV_B02P-NV_1x02_P5.00mm_Vertical -> Connector_PinHeader_2.54mm:PinHeader_1x02_P2.54mm_Vertical
- J9: value USB3_A -> USB3-PORT1
- L1: value 10uH -> 22uH
- R1, R10, R12, R14, R16, R21, R4, R6, R8: footprint Resistor_SMD:R_0603_1608Metric -> Capacitor_SMD:C_0402_1005Metric
- R100, R98, R99: value 18K -> 10K
- R101: value 10K -> 10 1%; footprint Resistor_SMD:R_0402_1005Metric -> Resistor_SMD:R_0805_2012Metric
- R102: value 10K -> 120; footprint Resistor_SMD:R_0402_1005Metric -> Resistor_SMD:R_0805_2012Metric
- R103: value 10K -> 330; footprint Resistor_SMD:R_0402_1005Metric -> Resistor_SMD:R_0805_2012Metric
- R104: value 10 1% -> 10K; footprint Resistor_SMD:R_0805_2012Metric -> Daxxn_Switches:Bourns_TC33X
- R105: value 120 -> 10K; footprint Resistor_SMD:R_0805_2012Metric -> Resistor_SMD:R_0402_1005Metric
- R106: value 330 -> 200K; footprint Resistor_SMD:R_0805_2012Metric -> Resistor_SMD:R_0402_1005Metric
- R107: value 10K -> 200K; footprint Daxxn_Switches:Bourns_TC33X -> Resistor_SMD:R_0402_1005Metric
- R108: value 10K -> 2.2K
- R109: value 200K -> 2.2K
- R110: value 200K -> 3K
- R111: value 2.2K -> 10K
- R112: value 2.2K -> 12K 1%
- R113: value 3K -> 50K
- R114: value 10K -> 50K
- R115: value 12K 1% -> 1K
- R116: value 50K -> 1K
- R117: value 50K -> 10K
- R118: value 1K -> 200K
- R23: value 5K -> 10K
- R32: value 33K -> 10K
- R33: value 5K -> 6.8K; footprint Daxxn_Switches:Bourns_TC33X -> Resistor_SMD:R_0402_1005Metric
- R34: value 1K -> 10K
- R35: value 10K -> 6.8K
- R36: value 6.8K -> 10K
- R37: value 10K -> 12K 1%
- R44, R46: value 1K -> 56
- R45: value 1K -> 100
- R48: value 100 -> 56
- R49, R50: value 56 -> 10K
- R52, R53: value 10K -> 56
- R70, R71: value 56 -> 240 1%
- R73: value 240 1% -> 10K; moved to B.Cu
- R74: value 240 1% -> 47K; moved to B.Cu
- R75: value 56 -> 47K; moved to B.Cu
- R76: value 10K -> 47K; moved to B.Cu
- R79, R80, R81, R89: value 47K -> 100
- R82: value 100 -> 10K
- R83, R84: value 100 -> 47K
- R85: value 10K -> 47K
- R88: value 47K -> 10K
- R90: value 47K -> 1K
- R91: value 10K -> 43K
- R92: value 100 -> 50K
- R93: value 1K -> 2.2K
- R94: value 43K -> 2.2K
- R95: value 50K -> 18K
- R96, R97: value 2.2K -> 18K
- U1: value TPS65400RGZT -> STM32MP157FAB1; footprint Package_DFN_QFN:QFN-48-1EP_7x7mm_P0.5mm_EP5.15x5.15mm_ThermalVias -> Daxxn_Packages:LFBGA354-P0.8mm
- U11: value AP2127K-3.3 -> IS43TR16256B-125KBLI; footprint Package_TO_SOT_SMD:SOT-23-5 -> Package_BGA:BGA-96_9.0x13.0mm_Layout2x3x16_P0.8mm
- U12: value IS43TR16256B-125KBLI -> UCS2114; footprint Package_BGA:BGA-96_9.0x13.0mm_Layout2x3x16_P0.8mm -> Daxxn_Packages:UCS2114T-1-V_LXVAO-Custom
- U15: value UCS2114 -> LM317L; footprint Daxxn_Packages:UCS2114T-1-V_LXVAO-Custom -> Package_TO_SOT_SMD:SOT-89-3
- U16: value LM317L -> AS321; footprint Package_TO_SOT_SMD:SOT-89-3 -> Package_TO_SOT_SMD:SOT-23-5
- U17: value AS321 -> 24LC08; footprint Package_TO_SOT_SMD:SOT-23-5 -> Package_SO:SOIC-8_3.9x4.9mm_P1.27mm
- U18: value 24LC08 -> USB2412; footprint Package_SO:SOIC-8_3.9x4.9mm_P1.27mm -> Package_DFN_QFN:QFN-28-1EP_5x5mm_P0.5mm_EP3.35x3.35mm; moved to B.Cu
- U2: value STM32MP157FAB1 -> TPS65400RGZT; footprint Daxxn_Packages:LFBGA354-P0.8mm -> Package_DFN_QFN:QFN-48-1EP_7x7mm_P0.5mm_EP5.15x5.15mm_ThermalVias
- U3: value MAX15027 -> NCP51200; footprint Package_DFN_QFN:DFN-10-1EP_3x3mm_P0.5mm_EP1.65x2.38mm -> Package_DFN_QFN:DFN-10-1EP_3x3mm_P0.5mm_EP1.7x2.5mm
- U4: value TPS7A94 -> ATTINY416-MNR; footprint Daxxn_Packages:WSON-10-1EP_3x3mm -> Package_DFN_QFN:VQFN-20-1EP_3x3mm_P0.4mm_EP1.7x1.7mm
- U5: value ATTINY416-MNR -> MAX15027; footprint Package_DFN_QFN:VQFN-20-1EP_3x3mm_P0.4mm_EP1.7x1.7mm -> Package_DFN_QFN:DFN-10-1EP_3x3mm_P0.5mm_EP1.65x2.38mm
- U6: value SN74LVC1G32 -> MAX15027; footprint Package_TO_SOT_SMD:SOT-23-5 -> Package_DFN_QFN:DFN-10-1EP_3x3mm_P0.5mm_EP1.65x2.38mm
- U7: value MAX15027 -> SN74LVC1G32; footprint Package_DFN_QFN:DFN-10-1EP_3x3mm_P0.5mm_EP1.65x2.38mm -> Package_TO_SOT_SMD:SOT-23-5
- U9: value MAX15027 -> AP2127K-3.3; footprint Package_DFN_QFN:DFN-10-1EP_3x3mm_P0.5mm_EP1.65x2.38mm -> Package_TO_SOT_SMD:SOT-23-5
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Connections:
- C100 pad 1: VDD -> VREF-DDR
- C101 pad 1: Net-(C101-Pad1) -> VDD-DDR
- C102 pad 1: VDD -> VDD-DDR
- C103 pad 1: Net-(C103-Pad1) -> VDD-DDR
- C104 pad 1: VDD -> VDD-DDR
- C105 pad 1: Net-(C105-Pad1) -> VREF-DDR
- C106 pad 1: VDD -> VDD-DDR
- C107 pad 1: VDD -> VDD-DDR
- C108 pad 1: VDD -> VDD-DDR
- C109 pad 1: VTT-DDR -> VDD-DDR
- C110 pad 1: VTT-DDR -> VDD-DDR
- C12 pad 1: Net-(C12-Pad1) -> /POWER/PWR-CB1
- C12 pad 2: Net-(C12-Pad2) -> /POWER/PWR-SW1
- C123 pad 1: VDD -> VTT-DDR
- C124 pad 1: VDD -> VTT-DDR
- C125 pad 1: VDD -> VTT-DDR
- C126 pad 1: VDD -> VTT-DDR
- C127 pad 1: VDD -> VDD-DDR
- C128 pad 1: VDD -> VDD-DDR
- C129 pad 1: VDD -> VDD-DDR
- C13 pad 2: Net-(C13-Pad2) -> /POWER/PWR-SS1
- C130 pad 1: VDD -> VDD-DDR
- C131 pad 1: VDD -> VDD-DDR
- C132 pad 1: VDD -> VDD-DDR
- C133 pad 1: VDD -> VDD-DDR
- C134 pad 1: GND -> VDD-DDR
- C134 pad 2: Net-(C134-Pad2) -> GND
- C135 pad 1: Net-(C135-Pad1) -> VDD-DDR
- C136 pad 1: Net-(C136-Pad1) -> VDD-DDR
- C136 pad 2: RESET -> GND
- C137 pad 1: GND -> VDD
- C137 pad 2: RESET -> GND
- C138 pad 1: VDD -> GND
- C138 pad 2: GND -> Net-(C138-Pad2)
- C139 pad 1: GND -> Net-(C139-Pad1)
- C139 pad 2: Net-(C139-Pad2) -> GND
- C14 pad 1: Net-(C14-Pad1) -> /POWER/PWR-FB1
- C140 pad 2: GND -> RESET
- C141 pad 2: VCC -> RESET
- C142 pad 1: GND -> VDD
- C142 pad 2: Net-(C142-Pad2) -> GND
- C144 pad 1: GND -> Net-(C144-Pad1)
- C144 pad 2: VCC -> GND
- C145 pad 2: Net-(C145-Pad2) -> VCC
- C146 pad 2: VCC -> /USB | DISPLAY/USBP1-VBUS
- C149 pad 2: Net-(C149-Pad2) -> /USB | DISPLAY/USBP2-VBUS
- C151 pad 2: Net-(C151-Pad2) -> /USB | DISPLAY/USBP3-VBUS
- C152 pad 1: Net-(C152-Pad1) -> GND
- C152 pad 2: GND -> VCC
- C153 pad 1: Net-(C152-Pad1) -> GND
- C153 pad 2: GND -> /USB | DISPLAY/USBP4-VBUS
- C154 pad 1: +30V -> GND
- C154 pad 2: GND -> VCC
- C155 pad 1: +30V -> GND
- C155 pad 2: GND -> /USB | DISPLAY/USBP5-VBUS
- C157 pad 1: +30V -> Net-(C156-Pad1)
- C158 pad 1: GND -> +30V
- C158 pad 2: VDD -> GND
- C159 pad 1: GND -> +30V
- C159 pad 2: VDD -> GND
- C160 pad 1: GND -> Net-(C160-Pad1)
- C160 pad 2: VDD -> GND
- C161 pad 1: GND -> +30V
- C161 pad 2: VDD -> GND
- C164 pad 2: VCC -> VDD
- C165 pad 2: VCC -> VDD
- C166 pad 1: Net-(C166-Pad1) -> GND
- C166 pad 2: GND -> VDD
- C167 pad 2: Net-(C167-Pad2) -> VDD
- C170 pad 1: Net-(C170-Pad1) -> /USB | DISPLAY/USB-IN-XIN
- C171 pad 2: Net-(C171-Pad2) -> /USB | DISPLAY/USB-IN-XOUT
- C172 pad 2: Net-(C172-Pad2) -> VCC
- C173 pad 2: Net-(C173-Pad2) -> VCC
- C174 pad 1: VDD -> Net-(C174-Pad1)
- C175 pad 1: VDD -> GND
- C175 pad 2: GND -> Net-(C175-Pad2)
- C176 pad 1: VDD -> GND
- C176 pad 2: GND -> Net-(C176-Pad2)
- C177 pad 1: VDD -> GND
- C177 pad 2: GND -> Net-(C177-Pad2)
- C24 pad 1: Net-(C24-Pad1) -> /POWER/PWR-CB2
- C24 pad 2: Net-(C24-Pad2) -> /POWER/PWR-SW2
- C25 pad 2: Net-(C25-Pad2) -> /POWER/PWR-SS2
- C26 pad 1: Net-(C26-Pad1) -> /POWER/PWR-FB2
- C32 pad 1: Net-(C32-Pad1) -> /POWER/PWR-CB3
- C32 pad 2: Net-(C32-Pad2) -> /POWER/PWR-SW3
- C34 pad 2: Net-(C34-Pad2) -> /POWER/PWR-SS3
- C35 pad 1: Net-(C35-Pad1) -> /POWER/PWR-FB3
- C35 pad 2: VDD -> VDD-DDR
- C36 pad 1: VDD -> VDD-DDR
- C37 pad 1: VDD -> VDD-DDR
- C38 pad 1: VDD -> VDD-DDR
- C51 pad 1: Net-(C51-Pad1) -> /POWER/PWR-CB4
- C51 pad 2: Net-(C51-Pad2) -> /POWER/PWR-SW4
- C53 pad 2: Net-(C53-Pad2) -> /POWER/PWR-SS4
- C54 pad 1: Net-(C54-Pad1) -> /POWER/PWR-FB4
- C59 pad 1: Net-(C59-Pad1) -> /POWER/VDDA1V1-REG
- C60 pad 1: Net-(C60-Pad1) -> /POWER/VDDG
- C64 pad 1: VDD -> VDD-DDR
- C65 pad 1: VTT-DDR -> VDD-DDR
- C66 pad 1: Net-(C66-Pad1) -> VTT-DDR
- C68 pad 1: VREF-DDR -> VDD
- C69 pad 1: VREF-DDR -> VDD-DISP
- C73 pad 1: Net-(C73-Pad1) -> /POWER/VDD-DISP-SS
- C74 pad 1: VDD -> VDD-PWR
- C77 pad 1: VDD-DISP -> VDDA
- C78 pad 1: Net-(C78-Pad1) -> /POWER/VDDA-SS
- C79 pad 1: VDD -> VCC
- C80 pad 1: VDD -> VDD-USB
- C81 pad 1: VDD -> VDD-PWR
- C82 pad 1: VDDA -> USB-CORE
- C83 pad 1: Net-(C83-Pad1) -> USB-CORE
- C89 pad 1: USB-CORE -> VDD
- C90 pad 1: USB-CORE -> VDD
- C96 pad 1: VDD -> VTT-DDR
- C97 pad 1: VDD -> VTT-DDR
- C98 pad 1: VCC -> Net-(C98-Pad1)
- C99 pad 1: VDD-USB -> VREF-DDR
- D7 pad 2: Net-(D7-Pad2) -> /USB | DISPLAY/USB-SUSP-IND
- D8 pad 2: Net-(D8-Pad2) -> /USB | DISPLAY/USB-HS-IND
- D9 pad 1: VCC -> unconnected-(D9-Pad1)
- D9 pad 2: Net-(D9-Pad2) -> /USB | DISPLAY/DSI-D1-
- ICSP1 pad 1: Net-(ICSP1-Pad1) -> /POWER/PWR-ICSP-COPI
- ICSP1 pad 7: Net-(ICSP1-Pad7) -> /POWER/PWR-ICSP-SCLK
- ICSP1 pad 9: Net-(ICSP1-Pad9) -> /POWER/PWR-ICSP-CIPO
- J10 pad 1: Net-(C143-Pad2) -> Net-(C147-Pad2)
- J11 pad 1: Net-(C145-Pad2) -> /USB | DISPLAY/USBP2-VBUS
- J12 pad 1: Net-(C147-Pad2) -> /USB | DISPLAY/USBP3-VBUS
- J13 pad 1: Net-(C149-Pad2) -> /USB | DISPLAY/USBP4-VBUS
- J14 pad 1: Net-(C151-Pad2) -> /USB | DISPLAY/USBP5-VBUS
- J16 pad 8: /INPUT | OUTPUT/DISP-USB-BUS.TE -> /INPUT | OUTPUT/DISP-BUS.TE
- J16 pad 9: RESET -> /INPUT | OUTPUT/DISP-BUS.RESET
- J18 pad 2: /COMMUNICATIONS/COMMS.PWR-SDA -> /COMMUNICATIONS/PWR-BUS.SDA
- J18 pad 3: /COMMUNICATIONS/COMMS.PWR-SCK -> /COMMUNICATIONS/PWR-BUS.SCK
- J19 pad 2: /COMMUNICATIONS/COMMS.ELOAD-SDA -> /COMMUNICATIONS/ELOAD-BUS.SDA
- J19 pad 3: /COMMUNICATIONS/COMMS.ELOAD-SCK -> /COMMUNICATIONS/ELOAD-BUS.SCK
- J20 pad 2: /COMMUNICATIONS/COMMS.RELAY-SDA -> /COMMUNICATIONS/SWITCHER-BUS.SDA
- J20 pad 3: /COMMUNICATIONS/COMMS.RELAY-SCK -> /COMMUNICATIONS/SWITCHER-BUS.SCK
- J21 pad 2: /COMMUNICATIONS/COMMS.LOGIC-SDA -> /COMMUNICATIONS/RELAY-BUS.1
- J21 pad 3: /COMMUNICATIONS/COMMS.LOGIC-SCK -> /COMMUNICATIONS/RELAY-BUS.2
- J21 pad 4: GND -> /COMMUNICATIONS/RELAY-BUS.3
- J4 pad 2: Net-(J4-Pad2) -> /INPUT | OUTPUT/BOOT0-JMP
- J5 pad 2: Net-(J5-Pad2) -> /INPUT | OUTPUT/BOOT1-JMP
- J6 pad 2: Net-(J6-Pad2) -> /INPUT | OUTPUT/BOOT2-JMP
- J9 pad 1: Net-(C142-Pad2) -> /USB | DISPLAY/USBP1-VBUS
- L1 pad 1: Net-(C12-Pad2) -> /POWER/PWR-SW1
- L2 pad 1: Net-(C24-Pad2) -> /POWER/PWR-SW2
- L3 pad 1: Net-(C32-Pad2) -> /POWER/PWR-SW3
- L3 pad 2: VDD -> VDD-DDR
- L4 pad 1: Net-(C51-Pad2) -> /POWER/PWR-SW4
- R1 pad 2: Net-(C14-Pad1) -> /POWER/PWR-FB1
- R10 pad 1: VDD -> VDD-DDR
- R10 pad 2: Net-(C35-Pad1) -> /POWER/PWR-FB3
- R100 pad 2: GND -> VDD
- R101 pad 1: Net-(R101-Pad1) -> Net-(C156-Pad1)
- R101 pad 2: VDD -> Net-(Q3-Pad3)
- R102 pad 2: VDD -> Net-(Q3-Pad1)
- R103 pad 1: Net-(R103-Pad1) -> /USB | DISPLAY/USB-BUS.BRIGHT
- R103 pad 2: VDD -> Net-(C160-Pad1)
- R104 pad 1: Net-(C152-Pad1) -> Net-(C156-Pad1)
- R104 pad 2: Net-(Q3-Pad3) -> Net-(R104-Pad2)
- R105 pad 1: Net-(R105-Pad1) -> GND
- R105 pad 2: Net-(Q3-Pad1) -> Net-(R105-Pad2)
- R106 pad 1: /INPUT | OUTPUT/DISP-USB-BUS.BRIGHT -> GND
- R106 pad 2: Net-(C156-Pad1) -> Net-(R106-Pad2)
- R107 pad 1: Net-(C152-Pad1) -> GND
- R108 pad 1: GND -> Net-(R108-Pad1)
- R108 pad 2: Net-(R108-Pad2) -> VDD
- R109 pad 1: GND -> Net-(R109-Pad1)
- R109 pad 2: Net-(R109-Pad2) -> VDD
- R110 pad 1: GND -> /USB | DISPLAY/USB-RREF
- R110 pad 2: Net-(R110-Pad2) -> GND
- R111 pad 1: Net-(R111-Pad1) -> /INPUT | OUTPUT/USB-BUS.RESET
- R112 pad 2: VDD -> GND
- R113 pad 1: Net-(R113-Pad1) -> /USB | DISPLAY/USB-SUSP-IND
- R114 pad 1: /INPUT | OUTPUT/DISP-USB-BUS.USB-RESET -> /USB | DISPLAY/USB-NONREM1
- R114 pad 2: VDD -> GND
- R115 pad 1: Net-(R115-Pad1) -> Net-(D7-Pad1)
- R116 pad 1: Net-(D7-Pad2) -> Net-(D8-Pad1)
- R117 pad 1: Net-(R117-Pad1) -> GND
- R117 pad 2: GND -> Net-(R117-Pad2)
- R118 pad 1: Net-(D7-Pad1) -> GND
- R118 pad 2: GND -> Net-(R118-Pad2)
- R12 pad 2: Net-(C35-Pad1) -> /POWER/PWR-FB3
- R14 pad 2: Net-(C54-Pad1) -> /POWER/PWR-FB4
- R16 pad 2: Net-(C54-Pad1) -> /POWER/PWR-FB4
- R17 pad 2: /POWER/PWR-I2C-SDA -> /POWER/PMBUS-SDA
- R18 pad 2: /POWER/PWR-I2C-SCK -> /POWER/PMBUS-SCK
- R19 pad 2: Net-(R19-Pad2) -> /POWER/PWR-CLK-OUT
- R20 pad 1: Net-(R20-Pad1) -> /POWER/PWR-CE
- R21 pad 1: Net-(R21-Pad1) -> /POWER/PMBUS-ADDR
- R22 pad 2: Net-(R22-Pad2) -> /POWER/PWR-RCLK-SY
- R23 pad 1: VTT-DDR -> Net-(C98-Pad1)
- R23 pad 2: Net-(R23-Pad2) -> VDD-DDR
- R24 pad 1: Net-(R23-Pad2) -> Net-(C98-Pad1)
- R25 pad 1: GND -> VDD
- R25 pad 2: /POWER/VDD-DDR-EN -> /POWER/VDD-DDR-PG
- R3 pad 1: Net-(R3-Pad1) -> /POWER/PWR-EN1
- R30 pad 1: GND -> VDD-PWR
- R30 pad 2: /POWER/VDD-DDR-EN -> /POWER/PWR-SWITCH
- R31 pad 1: VDD-PWR -> VDD-DISP
- R31 pad 2: POWER-RESET -> /POWER/VDD-DISP-FB
- R32 pad 1: Net-(R28-Pad2) -> VDD-PWR
- R32 pad 2: GND -> POWER-RESET
- R33 pad 1: Net-(C73-Pad1) -> /POWER/VDD-DISP-FB
- R33 pad 2: Net-(R33-Pad2) -> GND
- R34 pad 1: Net-(R33-Pad2) -> VDDA
- R34 pad 2: GND -> /POWER/VDDA-FB
- R35 pad 1: VDD-DISP -> /POWER/VDDA-FB
- R35 pad 2: Net-(R35-Pad2) -> GND
- R36 pad 1: Net-(R35-Pad2) -> VDD-PWR
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Routing:
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- added copper zone on F.Cu, net /POWER/PWR-SW1
- added copper zone on F.Cu, net /POWER/PWR-SW2
- added copper zone on F.Cu, net /POWER/PWR-SW3
- added copper zone on F.Cu, net /POWER/PWR-SW4
- added copper zone on F.Cu, net USB-CORE
- added copper zone on F.Cu, net VDD
- added copper zone on F.Cu, net VDD-CORE
- added copper zone on F.Cu, net VDD-DDR
- added copper zone on F.Cu, net VPWR
Other:
- board outline added: 160 x 100 mm
- board text added: "2"
- board text added: "3"
- board text added: "4"
- board text added: "5"
- board text added: "6"
- board text added: "7"
- board text added: "BGA SIGNAL BREAKOUT"
- board text added: "BOT - 8"
- board text added: "BOTTOM LAYER FOOTPRINTS / SIGNALS"
- board text added: "DDR3 SIGNAL BREAKOUT"
- board text added: "DESCRIPTION"
- board text added: "GND/PWR"
- board text added: "GROUND"
- board text added: "GROUND PLANE 1"
- board text added: "GROUND PLANE 2 / POWER PLANES"
- board text added: "GROUND PLANE 3"
- board text added: "GROUND PLANE 4"
- board text added: "LAYER"
- board text added: "SIGNAL"
- board text added: "STACK-UP"
- board text added: "TOP - 1"
- board text added: "TOP LAYER FOOTPRINTS / SIGNALS"
- board text added: "TYPE"
