File: MotherBoard/BenchyMotherBoard-PCB/power.kicad_sch (KiCad schematic)
At the start: 61 parts

Commit message: Add MORE regulators, USB, Display, and SDCard
Parts:
- removed C? (x3): 100nF, Capacitor_SMD:C_0603_1608Metric, symbol Device:C_Small
- removed R?: 10K, Resistor_SMD:R_0603_1608Metric, symbol Device:R_Small_US
- added C? (x25): 100nF, Capacitor_SMD:C_0402_1005Metric, symbol Device:C_Small
- added C? (x10): 1uF, Capacitor_SMD:C_0603_1608Metric, symbol Device:C_Small
- added C? (x7): 100nF, Capacitor_SMD:C_0603_1608Metric, symbol Device:C_Small
- added C? (x3): 4.7uF, Capacitor_SMD:C_0603_1608Metric, symbol Device:C_Small
- added C? (x2): 2.2uF, Capacitor_SMD:C_0603_1608Metric, symbol Device:C_Small
- added C? (x3): 200nF, Capacitor_SMD:C_0603_1608Metric, symbol Device:C_Small
- added C?: 10uF, Capacitor_SMD:C_1210_3225Metric, symbol Device:C_Small
- added C? (x3): 10uF, Capacitor_SMD:C_0603_1608Metric, symbol Device:C_Small
- added C?: 47uF, Capacitor_SMD:CP_Elec_6.3x7.7, symbol Device:C_Polarized_Small
- added J?: PWR-CONN, Daxxn_Connectors:4-Pin_Molex_Mini-Fit_Jr_Vertical_Mount, symbol Connector_Generic:Conn_02x02_Odd_Even
- added R? (x16): 10K, Resistor_SMD:R_0402_1005Metric, symbol Device:R_Small_US
- added R?: 30K, Daxxn_Switches:Bourns_TC33X, symbol Daxxn_Other:R_Pot_Small_US
- added R?: 10K, Resistor_SMD:R_0603_1608Metric, symbol Device:R_Small_US
- added R? (x2): 6.8K, Resistor_SMD:R_0402_1005Metric, symbol Device:R_Small_US
- added R?: 12K 1%, Resistor_SMD:R_0402_1005Metric, symbol Device:R_Small_US
- added R?: 5K, Daxxn_Switches:Bourns_TC33X, symbol Daxxn_Other:R_Pot_Small_US
- added R?: 72K, Resistor_SMD:R_0402_1005Metric, symbol Device:R_Small_US
- added R?: 1K, Resistor_SMD:R_0402_1005Metric, symbol Device:R_Small_US
- added R? (x3): 5K, Resistor_SMD:R_0402_1005Metric, symbol Device:R_Small_US
- added R?: 33K, Resistor_SMD:R_0402_1005Metric, symbol Device:R_Small_US
- added U?: USB7206C, SnapEDA:QFN40P1200X1200X90-101N, symbol Daxxn_IC:USB7206C
- added U?: TLV3401, Package_TO_SOT_SMD:SOT-23-5, symbol Daxxn_OPAMP:TLV3401
- added U? (x3): MAX15027, Package_DFN_QFN:DFN-10-1EP_3x3mm_P0.5mm_EP1.65x2.38mm, symbol Daxxn_Regulators:MAX15027
- added U?: LM317L_SOT-89, Package_TO_SOT_SMD:SOT-89-3, symbol Regulator_Linear:LM317L_SOT-89
- C?: footprint Capacitor_SMD:C_0603_1608Metric -> Capacitor_SMD:C_0402_1005Metric
- L? (x4): value 22uH -> 10uH
Connections:
- net VDDQ-DDR is gone; now on net VDD-DDR: U?.E15 (VDDQ-DDR), U?.F14 (VDDQ-DDR), U?.G15 (VDDQ-DDR), U?.H14 (VDDQ-DDR), U?.J15 (VDDQ-DDR), U?.K14 (VDDQ-DDR), U?.L15 (VDDQ-DDR), U?.M14 (VDDQ-DDR), U?.N15 (VDDQ-DDR), U?.P14 (VDDQ-DDR), U?.R15 (VDDQ-DDR)
- net +30V: now also J?.3 (Pin_3)
- net GND: now also C?.1, U?.11 (GND), U?.6 (GND), C?.1, C?.1, C?.1, C?.1, C?.1, C?.1, C?.1, C?.1, C?.1, C?.1, C?.1, C?.2, C?.2, C?.2, C?.2, C?.2, C?.2, C?.2, C?.2, C?.2, C?.2, C?.2, C?.2, C?.2, C?.2, C?.2, C?.2, C?.2, C?.2, C?.2, C?.2, C?.2, C?.2, C?.2, C?.2, C?.2, C?.2, C?.2, C?.2, C?.2, C?.2, C?.2, C?.2, C?.2, C?.2, C?.2, C?.2, C?.2, C?.2, C?.2, C?.2, C?.2, C?.2, C?.2, C?.2, J?.4 (Pin_4), R?.1, R?.2, R?.2, R?.2, R?.2, R?.2, R?.2, R?.2, R?.2, R?.2, R?.2, R?.2, R?.2, R?.3, U?.101 (GND), U?.11 (GND), U?.11 (GND), U?.11 (GND), U?.2 (V-), U?.4 (GND), U?.4 (GND), U?.4 (GND), U?.8 (GND), U?.8 (GND), U?.8 (GND)
- net VCC: now also C?.1, C?.1, J?.1 (Pin_1), U?.3 (VI)
- net VDD: now also U?.1 (IN), U?.2 (IN), U?.A12 (VDD-DSI), U?.G13 (VDD-PLL2), U?.J5 (VDD-PLL), U?.N3 (VREF+), C?.1, C?.1, C?.1, C?.1, C?.1, C?.1, C?.1, C?.1, C?.1, C?.1, C?.1, C?.1, C?.1, C?.1, C?.1, C?.1, C?.1, C?.1, C?.1, R?.1, R?.1, R?.1, R?.2, U?.1 (IN), U?.1 (IN), U?.1 (IN), U?.2 (IN), U?.2 (IN), U?.2 (IN), U?.26 (VDD33), U?.3 (IN), U?.3 (IN), U?.3 (IN), U?.43 (VDD33), U?.5 (V+), U?.53 (VDD33), U?.62 (VDD33), U?.67 (VDD33), U?.79 (VDD33), U?.88 (VDD33), U?.99 (VDD33)
- net VPWR: now also C?.1, C?.1
- net USB-CORE: now reaches C?.1, C?.1, C?.1, L?.2, R?.1
- net USB-CORE: now also C?.1, C?.1, C?.1, C?.1, C?.1, C?.1, C?.1, U?.18 (VCORE), U?.25 (VCORE), U?.31 (VCORE), U?.38 (VCORE), U?.55 (VCORE), U?.78 (VCORE), U?.85 (VCORE), U?.9 (VCORE), U?.93 (VCORE)
- net at U?.A16 (VDD1V2_DSI-PHY): now also U?.B16 (VDD1V2-DSI-REG)
- net VDDA-PWR: now reaches U?.L3 (VDD-ANA)
- net VDDA-PWR: now also U?.19 (VDDA), U?.M4 (VDDA), C?.1
- net VREF-DDR: now reaches U?.10 (OUT)
- net VREF-DDR: now also U?.8 (SNS), U?.9 (OUT), C?.1, C?.1, R?.1
- net at U?.3 (EN_UV): now also R?.2, R?.2
- net VREF-DDR-PG: now reaches U?.4 (PG)
- net VREF-DDR-PG: now also R?.1
- net at U?.5 (FB_PG): now also R?.1, R?.2
- net at U?.7 (NR/SS): now also C?.1, R?.1
- net at C?.2: now also U?.45 (SS1)
- net PMBUS-SDA: now reaches R?.2, U?.43 (SCL)
- net PMBUS-SCLK: now reaches R?.2, U?.42 (SDA)
- net PWR-DELAY: now reaches U?.13 (ENSW2)
- net PWR-DELAY: now also U?.27 (ENSW3), R?.1, R?.1, R?.2, U?.1 (OUT)
- net COMP2: now reaches U?.15 (COMP2)
- net COMP2: now also C?.2, R?.1
- net at U?.16 (SS2): now also C?.2
- net PWR-GOOD: now reaches U?.17 (PGOOD)
- net PWR-GOOD: now also R?.1, U?.5 (EN), U?.5 (EN), U?.5 (EN)
- net VDD-PWR: now reaches U?.20 (VDDD)
- net VDD-PWR: now also C?.1, J?.2 (Pin_2)
- net KILL-YOURSELF: now reaches U?.23 (CE)
- net at U?.24 (SS3): now also C?.2
- net COMP3: now reaches U?.25 (COMP3)
- net COMP3: now also C?.2, R?.1
- net at U?.34 (ENSW4): now also R?.1
- net COMP4: now reaches U?.36 (COMP4)
- net COMP4: now also C?.2, R?.1
- net at U?.37 (SS4): now also C?.2
- net RESET: now reaches U?.39 (~{RESET})
- net PMBUS-ALERT: now reaches U?.41 (I2CALERT)
- net COMP1: now reaches U?.46 (COMP1)
- net COMP1: now also C?.2, R?.1
- net at U?.48 (ENSW1/ENSEQ): now also R?.1
- new net: R?.1, R?.2, U?.7 (FB) (x3)
- new net: R?.1, U?.100 (RBIAS)
- new net: R?.1, R?.2, U?.4 (IN-)
- new net: C?.1, R?.2, U?.3 (IN+)
- new net: C?.1, U?.6 (SS) (x3)
- new net: C?.2, R?.2 (x4)
- new net: R?.1, R?.2, U?.1 (ADJ)
- new net: R?.1, R?.2, R?.3
- new net VDD-DISP: C?.1, C?.1, R?.1, U?.2 (VO)
- new net VDDA-ETH: C?.1, C?.1, R?.1, R?.1, U?.10 (OUT), U?.10 (OUT), U?.9 (OUT), U?.9 (OUT)
- new net VTT-DDR: C?.1, R?.1, U?.10 (OUT), U?.9 (OUT)
Other:
- note added: "+30V"
- note added: "0.75V"
- note added: "1.1V"
- note added: "1.2V"
- note added: "1.3V"
- note added: "1.5V"
- note added: "1.8V"
- note added: "12V"
- note added: "2.5V"
- note added: "2.5V-3.3V"
- note added: "3.3V"
- note added: "30V"
- note added: "Analog Adjustable Reference"
- note added: "Analog Main Supply"
- note added: "DDR3 Memory Digital Supply"
- note added: "High Voltage Supply For The Display Backlight"
- note added: "MPU Core Supply"
- note added: "Main Supply"
- note added: "Main Supply from External SMPS"
- note added: "POWER RAILS"
- note added: "Supply For DDR3 Pullup Resistors"
- note added: "Supply For Ethernet Analog Layer"
- note added: "Supply For Ethernet Digital Layer"
- note added: "Supply For The Display Logic & LCD Screen."
- note added: "USB Hub Core Supply"
- note added: "USB-CORE"
- note added: "VDD"
- note added: "VDD-CORE"
- note added: "VDD-DDR"
- note added: "VDD-DISP"
- note added: "VDD-ETH"
- note added: "VDDA"
- note added: "VDDA-ETH"
- note added: "VPWR"
- note added: "VREF"
- note added: "VTT-DDR"
- moved on the sheet: C?, R?, U?

Commit message: Initial schematic lock
Parts:
- removed C? (x2): 1uF, Capacitor_SMD:C_0603_1608Metric, symbol Device:C_Small
- removed C? (x2): 10uF, Capacitor_SMD:C_0603_1608Metric, symbol Device:C_Small
- removed C? (x2): 100nF, Capacitor_SMD:C_0603_1608Metric, symbol Device:C_Small
- removed R? (x5): 30K, Daxxn_Switches:Bourns_TC33X, symbol Daxxn_Other:R_Pot_Small_US
- removed R?: 10K, Resistor_SMD:R_0603_1608Metric, symbol Device:R_Small_US
- removed R? (x3): 10K, Resistor_SMD:R_0402_1005Metric, symbol Device:R_Small_US
- removed R?: 5K, Resistor_SMD:R_0402_1005Metric, symbol Device:R_Small_US
- removed U?: TLV3401, Package_TO_SOT_SMD:SOT-23-5, symbol Daxxn_OPAMP:TLV3401
- removed U?: LM317L_SOT-89, Package_TO_SOT_SMD:SOT-89-3, symbol Regulator_Linear:LM317L_SOT-89
- added C22, C35, C43, C7, C78, C?: 100nF, Capacitor_SMD:C_0603_1608Metric, symbol Device:C_Small
- added C70, C71, C72: 100nF, Capacitor_SMD:C_0402_1005Metric, symbol Device:C_Small
- added C97, C98: 1uF, Capacitor_SMD:C_0603_1608Metric, symbol Device:C_Small
- added ICSP1: ICSP, Connector:Tag-Connect_TC2050-IDC-FP_2x05_P1.27mm_Vertical, symbol Daxxn_Connectors:ICSP
- added JP?: PWR-ICSP-RST, Connector_PinHeader_2.54mm:PinHeader_1x02_P2.54mm_Vertical, symbol Jumper:Jumper_2_Open
- added R1: 24K, Resistor_SMD:R_0603_1608Metric, symbol Device:R_Small_US
- added R10: 13K, Resistor_SMD:R_0603_1608Metric, symbol Device:R_Small_US
- added R14: 4.3K, Resistor_SMD:R_0603_1608Metric, symbol Device:R_Small_US
- added R19, R20, R25, R30, R33, R37: 10K, Resistor_SMD:R_0402_1005Metric, symbol Device:R_Small_US
- added R22: 160K, Resistor_SMD:R_0402_1005Metric, symbol Device:R_Small_US
- added R6: 6.2K, Resistor_SMD:R_0603_1608Metric, symbol Device:R_Small_US
- added S1: POWER SWITCH, Daxxn_Switches:TL3365AF180QG, symbol Daxxn_Buttons:GENERIC-SWITCH-2P
- added U10: AP2127K-3.3, Package_TO_SOT_SMD:SOT-23-5, symbol Regulator_Linear:AP2127K-3.3
- added U5: ATTINY416-MNR, Package_DFN_QFN:VQFN-20-1EP_3x3mm_P0.4mm_EP1.7x1.7mm, symbol Daxxn_MicroControllers:ATTINY416-MNR
- added U7: 74HCT2G08, Package_SO:TSSOP-8_3x3mm_P0.65mm, symbol Daxxn_Logic:74HCT2G08
- added U?: SN74LVC1G32, Package_TO_SOT_SMD:SOT-23-5, symbol Daxxn_Logic:SN74LVC1G32
- C11: renamed from C?; value 100nF -> 47pF
- C12: renamed from C?; value 100nF -> 330pF
- C26: renamed from C?; value 100nF -> 117pF
- C27: renamed from C?; value 100nF -> 1nF
- C33: renamed from C?; value 100nF -> 100pF
- C39: renamed from C?; value 100nF -> 820pF
- C41: renamed from C?; value 100nF -> 150pF
- C47: renamed from C?; value 100nF -> 1.5nF
- R12: renamed from R?; value 10K -> 15K
- R13: renamed from R?; value 10K -> 8.2K
- R16: renamed from R?; value 10K -> 11K
- R2: renamed from R?; value 10K -> 24K
- gave numbers to parts that had none: 117
Connections:
- net +30V: no longer C23.1, C24.1, C25.1, C48.1, C49.1, C50.1, C51.1, C52.1, C53.1, C54.1, C55.1, C56.1, C57.1, C58.1, L2.2, U2.E11 (VDDCORE), U2.E13 (VDDCORE), U2.E7 (VDDCORE), U2.E9 (VDDCORE), U2.F10 (VDDCORE), U2.F12 (VDDCORE), U2.F4 (VDDCORE), U2.F6 (VDDCORE), U2.F8 (VDDCORE), U2.G11 (VDDCORE), U2.G5 (VDDCORE), U2.G7 (VDDCORE), U2.G9 (VDDCORE), U2.H10 (VDDCORE), U2.H12 (VDDCORE), U2.H4 (VDDCORE), U2.H6 (VDDCORE), U2.H8 (VDDCORE), U2.J11 (VDDCORE), U2.J13 (VDDCORE), U2.J7 (VDDCORE), U2.J9 (VDDCORE), U2.K10 (VDDCORE), U2.K12 (VDDCORE), U2.K8 (VDDCORE), U2.L11 (VDDCORE), U2.L13 (VDDCORE), U2.L9 (VDDCORE), U2.M10 (VDDCORE), U2.M12 (VDDCORE), U2.N11 (VDDCORE), U2.N13 (VDDCORE), U2.P12 (VDDCORE), U2.R13 (VDDCORE)
- net GND: now also U2.T15 (BYPASS-REG1V8), C70.2, C71.2, C72.2, C78.2, C97.2, C98.2, C?.2, ICSP1.10 (GND), ICSP1.4 (GND), ICSP1.6 (GND), ICSP1.8 (GND), R22.1, R25.1, S1.2, U10.2 (GND), U5.21 (GND), U5.3 (GND), U7.4, U?.3
- net PMBUS-ALERT: now also U5.7 (PA6)
- net RESET: now also U?.2; no longer U1.39 (~{RESET})
- net USB-CORE: now also C43.2, R14.1
- net VCC: now also C97.1, U10.1 (VIN)
- net VDD: now also U2.H3 (VBAT), U2.N1 (PDR-ON-CORE), U2.N2 (PDR-ON), C7.2, C78.1, C?.1, R1.1, U7.8, U?.5; no longer U2.A12 (VDD-DSI), U2.N3 (VREF+)
- net VDD-DDR: now also C35.2, R10.1
- net VDD-DISP: now also C76.1, R35.1, U6.10 (OUT), U6.9 (OUT)
- net VDD-PWR: now also C70.1, C71.1, C72.1, ICSP1.2 (VCC), R19.1, R20.2, R30.1, R33.1, R37.1, U5.4 (VDD); no longer J1.2 (Pin_2)
- net VDDA-PWR: no longer U2.L3 (VDD-ANA), U2.M4 (VDDA)
- net VPWR: now also J1.2 (Pin_2)
- net VDDA1V8-REG: now reaches C61.1, C62.1, U2.B12 (VDDA1V8-DSI), U2.V11 (VDDA1V8-REG)
- net VDD-USB: now reaches U2.W12 (VDD3V3-USBHS)
- net VDD-USB: now also U2.W15 (VDD3V3-USBFS), C98.1, U10.5 (VOUT)
- net at R16.2, U1.35 (VFB4): now also C43.1, R14.2
- net VDD-USB-CORE-EN: now reaches R15.1, U1.34 (ENSW4)
- net VDD-USB-CORE-EN: now also U5.16 (PC1)
- net at R8.2, U1.14 (VFB2): now also C22.1, R6.2
- net at R12.2, U1.26 (VFB3): now also C35.1, R10.2
- net VDD-DDR-EN: now reaches R26.2, R29.2, U4.3 (EN_UV)
- net VDD-DDR-EN: now also R11.1, U1.27 (ENSW3), U3.5 (EN), R25.2, U5.17 (PC2)
- net at R4.2, U1.47 (VFB1): now also C7.1, R1.2
- net at U1.40 (RCLOCK_SYNC): now also R22.2
- net at U1.44 (CLK-OUT): now also R19.2
- net KILL-YOURSELF: no longer names the net of U1.23 (CE)
- net KILL-YOURSELF: now also R20.1
- net PMBUS-SCLK renamed PWR-I2C-SDA
- net PWR-I2C-SDA: now also U5.13 (PB1)
- net PMBUS-SDA renamed PWR-I2C-SCK
- net PWR-I2C-SCK: now also U5.14 (PB0)
- net PWR-DELAY renamed PWR-ON
- net PWR-ON: now also U2.L1 (PWR-ON), U5.6 (PA5); no longer R11.1, U1.27 (ENSW3)
- removed net PWR-GOOD: U1.17 (PGOOD), U3.5 (EN), U6.5 (EN), U8.5 (EN)
- net VDDA-ETH renamed VDDA
- net VDDA: now also U2.A12 (VDD-DSI), U2.L3 (VDD-ANA), U2.M4 (VDDA), U2.N3 (VREF+); no longer C76.1, R35.1, U6.10 (OUT), U6.9 (OUT)
- net VREF-DDR-PG renamed VDD-DDR-PG
- net VDD-DDR-PG: now also U5.15 (PC0)
- new net: ICSP1.9 (CIPO), U5.1 (PA2)
- new net: ICSP1.7 (SCLK), U5.2 (PA3)
- new net: ICSP1.1 (COPI), U5.20 (PA1)
- new net: ICSP1.5 (RESET), JP?.2 (B)
- new net ALL-PGOOD: R37.2, U5.10 (PB4), U7.3 (Y)
- new net POWER-RESET: JP?.1 (A), R30.2, U1.39 (~{RESET}), U5.19 (~{RESET})
- new net PWR-BUS.RX: U5.12 (PB2)
- new net PWR-BUS.TX: U5.11 (PB3)
- new net PWR-LP: U2.P1 (PWR-LP), U?.1
- new net PWR-ON-RST: U5.5 (PA4), U?.4
- new net PWR-SWITCH: R33.2, S1.1, U5.8 (PA7)
- new net SMPS-PGOOD: U1.17 (PGOOD), U7.6 (B)
- new net VDD-CORE: C22.2, C23.1, C24.1, C25.1, C48.1, C49.1, C50.1, C51.1, C52.1, C53.1, C54.1, C55.1, C56.1, C57.1, C58.1, L2.2, R6.1, U2.E11 (VDDCORE), U2.E13 (VDDCORE), U2.E7 (VDDCORE), U2.E9 (VDDCORE), U2.F10 (VDDCORE), U2.F12 (VDDCORE), U2.F4 (VDDCORE), U2.F6 (VDDCORE), U2.F8 (VDDCORE), U2.G11 (VDDCORE), U2.G5 (VDDCORE), U2.G7 (VDDCORE), U2.G9 (VDDCORE), U2.H10 (VDDCORE), U2.H12 (VDDCORE), U2.H4 (VDDCORE), U2.H6 (VDDCORE), U2.H8 (VDDCORE), U2.J11 (VDDCORE), U2.J13 (VDDCORE), U2.J7 (VDDCORE), U2.J9 (VDDCORE), U2.K10 (VDDCORE), U2.K12 (VDDCORE), U2.K8 (VDDCORE), U2.L11 (VDDCORE), U2.L13 (VDDCORE), U2.L9 (VDDCORE), U2.M10 (VDDCORE), U2.M12 (VDDCORE), U2.N11 (VDDCORE), U2.N13 (VDDCORE), U2.P12 (VDDCORE), U2.R13 (VDDCORE)
- new net VDD-PERIPHERALS-EN: U10.3 (EN), U5.9 (PB5), U6.5 (EN)
- new net VDDA-EN: U5.18 (PC3), U8.5 (EN)
- new net VREF-DDR-PGOOD: U7.5 (A)
- no-connect marks 0 -> 3
Other:
- note added: "--"
- note added: "2.8V"
- note added: "3V"
- note added: "5V"
- note added: "COMP NOT CALCULATED YET"
- note added: "SIC451 Supply For General Purpose Use"
- note added: "Supply For the USB PHY"
- note added: "VCC"
- note added: "VDD-USB"
- note removed: "1.2V"
- note removed: "2.5V"
- note removed: "Supply For Ethernet Analog Layer"
- note removed: "Supply For Ethernet Digital Layer"
- note removed: "VDDA-ETH"
- moved on the sheet: C1, C10, C11, C12, C13, C14, C15, C16, C17, C18, C19, C2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

Commit message: (WIP) Start layout
Parts:
- gave numbers to parts that had none: 3
- renumbered C19 to C10, C20 to C11, C5 to C12, C6 to C13, C7 to C14, C8 to C15, C9 to C16, C10 to C17, C11 to C18, C29 to C19, C30 to C20, C31 to C21, C32 to C22, C12 to C23, C13 to C24, C21 to C25, C22 to C26, C23 to C27, C24 to C28, C25 to C29, C26 to C30, C27 to C31, C28 to C32, C48 to C40, C49 to C41, C50 to C42, C51 to C43, C52 to C44, C53 to C45, C54 to C46, C55 to C47, C56 to C48, C57 to C49, C14 to C5, C58 to C50, C40 to C51, C41 to C52, C42 to C53, C43 to C54, C44 to C55, C45 to C56, C46 to C57, C47 to C58, C60 to C59, C15 to C6, C59 to C60, C16 to C7, C74 to C75, C75 to C76, C76 to C77, C77 to C78, C78 to C79, C17 to C8, C79 to C80, C80 to C81, C81 to C82, C82 to C83, C83 to C84, C84 to C85, C85 to C86, C86 to C87, C87 to C88, C88 to C89, C18 to C9, C89 to C90, C90 to C91, C91 to C92, C92 to C93, C93 to C94, C94 to C95, C95 to C96, C96 to C97, C97 to C98, C98 to C99, R33 to R26, R26 to R27, R27 to R28, R28 to R29, R29 to R30, R30 to R31, R31 to R32, R32 to R33, U9 to U10, U10 to U11, U6 to U7, U7 to U8, U8 to U9
Other:
- title: Benchy Version 2 -> Benchy Reloaded
