File: MotherBoard/BenchyMotherBoard-PCB/power.kicad_sch (KiCad schematic)
At the start: 185 parts, among them J1 PWR CONN, J5 USB PWR CONN, U10 USB7206C, U2 TPS65400RGZT, U3 NCP51200, U6 MAX15027, U9 AP2127K-3.3

Commit message: (WIP) Finish more of the PS schematic
Parts:
- removed C185, C186, C187, C188, C189, C190, C191, C192, C193, C195, C40, C41, C42, C43, C44, C49, C50: 100nF, Capacitor_SMD:C_0402_1005Metric, symbol Device:C_Small
- removed C21, C22, C62, C70, C73: 1uF, Capacitor_SMD:C_0603_1608Metric, symbol Device:C_Small
- removed C59, C61, C69: 2.2uF, Capacitor_SMD:C_0603_1608Metric, symbol Device:C_Small
- removed TP10: TP-1V1-REG, TestPoint:TestPoint_Pad_D1.5mm, symbol Connector:TestPoint_Alt
- removed TP11: TP-1V8-REG, TestPoint:TestPoint_Pad_D1.5mm, symbol Connector:TestPoint_Alt
- removed TP12: TP-DSI-REG, TestPoint:TestPoint_Pad_D1.5mm, symbol Connector:TestPoint_Alt
- removed U9: AP2127K-3.3, Package_TO_SOT_SMD:SOT-23-5, symbol Regulator_Linear:AP2127K-3.3
- added L5: L_PWR, symbol Daxxn_Device:L_Power
- added R11: R, symbol Daxxn_Device:R
- added R3, R50, R51, R7: R, Resistor_SMD:R_0402_1005Metric, symbol Daxxn_Device:R
- added U20: TLV759P, Daxxn_Packages:DFN-6-1EP_2x2mm_P0.65mm_EP1x1.6mm, symbol Daxxn_Regulators:TLV75901P
- added U21: TLV7103318, Daxxn_Packages:WSON-6_1.5x1.5mm_P0.5mm, symbol Daxxn_Regulators:TLV7103318
- added U4: AM6254ATCGGAALW, Daxxn_Packages:ALW0425A-BGA-425-13x13mm, symbol Daxxn_TIMicros:AM6254ATCGGAALW
- added U5: SiI9022ACNU, Package_DFN_QFN:QFN-72-1EP_10x10mm_P0.5mm_EP6x6mm, symbol Daxxn_IC:SiI9022ACNU
- added U7: AP3401, Daxxn_Packages:DFN-6-1EP_2x2mm_P0.65mm_EP1x1.6mm, symbol Daxxn_Regulators:AP3401
- added U8: AP2127K-1.2, Package_TO_SOT_SMD:SOT-23-5, symbol Regulator_Linear:AP2127K-1.2
- added U9: MAX16043, Daxxn_Packages:TQFN-24-1EP_4x4mm_P0.5mm_EP2.1x2.1mm, symbol Daxxn_IC:MAX16043
- C10: value 100nF -> 10uF; footprint Capacitor_SMD:C_0402_1005Metric -> Capacitor_SMD:C_0805_2012Metric
- C20: value 1uF -> 100nF; footprint Capacitor_SMD:C_0603_1608Metric -> Capacitor_SMD:C_0402_1005Metric
- C45, C48, C6, C8: value 100nF -> 1uF; footprint Capacitor_SMD:C_0402_1005Metric -> Capacitor_SMD:C_0603_1608Metric
Connections:
- net GND: now also R51.2, R7.2, U20.3 (GND), U20.7 (GND), U21.4 (GND), U7.5 (GND), U7.7 (GND), U8.2 (GND), U9.25 (GND), U9.7 (GND)
- net USB-CORE: now also C8.1, C9.1, U8.5 (VOUT); no longer C200.1, C54.2, C55.1, C56.1, C57.1, L4.2, R14.1
- net VCC: now also C10.1, C11.1, C45.1, C46.1, C5.1, C6.1, C7.1, U20.6 (IN), U21.2 (VIN), U7.3 (VIN), U8.1 (VIN)
- net VDD: now also R11.1; no longer C10.1, C11.1, C19.1, C20.1, C5.1, C6.1, C7.1, C8.1, C9.1
- net VDD-CORE: now also U4.H8 (VDD-CORE), U4.J11 (VDD-CORE), U4.J14 (VDD-CORE), U4.K17 (VDD-CORE), U4.L12 (VDD-CORE), U4.L15 (VDD-CORE), U4.M16 (VDD-CORE), U4.N11 (VDD-CORE), U4.N13 (VDD-CORE), U4.N8 (VDD-CORE), U4.P17 (VDD-CORE), U4.R11 (VDD-CORE), U4.R14 (VDD-CORE), U4.U12 (VDD-CORE), U4.V15 (VDD-CORE), U4.V17 (VDD-CORE), U4.V8 (VDD-CORE); no longer C45.1, C46.1, C47.1, C48.1
- net VDD-DDR: now also C200.1, C54.2, C55.1, C56.1, C57.1, L4.2, R14.1; no longer C35.2, C36.1, C37.1, C38.1, L3.2, R10.1
- net VDD-USB: now also L5.2, R3.1
- net VDD-USB-EN: now also U7.1 (EN), U8.3 (EN)
- net VDDA: now also C47.1, C48.1, R50.1, U20.1 (OUT); no longer C77.1, R34.1, U6.10 (OUT), U6.9 (OUT)
- net VDDA-EN: now also U20.4 (EN)
- new net: R50.2, R51.1, U20.2 (FB)
- new net: C77.1, R34.1, U6.10 (OUT), U6.9 (OUT)
- new net: R3.2, R7.1, U7.6 (FB)
- new net: L5.1, U7.4 (LX)
- new net AVCC: U5.60 (AVCC), U5.66 (AVCC)
- new net DVDD: C35.2, C36.1, C37.1, C38.1, L3.2, R10.1
- new net VCC-CORE: U5.12 (VCC-CORE), U5.26 (VCC-CORE), U5.42 (VCC-CORE), U5.47 (VCC-CORE), U5.5 (VCC-CORE), U5.53 (VCC-CORE)
- new net VCC-IO: U5.21 (VCC-IO), U5.3 (VCC-IO), U5.46 (VCC-IO)
- new net VDD-MMC: C19.1, C20.1, U21.5 (OUT2), U21.6 (OUT1)
- new net VDD-USB-PG: U7.2 (PG)
- new net VDDR-CORE: U4.J12 (VDDR-CORE), U4.K16 (VDDR-CORE), U4.N12 (VDDR-CORE), U4.N14 (VDDR-CORE), U4.P16 (VDDR-CORE), U4.R12 (VDDR-CORE), U4.T10 (VDDR-CORE), U4.U14 (VDDR-CORE)
- new net VDDS-DDR: U4.K9 (VDDS-DDR), U4.L8 (VDDS-DDR), U4.P9 (VDDS-DDR), U4.R8 (VDDS-DDR)
- new net VDDSHV-MCU: U4.F11 (VDDSHV-MCU), U4.G12 (VDDSHV-MCU)
- new net VDDSHV0: U4.F15 (VDDSHV0), U4.G14 (VDDSHV0)
- new net VDDSHV1: U4.L18 (VDDSHV1), U4.M19 (VDDSHV1)
- new net VDDSHV2: U4.W16 (VDDSHV2), U4.W19 (VDDSHV2)
- new net VDDSHV3: U4.N18 (VDDSHV3), U4.P18 (VDDSHV3), U4.T19 (VDDSHV3), U4.U18 (VDDSHV3)
- new net VSEL-SD: R11.2, U21.1 (EN1)
- new net VSS: U4.A1 (VSS), U4.A24 (VSS), U4.A25 (VSS), U4.AA11 (VSS), U4.AB9 (VSS), U4.AD1 (VSS), U4.AD12 (VSS), U4.AD16 (VSS), U4.AD25 (VSS), U4.AD9 (VSS), U4.AE1 (VSS), U4.AE12 (VSS), U4.AE16 (VSS), U4.AE24 (VSS), U4.AE25 (VSS), U4.AE8 (VSS), U4.B25 (VSS), U4.F13 (VSS), U4.G13 (VSS), U4.G19 (VSS), U4.H13 (VSS), U4.H16 (VSS), U4.H18 (VSS), U4.H20 (VSS), U4.J13 (VSS), U4.J7 (VSS), U4.K13 (VSS), U4.K15 (VSS), U4.K19 (VSS), U4.K7 (VSS), U4.L20 (VSS), U4.M10 (VSS), U4.M12 (VSS), U4.M13 (VSS), U4.M17 (VSS), U4.M18 (VSS), U4.M7 (VSS), U4.M8 (VSS), U4.N15 (VSS), U4.P10 (VSS), U4.P13 (VSS), U4.P7 (VSS), U4.R13 (VSS), U4.R15 (VSS), U4.R18 (VSS), U4.R20 (VSS), U4.T13 (VSS), U4.T14 (VSS), U4.T16 (VSS), U4.T17 (VSS), U4.T18 (VSS), U4.T8 (VSS), U4.U19 (VSS), U4.U8 (VSS), U4.V10 (VSS), U4.V11 (VSS), U4.V13 (VSS), U4.V16 (VSS), U4.V18 (VSS), U4.V9 (VSS), U4.W7 (VSS), U4.Y2 (VSS)
- no-connect marks 6 -> 2
Other:
- note added: "0.85V"
- note added: "1.0A"
- note added: "1.2V"
- note added: "1.5A"
- note added: "1.8V"
- note added: "1.8V / 3.3V"
- note added: "100mA"
- note added: "2.7A"
- note added: "200mA"
- note added: "5.0A"
- note added: "50mA"
- note added: "900mA"
- note added: "ANALOG REGULATOR (1V8)"
- note added: "DDR4 Memory Digital Supply"
- note added: "DVDD"
- note added: "HDMI TRANSEIVER POWER"
- note added: "MPU Digital Supply"
- note added: "MPU POWER"
- note added: "MPU POWER MON"
- note added: "SDCard Supply"
- note added: "Supply For DDR4 Pullup Resistors"
- note added: "USB HUB CORE REGULATOR (1V2)"
- note added: "USB HUB VDD REGULATOR (3V3)"
- note added: "VDD-MMC"
- note added: "eMMC SELECTABLE REGULATOR (3V3/1V8)"
- note removed: "1.1V"
- note removed: "1.3V"
- note removed: "3V"
- note removed: "DDR3 Memory Digital Supply"
- note removed: "STM32 MPU POWER"
- note removed: "Supply For DDR3 Pullup Resistors"
- note removed: "USB VDD REGULATOR"
- moved on the sheet: C13, C25, C34, C53, C67, C68, C75, C76, C77, C78, C79, C80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

Commit message: (WIP) More work on power supply sequencing
Parts:
- added C100, C71, C72, C73, C74: C, Capacitor_SMD:C_0402_1005Metric, symbol Daxxn_Device:C
- added C49, C59: 1uF, Capacitor_SMD:C_0603_1608Metric, symbol Device:C_Small
- added C50, C61: 100nF, Capacitor_SMD:C_0402_1005Metric, symbol Device:C_Small
- added R15, R52: R, Resistor_SMD:R_0402_1005Metric, symbol Daxxn_Device:R
- added R55: 10K, Resistor_SMD:R_0402_1005Metric, symbol Daxxn_Device:R
- added TP10: TP-USB-CORE, TestPoint:TestPoint_Pad_D1.5mm, symbol Connector:TestPoint_Alt
- added TP11: TP-DVDD, TestPoint:TestPoint_Pad_D1.5mm, symbol Connector:TestPoint_Alt
- added TP12: TP-VPP-DDR, TestPoint:TestPoint_Pad_D1.5mm, symbol Connector:TestPoint_Alt
- added U22: AP2127K-1.2, Package_TO_SOT_SMD:SOT-23-5, symbol Regulator_Linear:AP2127K-1.2
Connections:
- net VCC-CORE is gone; now on net AVCC: U5.12 (VCC-CORE), U5.26 (VCC-CORE), U5.42 (VCC-CORE), U5.47 (VCC-CORE), U5.5 (VCC-CORE), U5.53 (VCC-CORE)
- net VCC-IO is gone; now on net DVDD: U5.21 (VCC-IO), U5.3 (VCC-IO), U5.46 (VCC-IO)
- net AVCC: now also C59.1, C61.1, TP10.1, U22.5 (VOUT)
- net DVDD: now also U9.3 (IN2), TP11.1
- net GND: now also U5.43 (GND-CORE), U5.57 (GND-IO), U5.63 (AGND), U5.73 (GND-PAD), C100.2, C49.2, C50.2, C59.2, C61.2, C71.2, C72.2, C73.2, C74.2, R52.1, U22.2 (GND)
- net VCC: now also C49.1, C50.1, U22.1 (VIN)
- net VDD: now also U9.5 (IN4)
- net VDD-CORE: now also U9.4 (IN3)
- net VDD-DDR: now also U9.2 (IN1)
- net VDD-DDR-EN: now also U9.11 (EN4), U9.15 (OUT3)
- net VDD-PWR: now also U9.1 (VCC)
- net VDD-USB-EN: now also U22.3 (EN)
- net VPP-DDR: now reaches C77.1, R34.1, U6.10 (OUT), U6.9 (OUT)
- net VPP-DDR: now also TP12.1
- net DVDD-EN: now reaches U9.10 (EN3)
- net DVDD-EN: now also U9.16 (OUT2)
- net VDD-CORE-EN: now reaches U9.14 (OUT4)
- net VDD-EN: now reaches U9.17 (OUT1)
- net VDD-EN: now also U9.9 (EN2)
- net MPU-POR: now reaches U9.18 (~{RESET})
- net MPU-POR: now also R55.2
- net at U9.20 (CRESET): now also C100.1
- net at U9.21 (CDLY4): now also C71.1
- net at U9.22 (CDLY3): now also C72.1
- net at U9.23 (CDLY2): now also C73.1
- net at U9.24 (CDLY1): now also C74.1
- net at U4.H10 (VMON-VSYS): now also R15.2, R52.2
- net SD-CARD-PWR-SEL: now reaches U21.3 (EN2)
Other:
- note added: "10mS"
- note added: "2.5V"
- note added: "2.5V SUPPLY FOR DDR4 MEMORY. REASON UNKNOWN ATM."
- note added: "2000mA"
- note added: "2700mA"
- note added: "400mA"
- note added: "5000mA"
- note added: "5mS"
- note added: "DDR VPP REGULATOR (2V5)"
- note added: "DELAY1"
- note added: "DELAY2"
- note added: "DELAY3"
- note added: "DELAY4"
- note added: "DELAYS"
- note added: "DESCRIPTION"
- note added: "EFuse Programming Supply"
- note added: "HDMI TRANSEIVER CORE REGULATOR (1V2)"
- note added: "MAIN POWER RAILS"
- note added: "MD1"
- note added: "MD2"
- note added: "MD3"
- note added: "MD4"
- note added: "MPU POWER RAILS"
- note added: "Main System Level Digital Supply"
- note added: "PIN NAMES"
- note added: "POWER UP SEQUENCE"
- note added: "RAIL"
- note added: "VDDA_1P8_CSIRX0"
- note added: "VDDA_1P8_OLDI0"
- note added: "VDDA_1P8_USB"
- note added: "VDDA_3P3_USB"
- note added: "VDDA_CORE_CSIRX0"
- note added: "VDDA_CORE_USB"
- note added: "VDDA_DDR_PLL0"
- note added: "VDDA_MCU"
- note added: "VDDA_PLL0"
- note added: "VDDA_PLL1"
- note added: "VDDA_PLL2"
- note added: "VDDA_TEMP0"
- note added: "VDDA_TEMP1"
- note added: "VDDR_CORE"
- note added: "VDDSHV0"
- note added: "VDDSHV1"
- note added: "VDDSHV2"
- note added: "VDDSHV3"
- note added: "VDDSHV4"
- note added: "VDDSHV5"
- note added: "VDDSHV6"
- note added: "VDDSHV_CANUART"
- note added: "VDDSHV_MCU"
- note added: "VDDS_DDR"
- note added: "VDDS_DDR_C"
- note added: "VDD_CANUART"
- note added: "VDD_CORE"
- note added: "VMON_1P8_SOC"
- note added: "VMON_3P3_SOC"
- note added: "VOLTAGE LOAD"
- note added: "VPP"
- note added: "VPP-DDR"
- note removed: "1.0A"
- note removed: "1.5A"
- note removed: "1.5V"
- note removed: "100mA"
- note removed: "2.7A"
- note removed: "5.0A"
- note removed: "ALWAYS ON"
- note removed: "ANALOG REGULATOR"
- note removed: "Main Digital Supply"
- note removed: "POWER RAILS"
- note removed: "POWER SEQUENCE"
- note removed: "RUN"
- note removed: "START"
- moved on the sheet: C10, C11, C67, C68, C82, C83, C84, C85, C86, C87, C88, C89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

Commit message: (WIP) Complete most of the PS and boot schematics
Parts:
- removed C63: 4.7uF, Capacitor_SMD:C_0603_1608Metric, symbol Device:C_Small
- removed C64, C65, C66, C96, C97: 10uF, Capacitor_SMD:C_0805_2012Metric, symbol Device:C_Small
- removed C98: 1nF, Capacitor_SMD:C_0402_1005Metric, symbol Device:C_Small
- removed C99: 100nF, Capacitor_SMD:C_0402_1005Metric, symbol Device:C_Small
- removed R23, R24, R25: 10K, Resistor_SMD:R_0402_1005Metric, symbol Device:R_Small_US
- removed R55: 10K, Resistor_SMD:R_0402_1005Metric, symbol Daxxn_Device:R
- removed TP5: TP-VTT, TestPoint:TestPoint_Pad_D1.5mm, symbol Connector:TestPoint_Alt
- removed TP6: TP-VREF-DDR, TestPoint:TestPoint_Pad_D1.5mm, symbol Connector:TestPoint_Alt
- removed U3: NCP51200, Daxxn_Packages:DFN-10-1EP_3x3mm_P0.5mm_EP1.65x2.38mm, symbol Daxxn_IC:NCP51200
- added C101, C222, C223, C224, C225, C226, C227, C228, C229: 100nF, Capacitor_SMD:C_0402_1005Metric, symbol Daxxn_Device:C
- added C102, C220, C221: 1uF, Capacitor_SMD:C_0402_1005Metric, symbol Daxxn_Device:C
- added C103, C104, C105, C106, C107, C108, C109, C110, C111, C112, C113, C114, C115, C116, C117, C118, C119, C120, C121, C122, C123, C124, C125, C126, C127, C128, C129, C130, C131, C132, C133, C134, C135, C136, C137, C142, C185, C186, C187, C188, C189, C190, C191, C192, C193, C194, C195, C198, C202, C203, C204, C205, C206, C207, C208, C209, C219, C233, C234, C235, C236, C237, C238, C239, C240, C241, C242, C243: 100nF, Capacitor_SMD:C_0201_0603Metric, symbol Daxxn_Device:C
- added C210, C211, C212, C213, C214, C215, C216, C217, C218: 1uF, Capacitor_SMD:C_0201_0603Metric, symbol Daxxn_Device:C
- added C264: 1uF, Capacitor_SMD:C_0603_1608Metric, symbol Daxxn_Device:C
- added D21, D22, D23, D24, D9: ORANGE, LED_SMD:LED_0805_2012Metric, symbol Daxxn_Device:LED
- added H11: M2, MountingHole:MountingHole_2.2mm_M2_ISO7380_Pad, symbol Mechanical:MountingHole_Pad
- added Q4, Q5, Q6, Q7: MMBT2222A, Package_TO_SOT_SMD:SOT-23, symbol Daxxn_Transistors:MMBT2222A
- added R136, R61, R62, R63, R64, R65: 10K, Resistor_SMD:R_0402_1005Metric, symbol Daxxn_Device:R
- added R137: 1.5K, Resistor_SMD:R_0402_1005Metric, symbol Daxxn_Device:R
- added R67: 6.8K, Resistor_SMD:R_0402_1005Metric, symbol Daxxn_Device:R
- added R68: 12K, Resistor_SMD:R_0402_1005Metric, symbol Daxxn_Device:R
- added R69: 4.7K, Resistor_SMD:R_0402_1005Metric, symbol Daxxn_Device:R
- added R70: 3.9K, Resistor_SMD:R_0402_1005Metric, symbol Daxxn_Device:R
- added R71, R73, R75, R76, R78: 500, Resistor_SMD:R_0603_1608Metric, symbol Daxxn_Device:R
- added R72, R74, R77, R82: 1K, Resistor_SMD:R_0603_1608Metric, symbol Daxxn_Device:R
- C1, C10, C11, C12, C13, C14, C15, C16, C17, C18, C182, C183, C184, C19, C196, C197, C199, C2, C20, C200, C201, C23, C24, C25, C26, C27, C28, C29, C30, C31, C32, C33, C34, C35, C36, C37, C38, C39, C4, C45, C46, C47, C48, C49, C5, C50, C51, C52, C53, C54, C55, C56, C57, C58, C59, C6, C60, C61, C67, C68, C7, C75, C76, C77, C78, C79, C8, C80, C81, C82, C83, C84, C85, C86, C87, C88, C89, C9, C90, C91, C92, C93, C94, C95: symbol Device:C_Small -> Daxxn_Device:C
- C100: value C -> 100nF
- C3: symbol Device:C_Polarized_Small -> Daxxn_Device:C_Pol
- C71, C72, C73: value C -> 2nF
- C74: value C -> 1nF
- D10, D11, D12, D13, D14, D15, D16: symbol Device:LED_Small -> Daxxn_Device:LED
- L1, L2, L3, L4: symbol Device:L_Small -> Daxxn_Device:L
- R1, R10, R12, R120, R13, R14, R16, R17, R18, R19, R2, R20, R21, R22, R26, R31, R33, R34, R35, R37, R38, R39, R4, R40, R5, R6, R8, R9: symbol Device:R_Small_US -> Daxxn_Device:R
- R11: value R -> 10K
- R15: value R -> 47K
- R52: value R -> 2.2K
Connections:
- net DVDD-EN is gone; now on net MD2: U9.10 (EN3), U9.16 (OUT2)
- net PWR-ERROR is gone; now on net VDD-USB-PG: D16.2 (A)
- net PWR-ON-RST is gone; now on net SMPS-PGOOD: D10.2 (A)
- net VDD-CORE-EN is gone; now on net MD4: U9.14 (OUT4)
- net VDD-DDR-EN is gone; now on net MD3: U9.11 (EN4), U9.15 (OUT3)
- net VDD-EN is gone; now on net MD1: U9.17 (OUT1), U9.9 (EN2)
- net VDDR-CORE is gone; now on net VDD-CORE: U4.J12 (VDDR-CORE), U4.K16 (VDDR-CORE), U4.N12 (VDDR-CORE), U4.N14 (VDDR-CORE), U4.P16 (VDDR-CORE), U4.R12 (VDDR-CORE), U4.T10 (VDDR-CORE), U4.U14 (VDDR-CORE)
- net VDDS-DDR is gone; now on net VDD-DDR: U4.K9 (VDDS-DDR), U4.L8 (VDDS-DDR), U4.P9 (VDDS-DDR), U4.R8 (VDDS-DDR)
- net VDDSHV-MCU is gone; now on net VDD: U4.F11 (VDDSHV-MCU), U4.G12 (VDDSHV-MCU)
- net VDDSHV0 is gone; now on net VDD: U4.F15 (VDDSHV0), U4.G14 (VDDSHV0)
- net VDDSHV1 is gone; now on net DVDD: U4.L18 (VDDSHV1), U4.M19 (VDDSHV1)
- net VDDSHV2 is gone; now on net VDD: U4.W16 (VDDSHV2), U4.W19 (VDDSHV2)
- net VDDSHV3 is gone; now on net VDD: U4.N18 (VDDSHV3), U4.P18 (VDDSHV3), U4.T19 (VDDSHV3), U4.U18 (VDDSHV3)
- net VSS is gone; now on net GND: U4.A1 (VSS), U4.A24 (VSS), U4.A25 (VSS), U4.AA11 (VSS), U4.AB9 (VSS), U4.AD1 (VSS), U4.AD12 (VSS), U4.AD16 (VSS), U4.AD25 (VSS), U4.AD9 (VSS), U4.AE1 (VSS), U4.AE12 (VSS), U4.AE16 (VSS), U4.AE24 (VSS), U4.AE25 (VSS), U4.AE8 (VSS), U4.B25 (VSS), U4.F13 (VSS), U4.G13 (VSS), U4.G19 (VSS), U4.H13 (VSS), U4.H16 (VSS), U4.H18 (VSS), U4.H20 (VSS), U4.J13 (VSS), U4.J7 (VSS), U4.K13 (VSS), U4.K15 (VSS), U4.K19 (VSS), U4.K7 (VSS), U4.L20 (VSS), U4.M10 (VSS), U4.M12 (VSS), U4.M13 (VSS), U4.M17 (VSS), U4.M18 (VSS), U4.M7 (VSS), U4.M8 (VSS), U4.N15 (VSS), U4.P10 (VSS), U4.P13 (VSS), U4.P7 (VSS), U4.R13 (VSS), U4.R15 (VSS), U4.R18 (VSS), U4.R20 (VSS), U4.T13 (VSS), U4.T14 (VSS), U4.T16 (VSS), U4.T17 (VSS), U4.T18 (VSS), U4.T8 (VSS), U4.U19 (VSS), U4.U8 (VSS), U4.V10 (VSS), U4.V11 (VSS), U4.V13 (VSS), U4.V16 (VSS), U4.V18 (VSS), U4.V9 (VSS), U4.W7 (VSS), U4.Y2 (VSS)
- net AVCC: now also C221.1, C222.1, C223.1, C224.1, C225.1
- net DVDD: now also U4.G10 (VMON-1P8-SOC), U4.J18 (VDDSHV6), U4.T7 (VDDSHV4), C115.1, C116.1, C117.1, C118.1, C226.1, C227.1, C228.1, C229.1, R74.2
- net GND: now also U9.12 (TH1), C101.2, C102.2, C103.2, C104.2, C105.2, C106.2, C107.2, C108.2, C109.2, C110.2, C111.2, C112.2, C113.2, C114.2, C115.2, C116.2, C117.2, C118.2, C119.2, C120.2, C121.2, C122.2, C123.2, C124.2, C125.2, C126.2, C127.2, C128.2, C129.2, C130.2, C131.2, C132.2, C133.2, C134.2, C135.2, C136.2, C137.2, C142.2, C185.2, C186.2, C187.2, C188.2, C189.2, C190.2, C191.2, C192.2, C193.2, C194.2, C195.2, C198.2, C202.2, C203.2, C204.2, C205.2, C206.2, C207.2, C208.2, C209.2, C210.2, C211.2, C212.2, C213.2, C214.2, C215.2, C216.2, C217.2, C218.2, C219.2, C220.2, C221.2, C222.2, C223.2, C224.2, C225.2, C226.2, C227.2, C228.2, C229.2, C233.2, C234.2, C235.2, C236.2, C237.2, C238.2, C239.2, C240.2, C241.2, C242.2, C243.2, C264.2, H11.1, Q4.1 (E), Q5.1 (E), Q6.1 (E), Q7.1 (E), R137.2, R68.2, R70.2, R71.2
- net SMPS-PGOOD: no longer D15.2 (A), U2.17 (PGOOD)
- net USB-CORE: now also R77.2
- net VCC: now also D11.2 (A), D21.2 (A), D22.2 (A), D23.2 (A), D24.2 (A); no longer D12.2 (A)
- net VDD: now also D12.2 (A), U4.H9 (VDDSHV-CANUART), U4.K10 (VMON-3P3-SOC), U4.Y13 (VDDA-3P3-USB), U9.2 (IN1), C103.1, C104.1, C105.1, C106.1, C107.1, C108.1, C109.1, C110.1, C111.1, C112.1, C113.1, C114.1, R61.1, R62.1, R63.1, R64.1, R65.1; no longer D11.2 (A), U9.5 (IN4)
- net VDD-CORE: now also U4.F8 (VDD-CANUART), U4.W12 (VDDA-CORE-USB), U4.W13 (VDDA-CORE-CSIRX0), C119.1, C120.1, C121.1, C122.1, C123.1, C124.1, C125.1, C126.1, C127.1, C128.1, C129.1, C130.1, C189.1, C190.1, C191.1, C192.1, C193.1, C194.1, C234.1, C235.1, C236.1, C237.1, C238.1, C239.1, C240.1, C241.1, C242.1, C243.1, R67.1, R72.2; no longer U9.4 (IN3)
- net VDD-DDR: now also U4.M9 (VDDS-DDR-C), C204.1, C205.1, C206.1, C207.1, C208.1, C209.1, R69.1; no longer U9.2 (IN1)
- net VDD-MMC: now also U4.G17 (VDDSHV5), C195.1, C198.1, C202.1, C203.1
- net VDD-PWR: now also U9.13 (TH0), U9.6 (TOL), U9.8 (EN1), C101.1, C102.1
- net VDDA: now also U4.G16 (VDDA-TEMP1), U4.G7 (VDDS-OSC0), U4.L11 (VDDA-MCU), U4.L14 (VDDA-PLL2), U4.T9 (VDDA-TEMP0), U4.U11 (VDDA-PLL0), U4.U15 (VDDA-PLL1), U4.W10 (VDDA-1P8-OLDI0), U4.W14 (VDDA-1P8-CSIRX0), U4.W9 (VDDA-1P8-OLDI0), U4.Y11 (VDDA-1P8-USB), C131.1, C132.1, C133.1, C134.1, C135.1, C136.1, C137.1, C142.1, C185.1, C186.1, C187.1, C188.1
- net VPP-DDR: now also R82.2
- net VPWR: now also R15.1, R136.1
- net VTT-DDR-PG: now also D15.2 (A)
- net PWR-SWITCH: now reaches U9.19 (MR)
- net VMON-SYS: now reaches R15.2, R52.2, U4.H10 (VMON-VSYS)
- net VMON-SYS: now also C233.1
- net at U4.G9 (CAP-VDDS-CANUART): now also C218.1
- net at U4.H11 (CAP-VDDS-MCU): now also C210.1
- net at U4.H15 (CAP-VDDS0): now also C217.1
- net at U4.H17 (CAP-VDDS5): now also C212.1
- net at U4.J19 (CAP-VDDS6): now also C211.1
- net VPP: now reaches U4.J8 (VPP)
- net VPP: now also C219.1, C220.1
- net at U4.K18 (CAP-VDDS1): now also C216.1
- net at U4.P19 (CAP-VDDS3): now also C214.1
- net at U4.U7 (CAP-VDDS4): now also C213.1
- net at U4.W17 (CAP-VDDS2): now also C215.1
- net MD4: now reaches U2.13 (ENSW2)
- net MD4: now also R62.2
- net MD2: now reaches U2.27 (ENSW3)
- net MD2: now also U20.4 (EN), U22.3 (EN), R64.2
- net MD3: now reaches U2.34 (ENSW4)
- net MD3: now also R20.2, U6.5 (EN), R63.2
- net MD1: now reaches U2.48 (ENSW1/ENSEQ)
- net MD1: now also U7.1 (EN), U8.3 (EN), R65.2
- net MPU-POR renamed ~{MCU-POR}
- net ~{MCU-POR}: now also R61.2
- net POWER-RESET renamed PWR-RESET
- net PWR-RESET: now also C264.1, R136.2, R137.1
- removed net VDD-USB-EN: U22.3 (EN), U7.1 (EN), U8.3 (EN)
- removed net VDDA-EN: R20.2, U20.4 (EN), U6.5 (EN)
- net VDDA-FB renamed VPP-FB
- net VDDA-SS renamed VPP-SS
- new net: Q7.2 (B), R82.1
- new net: Q7.3 (C), R78.2
- new net: D22.1 (K), R75.1
- new net: D24.1 (K), R76.1
- new net: D9.1 (K), R71.1
- new net: Q6.3 (C), R76.2
- new net: D23.1 (K), R78.1
- new net: Q4.2 (B), R72.1
- new net: Q4.3 (C), R75.2
- new net: D21.1 (K), R73.1
- new net: Q5.3 (C), R73.2
- new net: Q5.2 (B), R74.1
- new net: Q6.2 (B), R77.1
- new net POWER-PGOOD: U2.17 (PGOOD)
- new net VDD-CORE-SUP: R67.2, R68.1, U9.5 (IN4)
- new net VDD-DDR-SUP: R69.2, R70.1, U9.4 (IN3)
Other:
- note added: "POWER SWITCH"
- note added: "VDDS-OSC0"
- note removed: "DDR MEMORY REGULATOR"
- note removed: "VDDA_DDR_PLL0"
- moved on the sheet: C10, C100, C11, C19, C20, C45, C46, C47, C48, C49, C5, C50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

Commit message: Add new ethernet chip - KSZ9031
Parts:
- removed L1: 22uH, Daxxn_Passives:PA4341, symbol Daxxn_Device:L
- removed L2, L3, L4: 10uH, Daxxn_Passives:PA4341, symbol Daxxn_Device:L
- added C267, C269, C322, C324: 1uF, Capacitor_SMD:C_0603_1608Metric, symbol Daxxn_Device:C
- added C268, C270, C277, C308, C310, C311, C312, C313, C314, C315, C316, C317, C319, C323, C325, C326, C327, C329, C331, C334, C336, C337, C338, C339, C341, C343, C344, C345, C346, C348, C350, C351, C352, C353, C354, C355, C356, C357, C358, C359, C361, C363, C364, C365, C366, C368, C370, C373, C375, C377, C378: 100nF, Capacitor_SMD:C_0402_1005Metric, symbol Daxxn_Device:C
- added C271, C272, C273, C274, C275: 10uF, Capacitor_SMD:C_1210_3225Metric, symbol Daxxn_Device:C
- added C276, C321: 22pF, Capacitor_SMD:C_0402_1005Metric, symbol Daxxn_Device:C
- added C307, C309, C318, C320, C328, C330, C333, C335, C340, C342, C347, C349, C360, C362, C367, C369, C376, C379: 10uF, Daxxn_Passives:C_TANT_1206_3216Metric, symbol Daxxn_Device:C_Pol
- added C332, C371: 10nF, Capacitor_SMD:C_0402_1005Metric, symbol Daxxn_Device:C
- added C372, C374: 1uF, Capacitor_SMD:C_0402_1005Metric, symbol Daxxn_Device:C
- added FB1, FB10, FB11, FB12, FB2, FB3, FB4, FB5, FB6, FB7, FB8, FB9: 100 @ 100MHz, Inductor_SMD:L_0603_1608Metric, symbol Daxxn_Device:FerriteBead
- added JP1: Jumper, symbol Daxxn_Other:Jumper
- added L1: 4.7uH, Daxxn_Passives:Wuerth_MAPI-4030, symbol Daxxn_Device:L_Power
- added L2: 3.3uH, Daxxn_Passives:Wuerth_MAPI-4030, symbol Daxxn_Device:L_Power
- added L3: 5.6uH, Daxxn_Passives:Wuerth_MAPI-4030, symbol Daxxn_Device:L_Power
- added L4: 8.2uH, Daxxn_Passives:Wuerth_MAPI-4030, symbol Daxxn_Device:L_Power
- added L6: 2.2uH, Inductor_SMD:L_0805_2012Metric, symbol Daxxn_Device:L_Power
- added R147: 10K, Resistor_SMD:R_0402_1005Metric, symbol Daxxn_Device:R
- added R208, R209: 100K, Resistor_SMD:R_0402_1005Metric, symbol Daxxn_Device:R
- added TP15: TP-VDD-USB, TestPoint:TestPoint_Pad_D1.5mm, symbol Connector:TestPoint_Alt
- added TP6: TP-VPP, TestPoint:TestPoint_Pad_D1.5mm, symbol Connector:TestPoint_Alt
- added U23, U24: KSZ9031MNX, Daxxn_Packages:QFN-64-1EP_8x8mm_P0.4mm_EP6.5x6.5mm, symbol Daxxn_IC:KSZ9031MNX
- added U30: AP3401, Daxxn_Packages:DFN-6-1EP_2x2mm_P0.65mm_EP1x1.6mm, symbol Daxxn_Regulators:AP3401
- added U32: TLV75518PDRV, Package_SON:WSON-6-1EP_2x2mm_P0.65mm_EP1x1.6mm, symbol Regulator_Linear:TLV75518PDRV
- C14, C26, C35, C54: value 100nF -> 100pF
- C30: value 117pF -> 4.62pF
- C31: value 1nF -> 4.37n
- L5: value L_PWR -> 2.2uH; footprint (none) -> Inductor_SMD:L_0805_2012Metric
- R1: value 24K -> 10K
- R10: value 13K -> 10K
- R12: value 15K -> 8K
- R14: value 4.3K -> 10K
- R16: value 11K -> 20K
- R3: value R -> 430K
- R34: value 10K -> 40K
- R35: value 6.8K -> 10K
- R4: value 7.5K -> 3.2K
- R5: value 10K -> 4.32K
- R6: value 6.2K -> 16K
- R7: value R -> 100K
- R8: value 10K -> 1K
Connections:
- net AVCC: now also FB9.2; no longer C59.1, C61.1, TP10.1, U22.5 (VOUT)
- net COMP1: now also C30.2, R5.1; no longer C18.2, R2.1
- net COMP2: now also C18.2, R2.1; no longer C30.2, R5.1
- net DVDD: now also C273.1, C374.1, C375.1, FB10.1, L3.2; no longer C226.1, C227.1, C228.1, C229.1, U5.21 (VCC-IO), U5.3 (VCC-IO), U5.46 (VCC-IO)
- net MD1: now also U30.1 (EN)
- net PWR-SW1: now also L1.1
- net PWR-SW2: now also L2.1
- net PWR-SW3: now also L3.1
- net PWR-SW4: now also L4.1
- net USB-CORE: now also C378.1, C379.1, FB12.1; no longer C82.1, C83.1, C84.1, C85.1, C86.1, C87.1, C88.1, U10.18 (VCORE), U10.25 (VCORE), U10.31 (VCORE), U10.38 (VCORE), U10.55 (VCORE), U10.78 (VCORE), U10.85 (VCORE), U10.9 (VCORE), U10.93 (VCORE)
- net VCC: now also C267.1, C268.1, C322.1, C323.1, JP1.2 (B), U30.3 (VIN), U32.6 (IN)
- net VDD: now also C271.1, C275.1, C307.1, C308.1, C347.1, C348.1, C376.1, C377.1, FB1.1, FB11.1, FB6.1, L1.2; no longer C67.1, C68.1, C89.1, C90.1, C91.1, C92.1, C93.1, C94.1, C95.1, U10.26 (VDD33), U10.43 (VDD33), U10.53 (VDD33), U10.62 (VDD33), U10.67 (VDD33), U10.79 (VDD33), U10.88 (VDD33), U10.99 (VDD33)
- net VDD-CORE: now also R8.1, C272.1, L2.2; no longer R6.1
- net VDD-DDR: now also C274.1, L4.2
- net VDD-USB: now also C276.1
- net VDD-USB-PG: now also U30.2 (PG)
- net VPP: now also C269.1, C270.1, TP6.1, U32.1 (OUT)
- net VPP-DDR: now also C277.1
- net at R3.2, R7.1, U7.6 (FB): now also C276.2
- net GND renamed AGNDH
- net AGNDH: now also R6.1, C267.2, C268.2, C269.2, C270.2, C271.2, C272.2, C273.2, C274.2, C275.2, C277.2, C307.2, C308.2, C309.2, C310.2, C311.2, C312.2, C313.2, C314.2, C315.2, C316.2, C317.2, C318.2, C319.2, C320.2, C322.2, C323.2, C324.2, C325.2, C326.2, C327.2, C328.2, C329.2, C330.2, C331.2, C332.2, C333.2, C334.2, C335.2, C336.2, C337.2, C338.2, C339.2, C340.2, C341.2, C342.2, C343.2, C344.2, C345.2, C346.2, C347.2, C348.2, C349.2, C350.2, C351.2, C352.2, C353.2, C354.2, C355.2, C356.2, C357.2, C358.2, C359.2, C360.2, C361.2, C362.2, C363.2, C364.2, C365.2, C366.2, C367.2, C368.2, C369.2, C370.2, C371.2, C372.2, C373.2, C374.2, C375.2, C376.2, C377.2, C378.2, C379.2, R147.2, R209.2, U23.64 (AGNDH), U23.65 (GND), U23.9 (AGNDH), U24.64 (AGNDH), U24.65 (GND), U24.9 (AGNDH), U30.5 (GND), U30.7 (GND), U32.3 (GND), U32.7 (GND); no longer R8.1
- net ~{MCU-POR} renamed ~{MAIN-RESET}
- new net: JP1.1 (A), R147.1, U32.4 (EN)
- new net: C321.2, R208.2, R209.1, U30.6 (FB)
- new net: L6.1, U30.4 (LX)
- new net AVDDH: C309.1, C310.1, C311.1, C312.1, C313.1, C314.1, C315.1, C316.1, C317.1, C349.1, C350.1, C351.1, C352.1, C353.1, C354.1, C355.1, C356.1, C357.1, FB1.2, FB6.2, U23.1 (AVDDH), U23.16 (AVDDH), U23.18 (DVDDH), U23.30 (DVDDH), U23.40 (DVDDH), U23.46 (DVDDH), U24.1 (AVDDH), U24.16 (AVDDH), U24.18 (DVDDH), U24.30 (DVDDH), U24.40 (DVDDH), U24.46 (DVDDH)
- new net AVDDL: C320.1, C326.1, C327.1, C342.1, C343.1, C344.1, C345.1, C346.1, C358.1, C359.1, FB2.2, FB5.2, U23.12 (AVDDL), U23.13 (AVDDL), U23.4 (AVDDL), U23.5 (AVDDL), U24.12 (AVDDL), U24.13 (AVDDL), U24.4 (AVDDL), U24.5 (AVDDL)
- new net DVDDL: C335.1, C336.1, C337.1, C338.1, C339.1, C362.1, C363.1, C364.1, C365.1, C366.1, FB4.2, FB7.2, U23.20 (DVDDL), U23.25 (DVDDL), U23.36 (DVDDL), U23.42 (DVDDL), U23.54 (DVDDL), U24.20 (DVDDL), U24.25 (DVDDL), U24.36 (DVDDL), U24.42 (DVDDL), U24.54 (DVDDL)
- new net ETH-AVDDL-PLL: C330.1, C331.1, C332.1, C369.1, C370.1, C371.1, FB3.2, FB8.2, U23.59 (AVDDL-PLL), U24.59 (AVDDL-PLL)
- new net HDMI-CORE: C372.1, C373.1, C59.1, C61.1, FB9.1, TP10.1, U22.5 (VOUT)
- new net VCC-IO: C226.1, C227.1, C228.1, C229.1, FB10.2, U5.21 (VCC-IO), U5.3 (VCC-IO), U5.46 (VCC-IO)
- new net VCORE: C82.1, C83.1, C84.1, C85.1, C86.1, C87.1, C88.1, FB12.2, U10.18 (VCORE), U10.25 (VCORE), U10.31 (VCORE), U10.38 (VCORE), U10.55 (VCORE), U10.78 (VCORE), U10.85 (VCORE), U10.9 (VCORE), U10.93 (VCORE)
- new net VDD-ETH: C318.1, C319.1, C321.1, C324.1, C325.1, C328.1, C329.1, C333.1, C334.1, C340.1, C341.1, C360.1, C361.1, C367.1, C368.1, FB2.1, FB3.1, FB4.1, FB5.1, FB7.1, FB8.1, L6.2, R208.1, TP15.1
- new net VDD33: C67.1, C68.1, C89.1, C90.1, C91.1, C92.1, C93.1, C94.1, C95.1, FB11.2, U10.26 (VDD33), U10.43 (VDD33), U10.53 (VDD33), U10.62 (VDD33), U10.67 (VDD33), U10.79 (VDD33), U10.88 (VDD33), U10.99 (VDD33)
- no-connect marks 2 -> 4
Other:
- note added: "1.4uH - 3.9uH"
- note added: "120mA"
- note added: "150mA"
- note added: "2.6uH - 7.6uH"
- note added: "221mA"
- note added: "2uH - 5.9uH"
- note added: "4uH - 10uH"
- note added: "500mA"
- note added: "53.8mA"
- note added: "66.6mA"
- note added: "AVDDH"
- note added: "AVDDL"
- note added: "AVDDL-PLL"
- note added: "Analog IO (Transeiver) Supply"
- note added: "CHECK VALUES"
- note added: "Core Supply"
- note added: "DDR VPP REGULATOR - VPP-DDR (2V5)"
- note added: "DVDDH"
- note added: "DVDDL"
- note added: "Description"
- note added: "Digital IO Supply"
- note added: "EACH"
- note added: "ETHERNET CORE REGULATOR - VDD-ETH (1V2)"
- note added: "ETHERNET TRANSEIVER"
- note added: "HDMI TRANSEIVER CORE REGULATOR - HDMI-CORE (1V2)"
- note added: "IND RANGE"
- note added: "Internal LDO for Core Supply. (Optional)"
- note added: "LDO-OUT"
- note added: "NOT USED"
- note added: "PIN"
- note added: "PROGRAMMING REGULATOR - VPP (1V8)"
- note added: "TOTAL"
- note added: "USB HUB CORE REGULATOR - USB-CORE (1V2)"
- note added: "VDD-ETH"
- note added: "VOLT"
- note added: "X"
- note added: "eMMC SELECTABLE REGULATOR - VDD-MMC (3V3/1V8)"
- note removed: "DDR VPP REGULATOR (2V5)"
- note removed: "HDMI TRANSEIVER CORE REGULATOR (1V2)"
- note removed: "POWER SWITCH"
- note removed: "USB HUB CORE REGULATOR (1V2)"
- note removed: "eMMC SELECTABLE REGULATOR (3V3/1V8)"
- moved on the sheet: C18, C200, C221, C222, C223, C224, C225, C226, C227, C228, C229, C23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
