File: MotherBoard/BenchyMotherBoard-PCB/power.kicad_sch (KiCad schematic)
At the start: 397 parts, among them J1 PWR CONN, J5 USB PWR CONN, Q4 MMBT2222A, Q5 MMBT2222A, Q6 MMBT2222A, Q7 MMBT2222A, U10 USB7206C, U2 TPS65400RGZT, U20 TLV759P, U21 TLV7103318, U22 AP2127K-1.2, U23 KSZ9031MNX, U24 KSZ9031MNX, U30 AP3401, U32 TLV75518PDRV, U4 AM6254ATCGGAALW, U5 SiI9022ACNU, U6 MAX15027, U7 AP3401, U8 AP2127K-1.2, U9 MAX16043

Commit message: (WIP) Almost done with schematic
Parts:
- removed U23, U24: KSZ9031MNX, Daxxn_Packages:QFN-64-1EP_8x8mm_P0.4mm_EP6.5x6.5mm, symbol Daxxn_IC:KSZ9031MNX
- removed U30: AP3401, Daxxn_Packages:DFN-6-1EP_2x2mm_P0.65mm_EP1x1.6mm, symbol Daxxn_Regulators:AP3401
- added C305, C402, C404, C406, C408, C414: 1uF, Capacitor_SMD:C_0402_1005Metric, symbol Daxxn_Device:C
- added C306, C395, C396, C397, C398, C399, C400, C401, C403, C405, C407, C409, C415: 100nF, Capacitor_SMD:C_0402_1005Metric, symbol Daxxn_Device:C
- added C384, C385, C386, C387: 47uF, Capacitor_SMD:C_1210_3225Metric, symbol Daxxn_Device:C
- added C388: 10uF, Capacitor_SMD:C_1210_3225Metric, symbol Daxxn_Device:C
- added FB15, FB18: 100 @ 100MHz, Inductor_SMD:L_1812_4532Metric, symbol Daxxn_Device:FerriteBead
- added FB16, FB17, FB19, FB20: 100 @ 100MHz, Inductor_SMD:L_0603_1608Metric, symbol Daxxn_Device:FerriteBead
- added R230, R231: 22, Resistor_SMD:R_0402_1005Metric, symbol Daxxn_Device:R
- added R232, R238, R239, R240, R241: 10m, Daxxn_Passives:R_Shunt_0612, symbol Daxxn_Device:R_Sense
- added R89: 10K, Resistor_SMD:R_0402_1005Metric, symbol Daxxn_Device:R
- added U23, U24: KSZ9021RN, Daxxn_Packages:QFN-48-1EP_7x7mm_P0.5mm_EP5.15x5.15mm, symbol Daxxn_IC:KSZ9021RN
- added U46: TPS54308, Daxxn_Packages:TSOT-23-6, symbol Daxxn_Regulators:TPS54308
- added U47: PCA9517, Package_SO:SOIC-8_3.9x4.9mm_P1.27mm, symbol Daxxn_IC:PCA9517
- added U48, U49, U50, U51, U52: INA231AIYFFR, Daxxn_Packages:DSBGA-12_3x4_1.418x1.675mm(YFF12), symbol Daxxn_IC:INA231AIYFFR
- C321: value 22pF -> 100nF
- JP1: footprint (none) -> Connector_PinHeader_2.54mm:PinHeader_1x02_P2.54mm_Vertical
- L6: value 2.2uH -> 4.7uH
- R11: footprint (none) -> Resistor_SMD:R_0402_1005Metric
- R17, R18: value 2.2K -> 4.7K
- R208: value 100K -> 49.9K
- R209: value 100K -> 48.7K
- R3: value 430K -> 453K
- R50: value R -> 226K
- R51: value R -> 100K
- U10: footprint Daxxn_Packages:100-VQFN-GND_12X12 -> Daxxn_Packages:VQFN-100_EP_12x12_Pitch0.4mm
Connections:
- net SMPS-PGOOD is gone; now on net MAIN-PG: D10.2 (A)
- net AVDDH: now also U23.1 (AVDDH), U23.12 (AVDDH), U23.16 (DVDDH), U23.34 (DVDDH), U23.40 (DVDDH), U23.47 (AVDDH), U24.1 (AVDDH), U24.12 (AVDDH), U24.16 (DVDDH), U24.34 (DVDDH), U24.40 (DVDDH), U24.47 (AVDDH)
- net AVDDL: now also C335.1, C336.1, C337.1, C338.1, C339.1, C362.1, C363.1, C364.1, C365.1, C366.1, FB4.2, FB7.2, U23.4 (AVDDL), U23.9 (AVDDL), U24.4 (AVDDL), U24.9 (AVDDL); no longer C320.1, C326.1, C327.1, C342.1, C343.1, C344.1, C345.1, C346.1, C358.1, C359.1, FB2.2, FB5.2
- net DVDD: now also R232.1, U49.D1 (BUS); no longer C115.1, C116.1, C117.1, C118.1, U4.J18 (VDDSHV6), U4.L18 (VDDSHV1), U4.M19 (VDDSHV1), U4.T7 (VDDSHV4)
- net DVDDL: now also C320.1, C326.1, C327.1, C342.1, C343.1, C344.1, C345.1, C346.1, C358.1, C359.1, FB2.2, FB5.2, U23.14 (DVDDL), U23.18 (DVDDL), U23.23 (DVDDL), U23.26 (DVDDL), U23.30 (DVDDL), U23.39 (DVDDL), U24.14 (DVDDL), U24.18 (DVDDL), U24.23 (DVDDL), U24.26 (DVDDL), U24.30 (DVDDL), U24.39 (DVDDL); no longer C335.1, C336.1, C337.1, C338.1, C339.1, C362.1, C363.1, C364.1, C365.1, C366.1, FB4.2, FB7.2
- net ETH-AVDDL-PLL: now also U23.44 (AVDDL-PLL), U24.44 (AVDDL-PLL)
- net MD1: now also U46.5 (EN)
- net PMBUS-SCK: now also U47.7 (SCLK_{B})
- net PMBUS-SDA: now also U47.6 (SDA_{B})
- net VCC: now also C388.1, U46.3 (VIN)
- net VDD: now also C395.1, C397.1, C398.1, C399.1, C400.1, C401.1, R238.1, R89.1, U47.1 (VCC_{A}), U48.B1 (VCC), U48.B3 (A0), U48.C3 (A1), U49.B1 (VCC), U49.B3 (A0), U50.B1 (VCC), U50.D1 (BUS), U51.B1 (VCC), U52.B1 (VCC); no longer C103.1, C104.1, C105.1, C106.1, C107.1, C108.1, C109.1, C110.1, C111.1, C112.1, C113.1, C114.1, U4.F11 (VDDSHV-MCU), U4.F15 (VDDSHV0), U4.G12 (VDDSHV-MCU), U4.G14 (VDDSHV0), U4.H9 (VDDSHV-CANUART), U4.N18 (VDDSHV3), U4.P18 (VDDSHV3), U4.T19 (VDDSHV3), U4.U18 (VDDSHV3), U4.W16 (VDDSHV2), U4.W19 (VDDSHV2), U4.Y13 (VDDA-3P3-USB)
- net VDD-CORE: now also FB18.2, R240.1, U48.D1 (BUS)
- net VDD-DDR: now also R241.1, U51.D1 (BUS); no longer C204.1, C205.1, C206.1, C207.1, C208.1, C209.1, U4.K9 (VDDS-DDR), U4.L8 (VDDS-DDR), U4.M9 (VDDS-DDR-C), U4.P9 (VDDS-DDR), U4.R8 (VDDS-DDR)
- net VDD-ETH: now also C384.1, C385.1, C386.1, C387.1, R239.1, U52.D1 (BUS); no longer C318.1, C319.1, C321.1, C328.1, C329.1, C333.1, C334.1, C340.1, C341.1, C360.1, C361.1, C367.1, C368.1, FB2.1, FB3.1, FB4.1, FB5.1, FB7.1, FB8.1
- net VDD-MMC: now also C414.1, C415.1, FB20.1; no longer C195.1, C198.1, C202.1, C203.1, U4.G17 (VDDSHV5)
- net VDD-PWR: now also C396.1, U47.8 (VCC_{B})
- net VDDA: now also C305.1, C306.1, FB19.1; no longer C131.1, C132.1, C133.1, C134.1, C135.1, C136.1, C137.1, C142.1, C185.1, C186.1, C187.1, C188.1, U4.G16 (VDDA-TEMP1), U4.G7 (VDDS-OSC0), U4.L11 (VDDA-MCU), U4.L14 (VDDA-PLL2), U4.T9 (VDDA-TEMP0), U4.U11 (VDDA-PLL0), U4.U15 (VDDA-PLL1), U4.W10 (VDDA-1P8-OLDI0), U4.W14 (VDDA-1P8-CSIRX0), U4.W9 (VDDA-1P8-OLDI0), U4.Y11 (VDDA-1P8-USB)
- net VDDA-PWR: now also D9.2 (A)
- net at R208.2, R209.1: now also U46.4 (FB); no longer C321.2
- net at L6.1: now also C321.1, U46.2 (SW)
- net AGNDH renamed GND
- net GND: now also C305.2, C306.2, C384.2, C385.2, C386.2, C387.2, C388.2, C395.2, C396.2, C397.2, C398.2, C399.2, C400.2, C401.2, C402.2, C403.2, C404.2, C405.2, C406.2, C407.2, C408.2, C409.2, C414.2, C415.2, U23.13 (GND), U23.29 (GND), U23.49 (GND), U24.13 (GND), U24.29 (GND), U24.49 (GND), U46.1 (GND), U47.4 (GND), U48.C1 (GND), U49.C1 (GND), U49.C3 (A1), U50.B3 (A0), U50.C1 (GND), U50.C3 (A1), U51.C1 (GND), U52.C1 (GND)
- net POWER-PGOOD renamed MAIN-PG
- net VPP-SS renamed DDR-VPP-SS
- new net: C131.1, C132.1, C133.1, C134.1, C135.1, C136.1, C137.1, C142.1, C185.1, C186.1, C187.1, C188.1, FB19.2, U4.G16 (VDDA-TEMP1), U4.G7 (VDDS-OSC0), U4.L11 (VDDA-MCU), U4.L14 (VDDA-PLL2), U4.T9 (VDDA-TEMP0), U4.U11 (VDDA-PLL0), U4.U15 (VDDA-PLL1), U4.W10 (VDDA-1P8-OLDI0), U4.W14 (VDDA-1P8-CSIRX0), U4.W9 (VDDA-1P8-OLDI0), U4.Y11 (VDDA-1P8-USB)
- new net: U10.12 (NC), U10.13 (NC), U10.4 (NC), U10.80 (NC)
- new net: R241.2, U51.D3 (IN+)
- new net: R241.3, U51.D2 (IN-)
- new net: C195.1, C198.1, C202.1, C203.1, FB20.2, U4.G17 (VDDSHV5)
- new net: R239.2, U52.D3 (IN+)
- new net: R239.3, U52.D2 (IN-)
- new net: R232.2, U49.D3 (IN+)
- new net: R232.3, U49.D2 (IN-)
- new net: U49.B2 (NC), U49.C2 (NC)
- new net: C321.2, U46.6 (BOOT)
- new net: U52.B2 (NC), U52.C2 (NC)
- new net: R240.2, U48.D3 (IN+)
- new net: R240.3, U48.D2 (IN-)
- new net: R231.2, U47.2 (SCLK_{A})
- new net: R230.1, U47.3 (SDA_{A})
- new net: R89.2, U47.5 (EN)
- new net: U51.B2 (NC), U51.C2 (NC)
- new net: R238.2, U50.D3 (IN+)
- new net: R238.3, U50.D2 (IN-)
- new net: U48.B2 (NC), U48.C2 (NC)
- new net: U50.B2 (NC), U50.C2 (NC)
- new net I2C-SYS-SCL: R231.1, U48.A1 (SCL), U49.A1 (SCL), U50.A1 (SCL), U51.A1 (SCL), U52.A1 (SCL)
- new net I2C-SYS-SDA: R230.2, U48.A2 (SDA), U49.A2 (SDA), U50.A2 (SDA), U51.A2 (SDA), U52.A2 (SDA)
- new net SOC-DVDD: C404.1, C405.1, FB16.1, R232.4
- new net SOC-VDD: C402.1, C403.1, FB15.1, R238.4
- new net SOC-VDD-CORE: C408.1, C409.1, FB18.1, R240.4
- new net SOC-VDD-DDR: C406.1, C407.1, FB17.1, R241.4
- new net VDD-CORE-ETH: C318.1, C319.1, C328.1, C329.1, C333.1, C334.1, C340.1, C341.1, C360.1, C361.1, C367.1, C368.1, FB2.1, FB3.1, FB4.1, FB5.1, FB7.1, FB8.1, R239.4
- new net VDDS-DDR: C204.1, C205.1, C206.1, C207.1, C208.1, C209.1, FB17.2, U4.K9 (VDDS-DDR), U4.L8 (VDDS-DDR), U4.M9 (VDDS-DDR-C), U4.P9 (VDDS-DDR), U4.R8 (VDDS-DDR)
- new net VDDSHV-MCU: C103.1, C104.1, C105.1, C106.1, C107.1, C108.1, C109.1, C110.1, C111.1, C112.1, C113.1, C114.1, FB15.2, U4.F11 (VDDSHV-MCU), U4.F15 (VDDSHV0), U4.G12 (VDDSHV-MCU), U4.G14 (VDDSHV0), U4.H9 (VDDSHV-CANUART), U4.N18 (VDDSHV3), U4.P18 (VDDSHV3), U4.T19 (VDDSHV3), U4.U18 (VDDSHV3), U4.W16 (VDDSHV2), U4.W19 (VDDSHV2), U4.Y13 (VDDA-3P3-USB)
- new net VDDSHV1: C115.1, C116.1, C117.1, C118.1, FB16.2, U4.J18 (VDDSHV6), U4.L18 (VDDSHV1), U4.M19 (VDDSHV1), U4.T7 (VDDSHV4)
- new net ~{DVDD-ALERT}: U49.A3 (~{ALERT})
- new net ~{VDD-ALERT}: U50.A3 (~{ALERT})
- new net ~{VDD-CORE-ALERT}: U48.A3 (~{ALERT})
- new net ~{VDD-DDR-ALERT}: U51.A3 (~{ALERT})
- new net ~{VDD-ETH-ALERT}: U52.A3 (~{ALERT})
Other:
- note added: "116mA"
- note added: "1300mA"
- note added: "563mA"
- note added: "58mA"
- note added: "75mA"
- note added: "POWER SEQUENCER"
- note removed: "120mA"
- note removed: "221mA"
- note removed: "500mA"
- note removed: "53.8mA"
- note removed: "66.6mA"
- note removed: "POWER MANAGER"
- moved on the sheet: C195, C198, C202, C203, C307, C308, C309, C310, C311, C312, C313, C314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

Commit message: Start PCB layout
Parts:
- removed J5: USB PWR CONN, Daxxn_Connectors:8-Pin_Molex_Mini-Fit_Jr_Vertical_Mount, symbol Connector_Generic:Conn_02x04_Top_Bottom
- removed R11: 10K, Resistor_SMD:R_0402_1005Metric, symbol Daxxn_Device:R
- added C167: 100nF, Capacitor_SMD:C_0402_1005Metric, symbol Daxxn_Device:C
- added J26: PWR CONN, Daxxn_Connectors:4-Pin_Molex_Mini-Fit_Jr_Vertical_Mount, symbol Connector_Generic:Conn_02x02_Odd_Even
- added J3, J4: EN1 JUMPER, Connector_PinHeader_2.54mm:PinHeader_2x03_P2.54mm_Vertical, symbol Connector_Generic:Conn_02x03_Counter_Clockwise
- added R35: 100K, Resistor_SMD:R_0402_1005Metric, symbol Daxxn_Device:R
- added R45, R46, R48, R49: 10K, Resistor_SMD:R_0402_1005Metric, symbol Daxxn_Device:R
- added U7: MAX809, Daxxn_Packages:SOT-23-3, symbol Daxxn_IC:MAX809
- JP1: value Jumper -> VPP EN JUMPER
- U5: footprint Package_DFN_QFN:QFN-72-1EP_10x10mm_P0.5mm_EP6x6mm -> Daxxn_Packages:QFN-72-1EP_10x10mm_P0.5mm_EP6x6mm
- renumbered C102 to C1, C111 to C10, C272 to C100, C30 to C101, C18 to C102, C414 to C103, C415 to C104, C195 to C105, C198 to C106, C202 to C107, C203 to C108, C31 to C109, C110 to C11, C23 to C110, C32 to C111, C34 to C112, C35 to C113, C36 to C114, C37 to C115, C38 to C116, C273 to C117, C406 to C118, C407 to C119, C109 to C12, C204 to C120, C205 to C121, C206 to C122, C207 to C123, C208 to C124, C209 to C125, C51 to C126, C33 to C127, C52 to C128, C53 to C129, C108 to C13, C54 to C130, C200 to C131, C55 to C132, C56 to C133, C57 to C134, C274 to C135, C39 to C136, C58 to C137, C396 to C138, C395 to C139, C107 to C14, C218 to C140, C217 to C141, C216 to C142, C215 to C143, C214 to C144, C213 to C145, C212 to C146, C211 to C147, C210 to C148, C264 to C149, C106 to C15, C60 to C150, C307 to C151, C308 to C152, C309 to C153, C310 to C154, C311 to C155, C312 to C156, C313 to C157, C314 to C158, C315 to C159, C105 to C16, C316 to C160, C317 to C161, C399 to C162, C45 to C163, C46 to C164, C48 to C165, C47 to C166, C318 to C168, C319 to C169, C104 to C17, C320 to C170, C326 to C171, C327 to C172, C358 to C173, C359 to C174, C374 to C175, C375 to C176, C228 to C177, C229 to C178, C227 to C179, C103 to C18, C226 to C180, C360 to C181, C361 to C182, C362 to C183, C363 to C184, C364 to C185, C365 to C186, C366 to C187, C372 to C188, C373 to C189, C233 to C19, C221 to C190, C225 to C191, C224 to C192, C223 to C193, C222 to C194, C276 to C195, C367 to C196, C368 to C197, C369 to C198, C370 to C199, C101 to C2, C404 to C20, C371 to C200, C79 to C201, C5 to C202, C80 to C203, C81 to C204, C398 to C205, C347 to C206, C348 to C207, C349 to C208, C350 to C209, C405 to C21, C351 to C210, C352 to C211, C353 to C212, C354 to C213, C355 to C214, C356 to C215, C357 to C216, C6 to C217, C7 to C218, C8 to C219, C115 to C22, C9 to C220, C340 to C221, C341 to C222, C342 to C223, C343 to C224, C344 to C225, C345 to C226, C346 to C227, C397 to C228, C333 to C229, C116 to C23, C334 to C230, C335 to C231, C336 to C232, C337 to C233, C338 to C234, C339 to C235, C75 to C236, C76 to C237, C328 to C238, C329 to C239, C117 to C24, C330 to C240, C331 to C241, C332 to C242, C277 to C243, C77 to C244, C78 to C245, C400 to C246, C379 to C247, C378 to C248, C82 to C249, C118 to C25, C83 to C250, C84 to C251, C85 to C252, C86 to C253, C87 to C254, C88 to C255, C89 to C256, C90 to C257, C91 to C258, C92 to C259, C197 to C26, C67 to C260, C68 to C261, C93 to C262, C94 to C263, C95 to C264, C377 to C265, C376 to C266, C10 to C267, C11 to C268, C19 to C269, C1 to C27, C20 to C270, C401 to C271, C49 to C272, C50 to C273, C59 to C274, C61 to C275, C267 to C276, C268 to C277, C269 to C278, C270 to C279, C2 to C28, C321 to C280, C388 to C281, C322 to C282, C323 to C283, C387 to C284, C386 to C285, C385 to C286, C384 to C287, C324 to C288, C325 to C289, C196 to C29, C219 to C3, C3 to C30, C184 to C31, C4 to C32, C201 to C33, C182 to C34, C183 to C35, C408 to C36, C409 to C37, C119 to C38, C239 to C39, C220 to C4, C240 to C40, C241 to C41, C242 to C42, C243 to C43, C120 to C44, C193 to C45, C194 to C46, C121 to C47, C234 to C48, C235 to C49, C402 to C5, C236 to C50, C237 to C51, C238 to C52, C122 to C53, C123 to C54, C189 to C55, C190 to C56, C191 to C57, C192 to C58, C124 to C59, C403 to C6, C125 to C60, C126 to C61, C127 to C62, C128 to C63, C129 to C64, C130 to C65, C71 to C66, C72 to C67, C73 to C68, C74 to C69, C114 to C7, C100 to C70, C12 to C71, C13 to C72, C14 to C73, C15 to C74, C16 to C75, C17 to C76, C271 to C77, C275 to C78, C305 to C79, C113 to C8, C306 to C80, C131 to C81, C132 to C82, C133 to C83, C134 to C84, C135 to C85, C136 to C86, C137 to C87, C142 to C88, C185 to C89, C112 to C9, C186 to C90, C187 to C91, C188 to C92, C24 to C93, C25 to C94, C26 to C95, C199 to C96, C27 to C97, C28 to C98, C29 to C99, D21 to D1, D12 to D10, D14 to D11, D9 to D12, D22 to D2, D23 to D3, D24 to D4, D16 to D5, D15 to D6, D10 to D7, D13 to D8, D11 to D9, FB15 to FB1, FB7 to FB10, FB9 to FB11, FB8 to FB12, FB6 to FB13, FB5 to FB14, FB4 to FB15, FB3 to FB16, FB12 to FB17, FB11 to FB18, FB16 to FB2, FB18 to FB3, FB19 to FB4, FB20 to FB5, FB17 to FB6, FB1 to FB7, FB2 to FB8, FB10 to FB9, Q5 to Q1, Q4 to Q2, Q7 to Q3, Q6 to Q4, R61 to R1, R1 to R10, R67 to R11, R4 to R12, R68 to R13, R5 to R14, R2 to R15, R8 to R16, R6 to R17, R10 to R18, R12 to R19, R62 to R2, R9 to R20, R13 to R21, R14 to R22, R16 to R23, R19 to R24, R89 to R25, R136 to R26, R17 to R27, R18 to R28, R137 to R29, R63 to R3, R21 to R30, R230 to R31, R22 to R32, R231 to R33, R50 to R34, R51 to R36, R238 to R37, R3 to R38, R7 to R39, R64 to R4, R232 to R40, R240 to R41, R20 to R42, R34 to R43, R35 to R44, R241 to R47, R65 to R5, R37 to R50, R239 to R51, R73 to R52, R75 to R53, R78 to R54, R76 to R55, R147 to R56, R74 to R57, R72 to R58, R82 to R59, R15 to R6, R77 to R60, R208 to R61, R120 to R62, R40 to R63, R26 to R64, R38 to R65, R31 to R66, R33 to R67, R39 to R68, R71 to R69, R52 to R7, R209 to R70, R69 to R8, R70 to R9, TP9 to TP1, TP6 to TP11, TP15 to TP12, TP3 to TP2, TP1 to TP3, TP11 to TP4, TP2 to TP5, TP7 to TP6, TP8 to TP7, TP4 to TP8, TP12 to TP9, U4 to U1, U7 to U10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
Connections:
- net GND: now also U16.B3 (A0), U20.C3 (A1), C167.2, J26.2 (Pin_2), J26.4 (Pin_4), J3.4 (Pin_4), J4.4 (Pin_4), R48.1, R49.1, U7.1 (GND)
- net I2C-SYS-SCL: now also U20.B3 (A0)
- net VCC: now also J26.1 (Pin_1), J26.3 (Pin_3)
- net VDD: now also U16.C3 (A1), J3.6 (Pin_6), J4.6 (Pin_6), R45.2, R46.2
- net VDDA: now also C167.1, R35.1, U7.3 (VCC)
- net SD-CARD-PWR-SEL renamed MMC-EN2
- net MMC-EN2: now also J4.1 (Pin_1), J4.2 (Pin_2), J4.3 (Pin_3), R46.1, R49.2
- net VSEL-SD renamed MMC-EN1
- net MMC-EN1: now also J3.1 (Pin_1), J3.2 (Pin_2), J3.3 (Pin_3), R45.1, R48.2
- new net SD-CARD-PWR-SEL1: J3.5 (Pin_5)
- new net SD-CARD-PWR-SEL2: J4.5 (Pin_5)
- new net ~{ANALOG-RESET}: R35.2, U7.2 (~{RESET})
Other:
- note added: "ADDRESS: 0x40"
- note added: "ADDRESS: 0x41"
- note added: "ADDRESS: 0x44"
- note added: "ADDRESS: 0x45"
- note added: "ADDRESS: 0x4C"
- note added: "POWER INDICATORS"
- note removed: "CHECK VALUES"
- note removed: "INDICATORS"
- moved on the sheet: C10, C103, C104, C105, C106, C107, C108, C11, C118, C119, C12, C120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

Commit message: Fix power net names and increase PCB size
Connections:
- net SOC-DVDD is gone; now on net DVDD: C20.1, C21.1, FB2.1, R40.4
- net VDD-CORE-ETH is gone; now on net VDD-ETH: C168.1, C169.1, C181.1, C182.1, C196.1, C197.1, C221.1, C222.1, C229.1, C230.1, C238.1, C239.1, FB10.1, FB12.1, FB14.1, FB15.1, FB16.1, FB8.1, R51.4
- net VDDS-DDR is gone; now on net SOC-VDD-DDR: C120.1, C121.1, C122.1, C123.1, C124.1, C125.1, FB6.2, U1.K9 (VDDS-DDR), U1.L8 (VDDS-DDR), U1.M9 (VDDS-DDR-C), U1.P9 (VDDS-DDR), U1.R8 (VDDS-DDR)
- net VDDSHV-MCU is gone; now on net SOC-VDD: C10.1, C11.1, C12.1, C13.1, C14.1, C15.1, C16.1, C17.1, C18.1, C7.1, C8.1, C9.1, FB1.2, U1.F11 (VDDSHV-MCU), U1.F15 (VDDSHV0), U1.G12 (VDDSHV-MCU), U1.G14 (VDDSHV0), U1.H9 (VDDSHV-CANUART), U1.N18 (VDDSHV3), U1.P18 (VDDSHV3), U1.T19 (VDDSHV3), U1.U18 (VDDSHV3), U1.W16 (VDDSHV2), U1.W19 (VDDSHV2), U1.Y13 (VDDA-3P3-USB)
- net VDDSHV1 is gone; now on net DVDD: C22.1, C23.1, C24.1, C25.1, FB2.2, U1.J18 (VDDSHV6), U1.L18 (VDDSHV1), U1.M19 (VDDSHV1), U1.T7 (VDDSHV4)
- net DVDD: no longer C113.2, C114.1, C115.1, C116.1, C117.1, L3.2, R18.1, R40.1, TP4.1, U11.D1 (BUS)
- net SOC-VDD: no longer C5.1, C6.1, FB1.1, R37.4
- net SOC-VDD-CORE: now also C38.1, C39.1, C40.1, C41.1, C42.1, C43.1, C44.1, C45.1, C46.1, C47.1, C48.1, C49.1, C50.1, C51.1, C52.1, C53.1, C54.1, C55.1, C56.1, C57.1, C58.1, C59.1, C60.1, C61.1, C62.1, C63.1, C64.1, C65.1, FB3.2, U1.F8 (VDD-CANUART), U1.H8 (VDD_CORE), U1.J11 (VDD_CORE), U1.J12 (VDDR-CORE), U1.J14 (VDD_CORE), U1.K16 (VDDR-CORE), U1.K17 (VDD_CORE), U1.L12 (VDD_CORE), U1.L15 (VDD_CORE), U1.M16 (VDD_CORE), U1.N11 (VDD_CORE), U1.N12 (VDDR-CORE), U1.N13 (VDD_CORE), U1.N14 (VDDR-CORE), U1.N8 (VDD_CORE), U1.P16 (VDDR-CORE), U1.P17 (VDD_CORE), U1.R11 (VDD_CORE), U1.R12 (VDDR-CORE), U1.R14 (VDD_CORE), U1.T10 (VDDR-CORE), U1.U12 (VDD_CORE), U1.U14 (VDDR-CORE), U1.V15 (VDD_CORE), U1.V17 (VDD_CORE), U1.V8 (VDD_CORE), U1.W12 (VDDA-CORE-USB), U1.W13 (VDDA-CORE-CSIRX0); no longer C36.1, C37.1, FB3.1, R41.4
- net SOC-VDD-DDR: no longer C118.1, C119.1, FB6.1, R47.4
- net VDD: now also C5.1, C6.1, FB1.1, R37.4; no longer C73.2, C74.1, C75.1, C76.1, C77.1, C78.1, L1.2, R10.1, R37.1, TP2.1, U8.D1 (BUS)
- net VDD-CORE: now also C36.1, C37.1, FB3.1, R41.4; no longer C100.1, C38.1, C39.1, C40.1, C41.1, C42.1, C43.1, C44.1, C45.1, C46.1, C47.1, C48.1, C49.1, C50.1, C51.1, C52.1, C53.1, C54.1, C55.1, C56.1, C57.1, C58.1, C59.1, C60.1, C61.1, C62.1, C63.1, C64.1, C65.1, C95.2, C96.1, C97.1, C98.1, C99.1, FB3.2, L2.2, R11.1, R16.1, R41.1, TP3.1, U1.F8 (VDD-CANUART), U1.H8 (VDD-CORE), U1.J11 (VDD-CORE), U1.J12 (VDDR-CORE), U1.J14 (VDD-CORE), U1.K16 (VDDR-CORE), U1.K17 (VDD-CORE), U1.L12 (VDD-CORE), U1.L15 (VDD-CORE), U1.M16 (VDD-CORE), U1.N11 (VDD-CORE), U1.N12 (VDDR-CORE), U1.N13 (VDD-CORE), U1.N14 (VDDR-CORE), U1.N8 (VDD-CORE), U1.P16 (VDDR-CORE), U1.P17 (VDD-CORE), U1.R11 (VDD-CORE), U1.R12 (VDDR-CORE), U1.R14 (VDD-CORE), U1.T10 (VDDR-CORE), U1.U12 (VDD-CORE), U1.U14 (VDDR-CORE), U1.V15 (VDD-CORE), U1.V17 (VDD-CORE), U1.V8 (VDD-CORE), U1.W12 (VDDA-CORE-USB), U1.W13 (VDDA-CORE-CSIRX0), U14.D1 (BUS)
- net VDD-DDR: now also C118.1, C119.1, FB6.1, R47.4; no longer C130.2, C131.1, C132.1, C133.1, C134.1, C135.1, L4.2, R22.1, R47.1, TP5.1, U16.D1 (BUS)
- net VDD-ETH: no longer C284.1, C285.1, C286.1, C287.1, C288.1, C289.1, L6.2, R51.1, R61.1, TP12.1, U20.D1 (BUS)
- net SOC-VDDA: now reaches C81.1, C82.1, C83.1, C84.1, C85.1, C86.1, C87.1, C88.1, C89.1, C90.1, C91.1, C92.1, FB4.2, U1.G16 (VDDA-TEMP1), U1.G7 (VDDS-OSC0), U1.L11 (VDDA-MCU), U1.L14 (VDDA-PLL2), U1.T9 (VDDA-TEMP0), U1.U11 (VDDA-PLL0), U1.U15 (VDDA-PLL1), U1.W10 (VDDA-1P8-OLDI0), U1.W14 (VDDA-1P8-CSIRX0), U1.W9 (VDDA-1P8-OLDI0), U1.Y11 (VDDA-1P8-USB)
- net SOC-VDD-MMC: now reaches C105.1, C106.1, C107.1, C108.1, FB5.2, U1.G17 (VDDSHV5)
- net ETH-AVDDL-PLL renamed ETH1-AVDDL-PLL
- net ETH1-AVDDL-PLL: no longer C240.1, C241.1, C242.1, FB16.2, U24.44 (AVDDL-PLL)
- new net ETH2-AVDDL-PLL: C240.1, C241.1, C242.1, FB16.2, U24.44 (AVDDL-PLL)
- new net MON-DVDD: C113.2, C114.1, C115.1, C116.1, C117.1, L3.2, R18.1, R40.1, TP4.1, U11.D1 (BUS)
- new net MON-VDD: C73.2, C74.1, C75.1, C76.1, C77.1, C78.1, L1.2, R10.1, R37.1, TP2.1, U8.D1 (BUS)
- new net MON-VDD-CORE: C100.1, C95.2, C96.1, C97.1, C98.1, C99.1, L2.2, R16.1, R41.1, TP3.1, U14.D1 (BUS)
- new net MON-VDD-CORE-ETH: C284.1, C285.1, C286.1, C287.1, C288.1, C289.1, L6.2, R51.1, R61.1, TP12.1, U20.D1 (BUS)
- new net MON-VDD-DDR: C130.2, C131.1, C132.1, C133.1, C134.1, C135.1, L4.2, R22.1, R47.1, TP5.1, U16.D1 (BUS)

Commit message: (WIP) Still laying out PCB
Parts:
- removed C113, C130, C73, C95: 100pF, Capacitor_SMD:C_0402_1005Metric, symbol Daxxn_Device:C
- added C459, C460: 68uF, Capacitor_SMD:C_1206_3216Metric, symbol Daxxn_Device:C
- added C461, C462, C463: 47uF, Capacitor_SMD:C_1206_3216Metric, symbol Daxxn_Device:C
- added C464: 4.7pF, Capacitor_SMD:C_0402_1005Metric, symbol Daxxn_Device:C
- added C465: 10uF, Capacitor_SMD:C_1210_3225Metric, symbol Daxxn_Device:C
- C100: value 10uF -> 68uF; footprint Capacitor_SMD:C_1210_3225Metric -> Capacitor_SMD:C_1206_3216Metric
- C101: value 4.62pF -> 10pF
- C102: value 47pF -> 22pF
- C109: value 4.37n -> 2.7nF
- C110: value 330pF -> 2.7nF
- C112, C129, C72, C94: value 100nF -> 6.8nF
- C127: value 100pF -> 10pF
- C128: value 150pF -> 10pF
- C136: value 820pF -> 2.2nF
- C137: value 1.5nF -> 2.7nF
- C78: value 10uF -> 47uF; footprint Capacitor_SMD:C_1210_3225Metric -> Capacitor_SMD:C_1206_3216Metric
- L1: value 4.7uH -> 8.2uH
- L3: value 5.6uH -> 10uH
- L4: value 8.2uH -> 6.8uH
- R10: value 10K -> 316K
- R12: value 3.2K -> 100K
- R14: value 4.32K -> 13K
- R15: value 24K -> 15.4K
- R16: value 1K -> 7.5K
- R17: value 16K -> 100K
- R18, R22: value 10K -> 127K
- R19: value 8K -> 100K
- R21: value 8.2K -> 14.3K
- R23: value 20K -> 100K
- R32: value 160K -> 383K
- R42: now not fitted
Connections:
- net GND: now also J3.3 (Pin_3), J4.3 (Pin_3), C459.2, C460.2, C461.2, C462.2, C463.2, C464.2, C465.2; no longer R48.1, R49.1
- net MMC-EN1: no longer J3.1 (Pin_1), J3.3 (Pin_3), R45.1, R48.2
- net MMC-EN2: no longer J4.1 (Pin_1), J4.3 (Pin_3), R46.1, R49.2
- net MON-DVDD: now also C463.1
- net MON-VDD-CORE: now also C459.1, C460.1
- net MON-VDD-DDR: now also C461.1, C462.1
- net PWR-RCLK-SY: now also C464.1
- net VDD: now also R48.1, R49.1; no longer J3.6 (Pin_6), J4.6 (Pin_6)
- net VPWR: now also C465.1
- new net: J3.1 (Pin_1), R45.1
- new net: J3.6 (Pin_6), R48.2
- new net: J4.1 (Pin_1), R46.1
- new net: J4.6 (Pin_6), R49.2
Other:
- moved on the sheet: C100, C114, C115, C116, C117, C131, C132, C133, C134, C135, C30, C74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
