File: MotherBoard/BenchyMotherBoard-PCB/Control.kicad_sch (KiCad schematic)
At the start: 46 parts, among them J3 JTAG-MAIN-XDS110, SW2 POWER SWITCH, U1 74LVC1G17GV, U29 74LVC3G17GS, U30 SN74HCS21PWR, U31 PCA9634, U4 AM6254ATCGGAALW, Y2 32.7KHz, Y5 16MHz

Commit message: Add new ethernet chip - KSZ9031
Parts:
- removed U1: 74LVC1G17GV, Daxxn_Packages:SOT-753, symbol Daxxn_Logic:74LVC1G17GV
- removed U29: 74LVC3G17GS, Daxxn_Packages:X2SON-8_1.4x1mm_P0.35mm, symbol Daxxn_Logic:74LVC3G17GS
- removed U30: SN74HCS21PWR, Daxxn_Packages:TSSOP-14_4.4x5mm_P0.65mm, symbol Daxxn_Logic:SN74HCS21PWR
- added C99 (x4): 100nF, Capacitor_SMD:C_0201_0603Metric, symbol Daxxn_Device:C
- added D30: GREEN, LED_SMD:LED_0805_2012Metric, symbol Daxxn_Device:LED
- added JP3: Button Enable Jumper, Connector_PinHeader_2.54mm:PinHeader_1x02_P2.54mm_Vertical, symbol Daxxn_Other:Jumper
- added R120 (x2): 4.7K, Resistor_SMD:R_0402_1005Metric, symbol Daxxn_Device:R
- added R120 (x6), R55 (x5): 10K, Resistor_SMD:R_0402_1005Metric, symbol Daxxn_Device:R
- added R55: 1K, Resistor_SMD:R_0402_1005Metric, symbol Daxxn_Device:R
- added S1, S4: WARM RESET, Daxxn_Switches:TL3365AF180QG, symbol Daxxn_Buttons:GENERIC-SWITCH-2P
- added TP13: TP-~{POR}, symbol Connector:TestPoint_Alt
- added TP14: TP-~{RESET-STATUS}, symbol Connector:TestPoint_Alt
- added U1: SN74HCS125BQAR, Daxxn_Packages:WQFN-14_B3x2.5mm_P0.5mm, symbol Daxxn_Logic:SN74HCS125BQAR
- added U29: 74LVC1G17GV, Daxxn_Packages:SOT-753, symbol Daxxn_Logic:74LVC1G17GV
- added U43, U44: 74HCT2G08, Daxxn_Packages:WSON-6_1.5x1.5mm_P0.5mm, symbol Daxxn_Logic:SN74LVC1G11DRYR
Connections:
- net GND: now also SW2.5 (B), C99.2, C99.2, C99.2, C99.2, JP3.1 (A), R120.1, R120.1, R120.2, S1.1, S4.1, U1.15 (GND), U1.7 (GND), U29.3 (GND), U43.2 (GND), U44.2 (GND)
- net POWER-PGOOD: now also U43.3 (B)
- net PWR-SWITCH: now also U29.4 (Y)
- net VCC: now also D30.2 (A)
- net VDD: now also C99.1, R120.1, R120.1, R120.2, R120.2, R55.1, R55.1, R55.1, R55.1, R55.1, U1.14 (VCC), U29.5 (VCC), U43.5 (VCC)
- net ~{JTAG-RESET}: now also U44.6 (C)
- net ~{MCU-RESET}: now also R120.1, R120.2, U44.4 (Y)
- net ~{MCU-RESET}-DEBOUNCE: now also U1.5 (2A)
- net ~{POR-OUT}: now also R120.1, R120.2, TP13.1
- net ~{RESET-REQ}: now also U43.4 (Y)
- net ~{RESET-REQ}-DEBOUNCE: now also U1.9 (3A)
- net ~{RESET-STATUS}: now also R120.1, R120.2, TP14.1
- net at SW2.4 (A): now also R55.1
- net at SW2.1 (A): now also U29.2 (A)
- net WKUP-UART-RX: now reaches U4.B4 (WKUP-UART0-RXD)
- net WKUP-UART-TX: now reaches U4.C5 (WKUP-UART0-TXD)
- new net: D30.1 (K), R55.2
- new net BTN-ENABLE: JP3.2 (B), R55.2, U1.1 (1~{OE}), U1.10 (3~{OE}), U1.13 (4~{OE}), U1.4 (2~{OE})
- new net DVDD: C99.1, R120.1, U44.5 (VCC)
- new net ~{MAIN-RESET}: U44.1 (A)
- new net ~{MCU-RESET}-BTN: R55.2, U1.6 (2Y), U43.1 (A)
- new net ~{PWR-RESET}: R55.2, U1.11 (4Y)
- new net ~{PWR-RESET}-DEBOUNCE: C99.1, R120.2, S1.2, U1.12 (4A)
- new net ~{RESET-REQ}-BTN: R55.2, U1.8 (3Y), U43.6 (C)
- new net ~{TEST1-BTN}: R55.2, U1.3 (1Y)
- new net ~{TEST1-BTN}-DEBOUNCE: C99.1, R120.2, S4.2, U1.2 (1A)
- no-connect marks 5 -> 3
Other:
- note added: "POWER SWITCH"
- company: (none) -> Daxxn Industries
- title: (none) -> Benchy Reloaded
- moved on the sheet: C99, R55, SW2B

Commit message: (WIP) Almost done with schematic
Parts:
- removed Y5: 16MHz, Daxxn_Passives:Resonator_SMD_3Pin_3.0x1.1mm, symbol Daxxn_Device:Resonator
- added C143, C144: 18pF, Capacitor_SMD:C_0402_1005Metric, symbol Daxxn_Device:C
- added C158: 1uF, Capacitor_SMD:C_0402_1005Metric, symbol Daxxn_Device:C
- added C158 (x3): 100nF, Capacitor_SMD:C_0201_0603Metric, symbol Daxxn_Device:C
- added D31: RED, LED_SMD:LED_0805_2012Metric, symbol Daxxn_Device:LED
- added Q2: NX6008NBKWX, Package_TO_SOT_SMD:SOT-323_SC-70, symbol Daxxn_Transistors:NX6008NBKWX
- added R102: 10K, Resistor_SMD:R_0402_1005Metric, symbol Daxxn_Device:R
- added R120 (x4): 0, Resistor_SMD:R_0402_1005Metric, symbol Daxxn_Device:R
- added R120: 1K, Resistor_SMD:R_0402_1005Metric, symbol Daxxn_Device:R
- added R120: 100, Resistor_SMD:R_0402_1005Metric, symbol Daxxn_Device:R
- added R23 (x4): 22, Resistor_SMD:R_0201_0603Metric, symbol Daxxn_Device:R
- added SW3: SW_DIP_x08, Button_Switch_SMD:SW_DIP_SPSTx08_Slide_6.7x21.88mm_W6.73mm_P2.54mm_LowProfile_JPin, symbol Switch:SW_DIP_x08
- added U53: LMK1C1104DQFR, Daxxn_Packages:WSON-8_2x2mm_P0.5mm, symbol Daxxn_Logic:LMK1C1104DQFR
- added X1: 25MHz, Daxxn_Passives:Crystal_SMD_4Pin_2.5x2.0mm, symbol Daxxn_Device:CMOS-OSCILLATOR
- added Y1: 25MHz, Daxxn_Passives:Crystal_SMD_4Pin_3.2x2.5mm, symbol Daxxn_Device:Crystal
- D27, D28: footprint (none) -> LED_SMD:LED_0805_2012Metric
- J3: footprint Connector_IDC:IDC-Header_2x12_P2.54mm_Vertical -> Connector_IDC:IDC-Header_2x10_P2.54mm_Vertical
- R120: value 10K -> 4.7K
- TP13, TP14: footprint (none) -> TestPoint:TestPoint_Pad_1.5x1.5mm
Connections:
- net DVDD: now also C158.1, C158.1, C158.1, C158.1, U53.6 (VDD), X1.4 (Vcc)
- net GND: now also C143.2, C144.1, C143.2, C144.1, C158.2, C158.2, C158.2, C158.2, Q2.2 (S), R102.1, R120.2, U53.4 (GND), X1.2 (GND), Y1.2, Y1.4; no longer C143.1, C144.2
- net MCU-ERR: now also Q2.1 (G)
- net VDD: now also D31.2 (A), R120.1; no longer J3.5 (VTREF)
- net ~{MCU-RESET}: no longer R120.1, R120.2, U44.4 (Y)
- net ~{MCU-RESET}-BTN: now also U44.3 (B); no longer U43.1 (A)
- net at U4.C2 (WKUP-LFOSC0-XI), Y2.2: now also C143.1; no longer C143.2
- net at U4.A3 (MCU-OSC0-XO): now also R120.1, R120.1
- net at U4.B2 (MCU-OSC0-XI): now also R120.1, R120.2
- net at U4.C1 (WKUP-LFOSC0-XO), Y2.1: now also C144.2; no longer C144.1
- net POWER-PGOOD: no longer names the net of U43.3 (B)
- net ~{EXT-REFCLK}: no longer names the net of U4.A18 (EXT-REFCLK1)
- new net: C143.1, R120.1, Y1.1
- new net: C144.2, R120.2, Y1.3
- new net: D31.1 (K), R120.1
- new net: Q2.3 (D), R120.2
- new net: R102.2, U53.2 (EN)
- new net: R23.2, U53.8 (Y1)
- new net: J3.5 (VTREF), R120.2
- new net: R23.2, U53.3 (Y0)
- new net: R23.2, U53.5 (Y2)
- new net: R23.2, U53.7 (Y3)
- new net CLKOUT0: U53.1 (CLK-IN), X1.3 (OUT)
- new net ETH1-CLKIN: R23.1
- new net ETH2-CLKIN: R23.1
- new net SOC-CLKIN: R120.2, R23.1
- new net USB-HUB-CLKIN: R23.1
- new net ~{WARM-RESET}: R120.1, R120.2, U44.4 (Y)
- no-connect marks 3 -> 4
Other:
- note added: "0"
- note added: "1"
- note added: "10"
- note added: "11"
- note added: "12"
- note added: "13"
- note added: "14"
- note added: "15"
- note added: "2"
- note added: "3"
- note added: "4"
- note added: "5"
- note added: "6"
- note added: "7"
- note added: "8"
- note added: "9"
- note added: "BACKUP BOOT"
- note added: "BOOT MODE OPTIONS"
- note added: "DESCRIPTION"
- note added: "Engineering BOOT"
- note added: "M25"
- note added: "N23"
- note added: "N24"
- note added: "N25"
- note added: "NAME"
- note added: "NUMBER"
- note added: "P21"
- note added: "P22"
- note added: "P24"
- note added: "PIN"
- note added: "PLL CONFIG"
- note added: "PRIMARY BOOT"
- note added: "PRIMARY CONFIG"
- note added: "R21"
- note added: "R23"
- note added: "R24"
- note added: "R25"
- note added: "RESERVED"
- note added: "SD-CARD ON SDMMC1"
- note added: "SERIAL NAND FLASH (QSPI)"
- note added: "SERIAL NOR FLASH (QSPI)"
- note added: "SLC NAND FLASH ON FMC"
- note added: "T22"
- note added: "T24"
- note added: "T25"
- note added: "U24"
- note added: "U25"
- note added: "UART / USB"
- note added: "eMMC ON SDMMC2"
- moved on the sheet: C143, C144, C99, J3, R120, Y2

Commit message: Start PCB layout
Parts:
- removed J3: JTAG-MAIN-XDS110, Connector_IDC:IDC-Header_2x10_P2.54mm_Vertical, symbol Daxxn_Connectors:JTAG-MAIN-XDS110
- removed SW3: SW_DIP_x08, Button_Switch_SMD:SW_DIP_SPSTx08_Slide_6.7x21.88mm_W6.73mm_P2.54mm_LowProfile_JPin, symbol Switch:SW_DIP_x08
- added C99 (x4): 100nF, Capacitor_SMD:C_0201_0603Metric, symbol Daxxn_Device:C
- added D31: ORANGE, LED_SMD:LED_0805_2012Metric, symbol Daxxn_Device:LED
- added D32: RED, LED_SMD:LED_0805_2012Metric, symbol Daxxn_Device:LED
- added J21: JTAG-14, Connector:Tag-Connect_TC2070-IDC-FP_2x07_P1.27mm_Vertical, symbol Daxxn_Connectors:JTAG-14
- added J22, J23: WKUP-UART, Daxxn_Connectors:JST_XH_B4B-XH-A_Vertical, symbol Connector_Generic:Conn_01x04
- added R120 (x6): 10K, Resistor_SMD:R_0402_1005Metric, symbol Daxxn_Device:R
- added R120: 1K, Resistor_SMD:R_0402_1005Metric, symbol Daxxn_Device:R
- added R120 (x2): 4.7K, Resistor_SMD:R_0402_1005Metric, symbol Daxxn_Device:R
- added R120: 500, Resistor_SMD:R_0402_1005Metric, symbol Daxxn_Device:R
- added S5: WARM RESET, Daxxn_Switches:TL3365AF180QG, symbol Daxxn_Buttons:GENERIC-SWITCH-2P
- added U42: SN74AVC4T245, Daxxn_Packages:UQFN-16-ZTA_DIO-M, symbol Daxxn_Logic:SN74AVC4T245RSVR
- added U44: 74LVC1G08GW, Daxxn_Packages:SOT-353_SC-70-5, symbol Daxxn_Logic:74LVC1G08GW
- R120: now not fitted
- renumbered D25 to D22, D26 to D23, D27 to D24, D28 to D25, D30 to D28, D31 to D33, JP3 to JP2, Q2 to Q7, S2 to S1, S3 to S2, S1 to S3, SW2 to SW5, TP13 to TP15, U43 to U41, U31 to U43, U44 to U45, U1 to U46, U29 to U47, U53 to U48, Y1 to Y3
Connections:
- net ~{PWR-RESET} is gone; now on net ~{TEST1-BTN}: R55.2, U46.11 (4Y)
- net ~{WARM-RESET} is gone; now on net ~{MCU-POR}: R120.1, R120.2, U45.4 (Y)
- net DVDD: now also C99.1, C99.1, R120.1, U42.3 (VCC_{A}), U44.5 (VCC)
- net GND: now also C99.2, C99.2, C99.2, C99.2, J21.13 (GND), J21.5 (GND), J22.4 (Pin_4), J23.4 (Pin_4), R120.1, R120.1, R120.2, R120.2, R120.2, S5.1, U42.10 (GND), U42.11 (GND), U44.3 (GND)
- net JTAG-EMU0: now also J21.9 (GPIOOUT0)
- net JTAG-EMU1: now also J21.6 (GPIOOUT1)
- net JTAG-TCK: now also J21.12 (TCK)
- net JTAG-TDI: now also J21.3 (TDI)
- net JTAG-TDIS: now also J21.4 (TDIS)
- net JTAG-TMS: now also J21.10 (SWDIO/TMS)
- net MCU-ERR: now also R120.1
- net VDD: now also C99.1, J22.1 (Pin_1), J23.1 (Pin_1), R120.1, R120.1, R120.2, R120.2, U42.2 (VCC_{B})
- net WKUP-UART-RX: now also U42.7 (1A2)
- net WKUP-UART-TX: now also U42.6 (1A1)
- net ~{JTAG-RESET}: now also J21.14 (~{RESET})
- net ~{JTAG-TRST}: now also J21.2 (~{TRST})
- net ~{MCU-RESET}-BTN: now also U44.2 (A); no longer U45.3 (B)
- net ~{PWR-RESET}-DEBOUNCE: no longer U46.12 (4A)
- net ~{TEST1-BTN}: no longer R55.2, U46.3 (1Y)
- net ~{TEST1-BTN}-DEBOUNCE: now also U46.12 (4A); no longer U46.2 (1A)
- net at R120.1: now also J21.11 (SWO/TDO)
- net at U41.1 (A): now also R120.2
- net at R120.2: now also J21.1 (VTREF)
- net RMII-REF-CLK: now reaches U4.A18 (EXT-REFCLK1)
- net MCU-UART-TX: now reaches U4.A5 (MCU-UART0-TXD)
- net MCU-UART-TX: now also U42.8 (2A1)
- net MCU-UART-RX: now reaches U4.B5 (MCU-UART0-RXD)
- net MCU-UART-RX: now also U42.9 (2A2)
- new net: R120.1, R120.2, U42.4 (1DIR), U42.5 (2DIR)
- new net: J23.2 (Pin_2), U42.13 (2B1)
- new net: J23.3 (Pin_3), U42.12 (2B2)
- new net: R120.2, U44.4 (Y), U45.3 (B)
- new net: D32.1 (K), R120.1
- new net: J22.2 (Pin_2), U42.15 (1B1)
- new net: J22.3 (Pin_3), U42.14 (1B2)
- new net: D31.1 (K), R120.1
- new net MCU-UART-EN: R120.1, R120.2, U42.1 (~{1OE}), U42.16 (~{2OE})
- new net OVERTEMP-IND: D31.2 (A)
- new net TEST-IND: D32.2 (A)
- new net ~{ANALOG-RESET}: U44.1 (B)
- new net ~{TEST2-BTN}: R55.2, U46.3 (1Y)
- new net ~{TEST2-BTN}-DEBOUNCE: C99.1, R120.2, S5.2, U46.2 (1A)
Other:
- note added: "19.2MHz"
- note added: "20MHz"
- note added: "24MHz"
- note added: "25MHz"
- note added: "26MHz"
- note added: "27MHz"
- note added: "ADDR"
- note added: "ARM/THUMB"
- note added: "BOOTMODE"
- note added: "BUS RESET"
- note added: "CLK SOURCE"
- note added: "CLKOUT"
- note added: "CONFIG"
- note added: "CORE VOLT"
- note added: "C_{SEL}"
- note added: "Ethernet"
- note added: "Ethernet RGMII"
- note added: "Ethernet RMII"
- note added: "Fs/raw"
- note added: "GPMC NAND"
- note added: "GPMC NOR"
- note added: "GROUP"
- note added: "I2C"
- note added: "ICLK"
- note added: "IF"
- note added: "LANE SWAP"
- note added: "LINK INFO"
- note added: "MMCSD"
- note added: "MODE"
- note added: "NO/DEV"
- note added: "NONE"
- note added: "No Boot / Dev Boot"
- note added: "OSPI"
- note added: "PORT"
- note added: "QSPI"
- note added: "READ CMD"
- note added: "READ MODE 1"
- note added: "READ MODE 2"
- note added: "SFPD"
- note added: "SPI"
- note added: "See Tech Reference Manual (Page: 2465)"
- note added: "Serial NAND"
- note added: "UART"
- note added: "USB"
- note added: "eMMC Boot"
- note added: "xSPI"
- note removed: "DESCRIPTION"
- note removed: "Engineering BOOT"
- note removed: "NAME"
- note removed: "PIN"
- note removed: "SD-CARD ON SDMMC1"
- note removed: "SERIAL NAND FLASH (QSPI)"
- note removed: "SERIAL NOR FLASH (QSPI)"
- note removed: "SLC NAND FLASH ON FMC"
- note removed: "UART / USB"
- note removed: "eMMC ON SDMMC2"
- moved on the sheet: C99, D16, D33, Q7, R120, R23, R55, TP14, TP15, U41, U4C

Commit message: (WIP) Still laying out PCB
Connections:
- no-connect marks 4 -> 20
Changed lines of the file:
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@@
   )
   (no_connect (at 189.23 182.88))
+  (no_connect (at 205.74 72.39))
+  (no_connect (at 254 44.45))
   (no_connect (at 13.97 267.97))
   (no_connect (at 39.37 63.5))
+  (no_connect (at 205.74 74.93))
+  (no_connect (at 254 69.85))
+  (no_connect (at 254 54.61))
+  (no_connect (at 254 72.39))
+  (no_connect (at 196.85 115.57))
+  (no_connect (at 254 64.77))
+  (no_connect (at 254 46.99))
   (no_connect (at 39.37 60.96))
+  (no_connect (at 254 52.07))
+  (no_connect (at 254 74.93))
+  (no_connect (at 254 59.69))
+  (no_connect (at 254 67.31))
+  (no_connect (at 196.85 118.11))
+  (no_connect (at 254 57.15))
+  (no_connect (at 196.85 102.87))
   (polyline (pts (xy 425.45 170.18) (xy 436.88 170.18))
     (stroke (width 0) (type default))

Commit message: Replacing motherboard and more - SAVE
Parts:
- renumbered C99 to C394, C143 to C395, C144 to C396, C143 to C397, C144 to C398, C99 to C399, C99 to C400, C99 to C401, C99 to C402, C99 to C403, C99 to C404, C99 to C405, C99 to C406, C99 to C407, C99 to C408, C231 to C409, C99 to C410, C99 to C411, C99 to C412, C99 to C413, C158 to C414, C158 to C415, C158 to C416, C158 to C417, D16 to D26, D16 to D27, D16 to D29, D16 to D30, R120 to R187, R120 to R188, R120 to R189, R120 to R190, R120 to R191, R120 to R192, R120 to R193, R120 to R194, R120 to R195, R120 to R196, R120 to R197, R120 to R198, R120 to R199, R120 to R200, R120 to R201, R120 to R202, R55 to R203, R55 to R204, R120 to R205, R120 to R206, R120 to R207, R120 to R208, R120 to R209, R120 to R210, R120 to R211, R120 to R212, R55 to R213, R120 to R214, R120 to R215, R120 to R216, R120 to R217, R55 to R218, R55 to R219, R55 to R220, R55 to R221, R120 to R222, R120 to R223, R55 to R224, R120 to R225, R120 to R226, R120 to R227, R55 to R228, R120 to R229, R120 to R230, R55 to R231, R23 to R232, R120 to R233, R23 to R234, R23 to R235, R23 to R236, R120 to R237, R102 to R238, U4 to U1, Y2 to Y4
