File: MotherBoard/BenchyMotherBoard-PCB/Ethernet.kicad_sch (KiCad schematic)
At the start: 62 parts, among them U13 KSZ9021RN, U36 74HCT2G08, U4 AM6254ATCGGAALW, U49 RJ45, U9 KSZ9021RN

Commit message: Add docs for benchy reloaded
Parts:
- R102: value 10K -> 1K
- R102: value 10K -> 3K
Changed lines of the file:
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@@
       (effects (font (size 1.27 1.27)) (justify left))
     )
-    (property "Value" "10K" (at 261.874 78.232 0)
+    (property "Value" "1K" (at 261.874 78.232 0)
       (effects (font (size 1.27 1.27)) (justify left))
     )
@@
       (effects (font (size 1.27 1.27)) (justify left) hide)
     )
+    (property "Schematic" "" (at 139.7 265.43 0)
+      (effects (font (size 1.27 1.27)) hide)
+    )
+    (property "SupplierPN" "" (at 139.7 265.43 0)
+      (effects (font (size 1.27 1.27)) hide)
+    )
     (pin "1")
     (pin "2")
@@
       (effects (font (size 1.27 1.27)) (justify left))
     )
-    (property "Value" "10K" (at 261.874 64.262 0)
+    (property "Value" "3K" (at 261.874 64.262 0)
       (effects (font (size 1.27 1.27)) (justify left))
     )
@@
       (effects (font (size 1.27 1.27)) (justify left))
     )
-    (property "Value" "10K" (at 261.874 149.352 0)
+    (property "Value" "3K" (at 261.874 149.352 0)
       (effects (font (size 1.27 1.27)) (justify left))
     )
@@
       (effects (font (size 1.27 1.27)) (justify left))
     )
-    (property "Value" "10K" (at 261.874 163.322 0)
+    (property "Value" "1K" (at 261.874 163.322 0)
       (effects (font (size 1.27 1.27)) (justify left))
     )
@@
       (effects (font (size 1.27 1.27)) (justify left))
     )
-    (property "Value" "10K" (at 267.716 64.262 0)
+    (property "Value" "3K" (at 267.716 64.262 0)
       (effects (font (size 1.27 1.27)) (justify left))
     )
@@
       (effects (font (size 1.27 1.27)) (justify left))
     )
-    (property "Value" "10K" (at 267.716 149.352 0)
+    (property "Value" "3K" (at 267.716 149.352 0)
       (effects (font (size 1.27 1.27)) (justify left))
     )
@@
       (effects (font (size 1.27 1.27)) (justify left))
     )
-    (property "Value" "10K" (at 267.716 163.322 0)
+    (property "Value" "1K" (at 267.716 163.322 0)
       (effects (font (size 1.27 1.27)) (justify left))
     )
@@
       (effects (font (size 1.27 1.27)) (justify left))
     )
-    (property "Value" "10K" (at 267.716 78.232 0)
+    (property "Value" "1K" (at 267.716 78.232 0)
       (effects (font (size 1.27 1.27)) (justify left))
     )

Commit message: Replacing motherboard and more - SAVE
Parts:
- renumbered C158 to C418, C158 to C419, C158 to C420, C158 to C421, C158 to C422, C158 to C423, C158 to C424, C158 to C425, C158 to C426, C158 to C427, C158 to C428, C158 to C429, R23 to R239, R23 to R240, R23 to R241, R23 to R242, R102 to R243, R23 to R244, R102 to R245, R102 to R246, R102 to R247, R102 to R248, R102 to R249, R102 to R250, R102 to R251, R102 to R252, R102 to R253, R102 to R254, R102 to R255, R102 to R256, R102 to R257, R102 to R258, R102 to R259, R23 to R260, R102 to R261, R102 to R262, R102 to R263, R102 to R264, R102 to R265, R102 to R266, R102 to R267, R102 to R268, R102 to R269, R102 to R270, R102 to R271, R102 to R272, R102 to R273, R102 to R274, R102 to R275, R102 to R276, R102 to R277, R102 to R278, R102 to R279, R102 to R280, U4 to U1, U36 to U50, U36 to U51
