File: MotherBoard/BenchyMotherBoard-PCB/comms.kicad_sch (KiCad schematic)
At the start: 21 parts, among them J18 COMMS-PWR, J19 COMMS-ELOAD, J20 COMMS-SWITCHER, J21 RELAYS-CONN, J22 COMMS-LOGIC, U33 TCAN1044

Commit message: (WIP) Almost done with schematic
Parts:
- R148, R149: footprint (none) -> Resistor_SMD:R_0402_1005Metric
- R150, R151, R152, R153, R154, R155: value 60 -> 22; footprint (none) -> Resistor_SMD:R_0402_1005Metric
Changed lines of the file:
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@@
+    )
+  )
+  (global_label "RELAY-BUS[1..6]" (shape input) (at 27.94 44.45 180) (fields_autoplaced)
+    (effects (font (size 1.016 1.016)) (justify right))
+    (property "Intersheetrefs" "${INTERSHEET_REFS}" (at 12.5527 44.45 0)
+      (effects (font (size 1.27 1.27)) (justify right))
     )
   )
@@
       (effects (font (size 1.27 1.27)) (justify right))
     )
-  )
-  (hierarchical_label "RELAY-BUS[1..6]" (shape input) (at 27.94 44.45 180) (fields_autoplaced)
-    (effects (font (size 1.016 1.016)) (justify right))
   )
   (symbol (lib_id "power:GND") (at 95.25 40.64 0) (unit 1)
@@
       (effects (font (size 1.27 1.27)) (justify left))
     )
-    (property "Value" "60" (at 78.994 30.734 0)
-      (effects (font (size 1.27 1.27)) (justify left))
-    )
-    (property "Footprint" "" (at 80.01 31.75 0)
+    (property "Value" "22" (at 78.994 30.734 0)
+      (effects (font (size 1.27 1.27)) (justify left))
+    )
+    (property "Footprint" "Resistor_SMD:R_0402_1005Metric" (at 80.01 31.75 0)
       (effects (font (size 1.27 1.27)) hide)
     )
@@
       (effects (font (size 1.27 1.27)) (justify left))
     )
-    (property "Value" "60" (at 86.614 25.654 0)
-      (effects (font (size 1.27 1.27)) (justify left))
-    )
-    (property "Footprint" "" (at 87.63 26.67 0)
+    (property "Value" "22" (at 86.614 25.654 0)
+      (effects (font (size 1.27 1.27)) (justify left))
+    )
+    (property "Footprint" "Resistor_SMD:R_0402_1005Metric" (at 87.63 26.67 0)
       (effects (font (size 1.27 1.27)) hide)
     )
@@
       (effects (font (size 1.27 1.27)) (justify left))
     )
-    (property "Value" "60" (at 75.184 33.274 0)
-      (effects (font (size 1.27 1.27)) (justify left))
-    )
-    (property "Footprint" "" (at 76.2 34.29 0)
+    (property "Value" "22" (at 75.184 33.274 0)
+      (effects (font (size 1.27 1.27)) (justify left))
+    )
+    (property "Footprint" "Resistor_SMD:R_0402_1005Metric" (at 76.2 34.29 0)
       (effects (font (size 1.27 1.27)) hide)
     )
@@
       (effects (font (size 1.27 1.27)) (justify left))
     )
-    (property "Value" "60" (at 71.374 35.814 0)
-      (effects (font (size 1.27 1.27)) (justify left))
-    )
-    (property "Footprint" "" (at 72.39 36.83 0)
+    (property "Value" "22" (at 71.374 35.814 0)
+      (effects (font (size 1.27 1.27)) (justify left))
+    )
+    (property "Footprint" "Resistor_SMD:R_0402_1005Metric" (at 72.39 36.83 0)
       (effects (font (size 1.27 1.27)) hide)
     )
@@
       (effects (font (size 1.27 1.27)) (justify left))
     )
-    (property "Footprint" "" (at 55.88 85.09 0)
+    (property "Footprint" "Resistor_SMD:R_0402_1005Metric" (at 55.88 85.09 0)
       (effects (font (size 1.27 1.27)) hide)
     )
@@
       (effects (font (size 1.27 1.27)) (justify left))
     )
-    (property "Value" "60" (at 82.804 28.194 0)
-      (effects (font (size 1.27 1.27)) (justify left))
-    )
-    (property "Footprint" "" (at 83.82 29.21 0)
+    (property "Value" "22" (at 82.804 28.194 0)
+      (effects (font (size 1.27 1.27)) (justify left))
+    )
+    (property "Footprint" "Resistor_SMD:R_0402_1005Metric" (at 83.82 29.21 0)
       (effects (font (size 1.27 1.27)) hide)
     )
@@
       (effects (font (size 1.27 1.27)) (justify left))
     )
-    (property "Footprint" "" (at 55.88 92.71 0)
+    (property "Footprint" "Resistor_SMD:R_0402_1005Metric" (at 55.88 92.71 0)
       (effects (font (size 1.27 1.27)) hide)
     )
@@
       (effects (font (size 1.27 1.27)) (justify left))
     )
-    (property "Value" "60" (at 90.424 23.114 0)
-      (effects (font (size 1.27 1.27)) (justify left))
-    )
-    (property "Footprint" "" (at 91.44 24.13 0)
-      (effects (font (size 1.27 1.27)) hide)
-    )
+    (property "Value" "22" (at 90.424 23.114 0)
+      (effects (font (size 1.27 1.27)) (justify left))
+    )
+    (property "Footprint" "Resistor_SMD:R_0402_1005Metric" (at 91.44 24.13 0)
+      (effects (font (size 1.27 1.27)) hide)
+    )

Commit message: Start PCB layout
Parts:
- renumbered C278 to C373, C178 to C374, C179 to C375, C180 to C376, C181 to C377, C279 to C378, D29 to D21, J21 to J14, J18 to J15, J19 to J16, J20 to J17, J22 to J18, R150 to R165, R151 to R166, R152 to R167, R153 to R168, R154 to R169, R155 to R170, R148 to R171, R149 to R172, U33 to U36
