File: MotherBoard/BenchyMotherBoard-PCB/usb.kicad_sch (KiCad schematic)
At the start: 112 parts, among them J10 USB3_B, J11 USB3-PORT2, J12 USB3-PORT3, J13 USB3-PORT4, J14 USB3-PORT5, J15 USB-INTERNAL-PORT1, J17 USB-INTERNAL-PORT2, J9 USB3-PORT1, U10 USB7206C, U12 UCS2114, U13 UCS2114, U14 UCS2114, U17 24LC08, U18 USB2412, U4 AM6254ATCGGAALW, U54 AP2156SG, U55 74LVC1G08GW, Y3 24MHz, Y4 25MHz

Commit message: Start PCB layout
Parts:
- removed JP2: WP-JMP, Connector_PinSocket_2.54mm:PinSocket_1x03_P2.54mm_Vertical, symbol Jumper:Jumper_3_Bridged12
- removed R108, R109: 2.2K, Resistor_SMD:R_0402_1005Metric, symbol Daxxn_Device:R
- removed R259: 10K, Resistor_SMD:R_0402_1005Metric, symbol Daxxn_Device:R
- removed U17: 24LC08, Package_SO:SOIC-8_3.9x4.9mm_P1.27mm, symbol Memory_EEPROM:24LC08
- added C362, C369: 100nF, Capacitor_SMD:C_0402_1005Metric, symbol Daxxn_Device:C
- added R149: 100K, Resistor_SMD:R_0402_1005Metric, symbol Daxxn_Device:R
- added R154, R157, R162: 10K, Resistor_SMD:R_0402_1005Metric, symbol Daxxn_Device:R
- added R159: 200K, Resistor_SMD:R_0402_1005Metric, symbol Daxxn_Device:R
- added U32: MIC803-29D3VM3, Daxxn_Packages:SOT-23-3, symbol Daxxn_IC:MIC803-29D3VM3
- added U33: W25Q16JVUXIQ, Daxxn_Packages:USON-8_2x3mm_P0.5mm, symbol Daxxn_Memory:W25Q16JVUXIQ
- added U34: 74HCT2G08, Daxxn_Packages:WSON-6_1.5x1.5mm_P0.5mm, symbol Daxxn_Logic:SN74LVC1G11DRYR
- C372: renamed from C436; now not fitted
- R52: now not fitted
- renumbered C441 to C322, C443 to C323, C145 to C324, C146 to C325, C431 to C326, C444 to C327, C152 to C328, C153 to C329, C430 to C330, C147 to C331, C440 to C332, C442 to C333, C148 to C334, C149 to C335, C432 to C336, C445 to C337, C154 to C338, C155 to C339, C429 to C340, C439 to C341, C446 to C342, C150 to C343, C151 to C344, C433 to C345, C168 to C346, C169 to C347, C422 to C348, C423 to C349, C421 to C350, C165 to C351, C166 to C352, C167 to C353, C162 to C354, C163 to C355, C164 to C356, C170 to C357, C171 to C358, C424 to C359, C425 to C360, C426 to C361, C174 to C363, C175 to C364, C176 to C365, C427 to C366, C428 to C367, C177 to C368, C434 to C370, C435 to C371, D1 to D13, D4 to D14, D2 to D15, D5 to D16, D3 to D17, D6 to D18, D7 to D19, D8 to D20, J14 to J10, J12 to J11, J15 to J12, J17 to J13, J9 to J6, J13 to J7, J10 to J8, J11 to J9, R91 to R128, R92 to R129, R95 to R130, R96 to R131, R97 to R132, R98 to R133, R99 to R134, R100 to R135, R93 to R136, R105 to R137, R106 to R138, R107 to R139, R56 to R140, R110 to R141, R94 to R143, R112 to R144, R117 to R145, R111 to R146, R113 to R147, R114 to R148, R115 to R151, R116 to R152, R265 to R155, R118 to R160, R264 to R163, U10 to U18, U12 to U27, U13 to U28, U14 to U29, U54 to U30, U18 to U31, U55 to U35, Y3 to Y1, Y4 to Y2
Connections:
- net GND: now also C362.1, C369.1, R157.2, R159.1, R162.2, U32.1 (GND), U33.4 (GND), U34.2 (GND); no longer R145.1
- net VDD: now also R145.2, C362.2, C369.2, R149.1, R154.1, U32.3 (VCC), U33.8 (VDD), U34.5 (VCC)
- net ~{RESET-STATUS}: now also U34.6 (C)
- net ~{USB-RESET}: no longer R146.1, U18.1 (~{RESET})
- net USB-PERIPH-DRV: now reaches R155.1, U4.F18 (USB1-DRVVBUS)
- net USB-PERIPH-DRV: now also R154.2, R157.1
- net at U18.70 (SPI-D0): now also U33.5 (IO0); no longer R160.2
- net at U18.69 (~{SPI_CE}): now also R145.1, U33.1 (~{CS}); no longer R145.2
- net at U18.68 (SPI-SCLK): now also R160.2, U33.6 (CLK)
- net at U18.71 (SPI-D1): now also R159.2, U33.2 (IO1)
- net at U18.72 (SPI-D2): now also U33.3 (IO2)
- net at U18.73 (SPI-D3): now also U33.7 (IO3)
- net I2C-SYS-SCL renamed I2C-MAIN-SCL
- net I2C-SYS-SDA renamed I2C-MAIN-SDA
- net USB-HUB-INU-EN renamed USB-PERIPH-EN
- net USB-INU-D+ renamed USB-PERIPH-D+
- net USB-INU-D- renamed USB-PERIPH-D-
- net USB-INU-VBUS renamed USB-PERIPH-VBUS
- new net ~{RESET-USB-HUB}: U34.1 (A)
- new net ~{USB-HUB-RESET}: R146.1, R162.1, U18.1 (~{RESET}), U34.4 (Y)
- new net ~{USB-HUB-SUP-RESET}: R149.2, U32.2 (~{RESET}), U34.3 (B)
- no-connect marks 33 -> 29
Other:
- note removed: "DISPLAY"
- moved on the sheet: C322, C332, C341, C363, C368, C370, C371, R130, R131, R132, R133, R134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

Commit message: Fix power net names and increase PCB size
Parts:
- C347, C360: footprint Capacitor_SMD:C_1210_3225Metric -> Capacitor_SMD:C_0805_2012Metric
Changed lines of the file:
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@@
       (effects (font (size 1.27 1.27)) (justify left))
     )
-    (property "Footprint" "Capacitor_SMD:C_1210_3225Metric" (at 325.12 212.09 0)
+    (property "Footprint" "Capacitor_SMD:C_0805_2012Metric" (at 325.12 212.09 0)
       (effects (font (size 1.27 1.27)) hide)
     )
     (property "Datasheet" "~" (at 325.12 212.09 0)
+      (effects (font (size 1.27 1.27)) hide)
+    )
+    (property "Schematic" "" (at 325.12 212.09 0)
+      (effects (font (size 1.27 1.27)) hide)
+    )
+    (property "PartNumber" "" (at 325.12 212.09 0)
+      (effects (font (size 1.27 1.27)))
+    )
+    (property "SupplierPN" "" (at 325.12 212.09 0)
       (effects (font (size 1.27 1.27)) hide)
     )
@@
       (effects (font (size 1.27 1.27)) (justify left))
     )
-    (property "Footprint" "Capacitor_SMD:C_1210_3225Metric" (at 334.01 151.13 0)
+    (property "Footprint" "Capacitor_SMD:C_0805_2012Metric" (at 334.01 151.13 0)
       (effects (font (size 1.27 1.27)) hide)
     )
@@
       (effects (font (size 1.27 1.27)) hide)
     )
+    (property "Schematic" "" (at 334.01 151.13 0)
+      (effects (font (size 1.27 1.27)) hide)
+    )
+    (property "PartNumber" "" (at 334.01 151.13 0)
+      (effects (font (size 1.27 1.27)))
+    )
+    (property "SupplierPN" "" (at 334.01 151.13 0)
+      (effects (font (size 1.27 1.27)) hide)
+    )

Commit message: Replacing motherboard and more - SAVE
Parts:
- renumbered R23 to R142, R23 to R150, R23 to R153, R52 to R156, R52 to R158, R52 to R161, R52 to R164, U4 to U1
