File: FrontPanel/BenchyFrontPanel/BenchyFrontPanel.kicad_pcb (KiCad board)
At the start: 2 copper layers, 400 x 50 mm, 91 parts, among them J1 FRONT PANEL, SW1 TL3215AF160GQ, SW10 TL3215AF160BQ, SW11 TL3215AF160BQ, SW12 TL3215AF160BQ, SW2 TL3215AF160YQ, SW3 TL3215AF160RQ, SW4 228CMVARGBFR, SW5 TL3215AF160GQ, SW6 TL3215AF160BQ, SW7 B3W-9000-RG2N, SW8 TL3215AF160BQ, SW9 TL3215AF160BQ, U1 MCP23S08-E/ML, U2 SN74HCS125BQAR, U3 SN74HCS365PWR, U4 MCP23S08-E/ML, U5 SN74LVC1G17DCKR, U6 STP16CP05MTR, U7 SN74HCS365PWR

Commit message: Schematic capture mostly complete. Starting PCB layout
Parts:
- removed S2, S4, S5: ILS-TB180-60, Daxxn_Controls_Buttons:ILS-TB
- removed S3: ILS-TB250-10, Daxxn_Controls_Buttons:ILS-TB
- removed TP1: TP-VCC-STBY, TestPoint:TestPoint_Pad_D2.0mm
- removed TP2: TP-VDD-SYS, TestPoint:TestPoint_Pad_D2.0mm
- added C25: 100n, Daxxn_Standard_Capacitors:CAP_0402, B.Cu at (241.2, 65.6)
- added C26: 100n, Daxxn_Standard_Capacitors:CAP_0402, B.Cu at (241.2, 63.6)
- added C27: 100n, Daxxn_Standard_Capacitors:CAP_0402, B.Cu at (241.2, 61.6)
- added C28: 100n, Daxxn_Standard_Capacitors:CAP_0402, B.Cu at (241.2, 59.6)
- added C29: 100n, Daxxn_Standard_Capacitors:CAP_0402, B.Cu at (241.2, 57.6)
- added C30: 100n, Daxxn_Standard_Capacitors:CAP_0402, B.Cu at (285.9, 59.8)
- added C31: 100n, Daxxn_Standard_Capacitors:CAP_0402, B.Cu at (285.9, 57.8)
- added C32: 100n, Daxxn_Standard_Capacitors:CAP_0402, B.Cu at (285.9, 55.8)
- added C33: 100n, Daxxn_Standard_Capacitors:CAP_0402, B.Cu at (285.9, 53.9)
- added C34: 100n, Daxxn_Standard_Capacitors:CAP_0402, B.Cu at (285.9, 51.9)
- added C35: 100n, Daxxn_Standard_Capacitors:CAP_0402, B.Cu at (285.9, 49.9)
- added C36: 100n, Daxxn_Standard_Capacitors:CAP_0402, B.Cu at (288.8, 59.8)
- added C37: 100n, Daxxn_Standard_Capacitors:CAP_0402, B.Cu at (288.8, 57.8)
- added C38: 100n, Daxxn_Standard_Capacitors:CAP_0402, B.Cu at (288.8, 55.8)
- added C39: 100n, Daxxn_Standard_Capacitors:CAP_0402, B.Cu at (288.8, 53.9)
- added C40: 100n, Daxxn_Standard_Capacitors:CAP_0402, B.Cu at (288.8, 51.9)
- added C41: 100n, Daxxn_Standard_Capacitors:CAP_0402, B.Cu at (288.8, 49.9)
- added C42: 100n, Daxxn_Standard_Capacitors:CAP_0402, B.Cu at (286.1, 68.1)
- added D10: CZ5-0603-RED, Daxxn_LEDs:LED_0603_1608Metric, F.Cu at (102.9, 64.5)
- added D11: CZ1-0603-BLUE, Daxxn_LEDs:LED_0603_1608Metric, F.Cu at (158.9, 72.5)
- added D12: CZ3-0603-ORANGE, Daxxn_LEDs:LED_0603_1608Metric, F.Cu at (31.5, 58.5)
- added D13: CZ2-0603-GREEN, Daxxn_LEDs:LED_0603_1608Metric, F.Cu at (64.9, 62.5)
- added D14: CZ2-0603-GREEN, Daxxn_LEDs:LED_0603_1608Metric, F.Cu at (121.9, 62.5)
- added D15: CZ1-0603-BLUE, Daxxn_LEDs:LED_0603_1608Metric, F.Cu at (158.9, 74.5)
- added D16: CZ5-0603-RED, Daxxn_LEDs:LED_0603_1608Metric, F.Cu at (64.9, 64.5)
- added D17: CZ5-0603-RED, Daxxn_LEDs:LED_0603_1608Metric, F.Cu at (121.9, 64.5)
- added D18: CZ1-0603-BLUE, Daxxn_LEDs:LED_0603_1608Metric, F.Cu at (158.9, 76.5)
- added D19: CZ1-0603-BLUE, Daxxn_LEDs:LED_0603_1608Metric, F.Cu at (158.9, 78.5)
- added D20: CZ3-0603-ORANGE, Daxxn_LEDs:LED_0603_1608Metric, F.Cu at (31.5, 53.5)
- added D21: CZ2-0603-GREEN, Daxxn_LEDs:LED_0603_1608Metric, F.Cu at (83.9, 62.5)
- added D22: CZ1-0603-BLUE, Daxxn_LEDs:LED_0603_1608Metric, F.Cu at (158.9, 80.5)
- added D23: CZ5-0603-RED, Daxxn_LEDs:LED_0603_1608Metric, F.Cu at (83.9, 64.5)
- added D24: CZ1-0603-BLUE, Daxxn_LEDs:LED_0603_1608Metric, F.Cu at (158.9, 82.5)
- added D25: CZ3-0603-ORANGE, Daxxn_LEDs:LED_0603_1608Metric, F.Cu at (31.5, 43.5)
- added D26: CZ3-0603-ORANGE, Daxxn_LEDs:LED_0603_1608Metric, F.Cu at (31.5, 63.5)
- added D27: CZ8-0603-YLW-GREEN, Daxxn_LEDs:LED_0603_1608Metric, F.Cu at (50.0, 89.0)
- added D28: CZ2-0603-GREEN, Daxxn_LEDs:LED_0603_1608Metric, F.Cu at (50.0, 86.0)
- added D29: CZ8-0603-YLW-GREEN, Daxxn_LEDs:LED_0603_1608Metric, F.Cu at (60.0, 89.0)
- added D30: CZ2-0603-GREEN, Daxxn_LEDs:LED_0603_1608Metric, F.Cu at (60.0, 86.0)
- added D5: CZ2-0603-GREEN, Daxxn_LEDs:LED_0603_1608Metric, F.Cu at (45.9, 62.5)
- added D6: CZ2-0603-GREEN, Daxxn_LEDs:LED_0603_1608Metric, F.Cu at (102.9, 62.5)
- added D7: CZ1-0603-BLUE, Daxxn_LEDs:LED_0603_1608Metric, F.Cu at (158.9, 68.5)
- added D8: CZ1-0603-BLUE, Daxxn_LEDs:LED_0603_1608Metric, F.Cu at (158.9, 70.5)
- added D9: CZ5-0603-RED, Daxxn_LEDs:LED_0603_1608Metric, F.Cu at (45.9, 64.5)
- added EN1: PEC11R-4220F-S0024, Daxxn_Controls_Encoders:PEC11R, F.Cu at (29.0, 74.0)
- added H10: M2.5, MountingHole:MountingHole_2.7mm_M2.5_ISO7380_Pad, F.Cu at (159.0, 62.0)
- added H11: M2.5, MountingHole:MountingHole_2.7mm_M2.5_ISO7380_Pad, F.Cu at (179.0, 62.0)
- added H9: M2.5, MountingHole:MountingHole_2.7mm_M2.5_ISO7380_Pad, F.Cu at (159.0, 87.0)
- added J2: 046841045100846+, Daxxn_Connectors_FFC:046841045100846+, B.Cu at (202.0, 78.2)
- added R26: 1K3, Daxxn_Standard_Resistors:RES_0402, B.Cu at (247.0, 49.6)
- added R27: 100K, Daxxn_Standard_Resistors:RES_0402, B.Cu at (249.9, 69.5)
- added R28: 2K2, Daxxn_Standard_Resistors:RES_0402, B.Cu at (249.9, 67.5)
- added R29: 2K2, Daxxn_Standard_Resistors:RES_0402, B.Cu at (249.9, 65.6)
- added R30: 2K2, Daxxn_Standard_Resistors:RES_0402, B.Cu at (249.9, 63.6)
- added R31: 100K, Daxxn_Standard_Resistors:RES_0402, B.Cu at (249.9, 61.6)
- added R32: 100K, Daxxn_Standard_Resistors:RES_0402, B.Cu at (249.9, 59.6)
- added R33: 10K, Daxxn_Standard_Resistors:RES_0402, B.Cu at (249.9, 57.6)
- added R34: 10K, Daxxn_Standard_Resistors:RES_0402, B.Cu at (249.9, 55.6)
- added R35: 10K, Daxxn_Standard_Resistors:RES_0402, B.Cu at (249.9, 53.6)
- added R36: 100K, Daxxn_Standard_Resistors:RES_0402, B.Cu at (249.9, 51.6)
- added R37: 100K, Daxxn_Standard_Resistors:RES_0402, B.Cu at (291.7, 59.8)
- added R38: 100K, Daxxn_Standard_Resistors:RES_0402, B.Cu at (291.7, 57.8)
- added R39: 100K, Daxxn_Standard_Resistors:RES_0402, B.Cu at (291.7, 55.8)
- added R40: 10K, Daxxn_Standard_Resistors:RES_0402, B.Cu at (291.7, 53.9)
- added R41: 10K, Daxxn_Standard_Resistors:RES_0402, B.Cu at (291.7, 51.9)
- added R42: 10K, Daxxn_Standard_Resistors:RES_0402, B.Cu at (291.7, 49.9)
- added R43: 10K, Daxxn_Standard_Resistors:RES_0402, B.Cu at (294.6, 59.8)
- added R44: 10K, Daxxn_Standard_Resistors:RES_0402, B.Cu at (294.6, 57.8)
- added R45: 10K, Daxxn_Standard_Resistors:RES_0402, B.Cu at (294.6, 55.8)
- added R46: 10K, Daxxn_Standard_Resistors:RES_0402, B.Cu at (294.6, 53.9)
- added R47: 10K, Daxxn_Standard_Resistors:RES_0402, B.Cu at (294.6, 51.9)
- added R48: 100K, Daxxn_Standard_Resistors:RES_0402, B.Cu at (286.1, 66.1)
- added SW13: TL3215AF160GQ, Daxxn_Controls_Buttons:TL3215A, F.Cu at (87.5, 41.5)
- added SW14: TL3365AF180QG, Daxxn_Controls_Buttons:TL3365AF180QG, F.Cu at (127.0, 28.5)
- added SW15: TL3365AF180QG, Daxxn_Controls_Buttons:TL3365AF180QG, F.Cu at (127.0, 37.5)
- added SW16: 228CMVARGBFR, Daxxn_Controls_Buttons:228C, F.Cu at (50.0, 32.0)
- added SW17: TL3365AF180QG, Daxxn_Controls_Buttons:TL3365AF180QG, F.Cu at (22.5, 60.0)
- added SW18: TL3365AF180QG, Daxxn_Controls_Buttons:TL3365AF180QG, F.Cu at (115.0, 46.5)
- added SW19: TL3365AF180QG, Daxxn_Controls_Buttons:TL3365AF180QG, F.Cu at (115.0, 37.5)
- added SW20: TL3365AF180QG, Daxxn_Controls_Buttons:TL3365AF180QG, F.Cu at (115.0, 28.5)
- added SW21: TL3365AF180QG, Daxxn_Controls_Buttons:TL3365AF180QG, F.Cu at (32.0, 87.5)
- added TP5: TP-VCC-USB, TestPoint:TestPoint_Pad_D2.0mm, F.Cu at (28.5, 53.5)
- added TP6: TP-12V, TestPoint:TestPoint_Pad_D2.0mm, F.Cu at (28.5, 43.5)
- added TP7: TP-VDD, TestPoint:TestPoint_Pad_D2.0mm, F.Cu at (28.5, 63.5)
- added U10: SN74HCS365PWR, Daxxn_Packages:TSSOP-16_4.4x5mm_P0.65mm, B.Cu at (277.8, 52.5)
- added U11: SN74HCS365PWR, Daxxn_Packages:TSSOP-16_4.4x5mm_P0.65mm, B.Cu at (277.8, 59.1)
- added U12: SN74HCS125BQAR, Daxxn_Packages:WQFN-14_B3x2.5mm_P0.5mm, B.Cu at (266.5, 60.9)
- added U8: MCP23S08-E/ML, Daxxn_Packages:QFN-20-1EP_4x4mm_P0.5mm_EP2.7x2.7mm, B.Cu at (226.9, 54.7)
- added U9: SN74HCS365PWR, Daxxn_Packages:TSSOP-16_4.4x5mm_P0.65mm, B.Cu at (161.0, 54.0)
- C1, C10, C11, C12, C13, C14, C15, C16, C17, C18, C19, C20, C21, C22, C23, C24, C4, C5, C6, C7, C8, C9, R1, R11, R15, U4: moved to B.Cu
- C2, C3: value 100n -> 10n; moved to B.Cu
- D2: value CZ3-0603-ORANGE -> CZ2-0603-GREEN
- D3: value CZ3-0603-ORANGE -> CZ1-0603-BLUE
- J1: value FRONT PANEL -> RIGOL-LA-PROBE; footprint Connector_PinHeader_2.54mm:PinHeader_2x12_P2.54mm_Vertical_SMD -> Daxxn_Connectors_PCI:10018784-10200TLF
- R10: value 10K -> 2K94; moved to B.Cu
- R12: value 2K2 -> 1K3; moved to B.Cu
- R13: value 2K2 -> 2K94; moved to B.Cu
- R14: value 2K2 -> 100K; moved to B.Cu
- R16, R18, R19, R20, R21, R9: value 10K -> 100K; moved to B.Cu
- R17: value 4K7 -> 1K3; moved to B.Cu
- R2, R5, R6: value 100K -> 10K; moved to B.Cu
- R22, R24: value 2K94 -> 1K3; moved to B.Cu
- R23: value 1K3 -> 100K; moved to B.Cu
- R25: value 10K -> 1K3; moved to B.Cu
- R3, R4: value 100K -> 1K3; moved to B.Cu
- R7, R8: value 10K -> 4K7; moved to B.Cu
- S1: value B3F-4050 -> BOJACK-BTN-6X6X5-2; footprint Daxxn_Controls_Buttons:B3F-4050 -> Daxxn_Controls_Buttons:BOJACK-BTN-6x6x5
- SW1: value TL3215AF160GQ -> TL3215AF160RQ
- SW11: value TL3215AF160BQ -> TL3215AF160YQ
- SW2: value TL3215AF160YQ -> B3W-9000-RG2N; footprint Daxxn_Controls_Buttons:TL3215A -> Daxxn_Controls_Buttons:B3W-9000
- SW3: value TL3215AF160RQ -> TL3215AF160BQ
- SW4: value 228CMVARGBFR -> TL3215AF160BQ; footprint Daxxn_Controls_Buttons:228C -> Daxxn_Controls_Buttons:TL3215A
- SW5: value TL3215AF160GQ -> TL3365AF180QG; footprint Daxxn_Controls_Buttons:TL3215A -> Daxxn_Controls_Buttons:TL3365AF180QG
- SW6: value TL3215AF160BQ -> TL3215AF160GQ
- SW7: value B3W-9000-RG2N -> TL3215AF160BQ; footprint Daxxn_Controls_Buttons:B3W-9000 -> Daxxn_Controls_Buttons:TL3215A
- TP3: value TP-VCC-USB -> TP-VCC-STBY
- TP4: value TP-12V -> TP-VDD-SYS
- U1: value MCP23S08-E/ML -> 74LVC3G17GS,115; footprint Daxxn_Packages:QFN-20-1EP_4x4mm_P0.5mm_EP2.7x2.7mm -> Daxxn_Packages:X2SON-8_1.4x1mm_P0.35mm; moved to B.Cu
- U2: value SN74HCS125BQAR -> STP16CP05MTR; footprint Daxxn_Packages:WQFN-14_B3x2.5mm_P0.5mm -> Daxxn_Packages:SOIC-24W_7.5x15.4mm_P1.27mm; moved to B.Cu
- U3: value SN74HCS365PWR -> STP16CP05MTR; footprint Daxxn_Packages:TSSOP-16_4.4x5mm_P0.65mm -> Daxxn_Packages:SOIC-24W_7.5x15.4mm_P1.27mm; moved to B.Cu
- U5: value SN74LVC1G17DCKR -> MCP23S08-E/ML; footprint Daxxn_Packages:SOT-353_SC-70-5 -> Daxxn_Packages:QFN-20-1EP_4x4mm_P0.5mm_EP2.7x2.7mm; moved to B.Cu
- U6: value STP16CP05MTR -> TC7PZ17FU,LJ(CT; footprint Daxxn_Packages:SOIC-24W_7.5x15.4mm_P1.27mm -> Daxxn_Packages:SOT-363_SC-70-6; moved to B.Cu
- U7: value SN74HCS365PWR -> TC7PZ17FU,LJ(CT; footprint Daxxn_Packages:TSSOP-16_4.4x5mm_P0.65mm -> Daxxn_Packages:SOT-363_SC-70-6; moved to B.Cu
- moved H3 488.4 mm to (417.0, 87.0)
- moved H4 486.3 mm to (417.0, 43.0)
- moved U6 359.3 mm to (257.1, 59.0)
- moved U4 356.2 mm to (268.0, 52.7)
- moved U5 352.9 mm to (257.5, 51.5)
- moved U1 346.7 mm to (258.4, 67.5)
- moved U7 314.0 mm to (226.9, 61.4)
- moved C1 309.7 mm to (235.3, 69.5)
- moved R5 309.7 mm to (244.1, 69.5)
- moved R16 309.4 mm to (247.0, 69.5)
- moved C12 309.3 mm to (238.3, 69.5)
- moved R17 309.3 mm to (247.0, 67.5)
- moved R6 309.1 mm to (244.1, 67.5)
- moved C2 308.9 mm to (235.3, 67.5)
- moved C23 308.9 mm to (241.2, 69.5)
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Connections:
- C1 pad 1: VDD -> VDD-STBY
- C10 pad 1: /NAV-BACK-SW-IN -> /MB-CFG-SW3-IN
- C11 pad 1: Net-(U2C-3A) -> VDD-STBY
- C12 pad 1: VDD-STBY -> /MB-SYS-PWR-SW-IN
- C13 pad 1: Net-(U2D-4A) -> /MB-SOC-PWR-SW-IN
- C14 pad 1: /FP-SOC-PWR-SW-IN -> /MB-SOC-RST-SW-IN
- C15 pad 1: VDD -> /MB-SOC-SLP-SW-IN
- C16 pad 1: Net-(U7A-A1) -> /MB-CFG-SW4-IN
- C17 pad 1: VDD -> /MB-CFG-SW5-IN
- C18 pad 1: Net-(U7B-A2) -> VDD-STBY
- C19 pad 1: Net-(U7C-A3) -> VDD-STBY
- C2 pad 1: Net-(U2A-1A) -> GND
- C2 pad 2: GND -> Net-(C2-Pad2)
- C20 pad 1: Net-(U7E-A5) -> VDD-STBY
- C21 pad 1: Net-(U7D-A4) -> /MB-CFG-SW6-IN
- C22 pad 1: Net-(U7F-A6) -> /NAV-UP-SW-RAW
- C23 pad 1: VDD -> Net-(U10E-A5)
- C24 pad 1: VDD -> Net-(U10F-A6)
- C3 pad 1: /NAV-UP-SW-RAW -> Net-(C3-Pad1)
- C4 pad 1: /NAV-DOWN-SW-RAW -> VDD-STBY
- C5 pad 1: /NAV-PUSH-SW-RAW -> VDD-STBY
- C6 pad 1: /NAV-LEFT-SW-RAW -> /ENC-SW-IN
- C7 pad 1: /NAV-RIGHT-SW-RAW -> /MB-CFG-SW1-IN
- C8 pad 1: Net-(U2B-2A) -> VDD-STBY
- C9 pad 1: VDD -> /MB-CFG-SW2-IN
- D1 pad 2: VCC-STBY -> /MB-SOC-USB-HS-IND
- D2 pad 2: VDD-SYS -> /MB-SOC-USB-SUSP-IND
- D3 pad 2: VCC-USB -> VDD-STBY
- D4 pad 2: +12V -> VCC-STBY
- R1 pad 1: VDD -> /ENC-A-IN
- R1 pad 2: Net-(U2A-1A) -> Net-(C2-Pad2)
- R10 pad 1: VDD -> Net-(D4-K)
- R10 pad 2: Net-(U2D-4A) -> GND
- R11 pad 2: /FP-SOC-PWR-SW-IN -> /MB-CFG-SW1-IN
- R12 pad 1: /MB-IND-ERROR -> Net-(D12-K)
- R12 pad 2: Net-(SW4B-LED-R) -> GND
- R13 pad 1: /MB-SOC-PWR-IND -> Net-(D20-K)
- R13 pad 2: Net-(SW4B-LED-G) -> GND
- R14 pad 1: /MB-IND-STATUS -> VDD-STBY
- R14 pad 2: Net-(SW4B-LED-B) -> /MB-CFG-SW2-IN
- R15 pad 1: VDD -> Net-(D25-K)
- R15 pad 2: Net-(U7A-A1) -> GND
- R16 pad 1: VDD -> VDD-STBY
- R16 pad 2: Net-(U7B-A2) -> /MB-CFG-SW3-IN
- R17 pad 1: Net-(U6-REXT) -> Net-(D26-K)
- R18 pad 1: VDD -> VDD-STBY
- R18 pad 2: Net-(U7C-A3) -> /MB-SYS-PWR-SW-IN
- R19 pad 1: VDD -> VDD-STBY
- R19 pad 2: Net-(U7E-A5) -> /MB-SOC-PWR-SW-IN
- R2 pad 1: VDD -> /ENC-B-IN
- R2 pad 2: /NAV-UP-SW-RAW -> Net-(C3-Pad1)
- R20 pad 1: VDD -> VDD-STBY
- R20 pad 2: Net-(U7D-A4) -> /MB-SOC-RST-SW-IN
- R21 pad 1: VDD -> VDD-STBY
- R21 pad 2: Net-(U7F-A6) -> /MB-SOC-SLP-SW-IN
- R22 pad 1: Net-(D1-K) -> Net-(D27-K)
- R23 pad 1: Net-(D2-K) -> VDD-STBY
- R23 pad 2: GND -> /MB-CFG-SW4-IN
- R24 pad 1: Net-(D3-K) -> Net-(D28-K)
- R25 pad 1: Net-(D4-K) -> Net-(D29-K)
- R3 pad 1: VDD -> Net-(D1-K)
- R3 pad 2: /NAV-DOWN-SW-RAW -> GND
- R4 pad 1: VDD -> Net-(D2-K)
- R4 pad 2: /NAV-PUSH-SW-RAW -> GND
- R5 pad 2: /NAV-LEFT-SW-RAW -> Net-(C2-Pad2)
- R6 pad 1: VDD -> Net-(C3-Pad1)
- R6 pad 2: /NAV-RIGHT-SW-RAW -> VDD
- R7 pad 1: VDD -> Net-(U2-REXT)
- R7 pad 2: Net-(U2B-2A) -> GND
- R8 pad 1: VDD -> Net-(U3-REXT)
- R8 pad 2: /NAV-BACK-SW-IN -> GND
- R9 pad 2: Net-(U2C-3A) -> /ENC-SW-IN
- SW1 pad 1: Net-(U2A-1A) -> Net-(U12C-3A)
- SW1 pad 2: Net-(U2A-1A) -> Net-(U12C-3A)
- SW1 pad 6: VDD -> VDD-STBY
- SW10 pad 1: Net-(U7C-A3) -> /MB-SOC-RST-SW-IN
- SW10 pad 2: Net-(U7C-A3) -> /MB-SOC-RST-SW-IN
- SW10 pad 6: VDD -> VDD-STBY
- SW11 pad 1: Net-(U7F-A6) -> Net-(U12B-2A)
- SW11 pad 2: Net-(U7F-A6) -> Net-(U12B-2A)
- SW11 pad 6: VDD -> VDD-STBY
- SW12 pad 1: Net-(U7E-A5) -> Net-(U10B-A2)
- SW12 pad 2: Net-(U7E-A5) -> Net-(U10B-A2)
- SW12 pad 6: VDD -> VDD-STBY
- SW2 pad 1: Net-(U2B-2A) -> /MB-SYS-PWR-SW-IN
- SW2 pad 2: Net-(U2B-2A) -> GND
- SW2 pad 3: GND -> /MB-SYS-PWR-SW-IN
- SW2 pad 5: Net-(SW2B-LED-K) -> VDD-STBY
- SW2 pad 6: VDD -> Net-(SW2B-LED-GK)
- SW3 pad 1: Net-(U2C-3A) -> Net-(U10A-A1)
- SW3 pad 2: Net-(U2C-3A) -> Net-(U10A-A1)
- SW3 pad 6: VDD -> VDD-STBY
- SW4 pad 1: /FP-SOC-PWR-SW-IN -> Net-(U10F-A6)
- SW4 pad 2: /FP-SOC-PWR-SW-IN -> Net-(U10F-A6)
- SW5 pad 1: Net-(U2D-4A) -> /MB-CFG-SW1-IN
- SW5 pad 2: Net-(U2D-4A) -> GND
- SW6 pad 1: Net-(U7A-A1) -> Net-(U12A-1A)
- SW6 pad 2: Net-(U7A-A1) -> Net-(U12A-1A)
- SW6 pad 6: VDD -> VDD-STBY
- SW7 pad 1: Net-(SW7A-SWA-Pad1) -> Net-(U10D-A4)
- SW7 pad 2: Net-(SW7A-SWB-Pad2) -> Net-(U10D-A4)
- SW7 pad 3: Net-(SW7A-SWA-Pad1) -> GND
- SW7 pad 4: Net-(SW7A-SWB-Pad2) -> GND
- SW7 pad 5: VDD -> Net-(SW7B-LED-K)
- SW7 pad 6: Net-(SW7B-LED-GK) -> VDD-STBY
- SW8 pad 1: Net-(U7D-A4) -> Net-(U10E-A5)
- SW8 pad 2: Net-(U7D-A4) -> Net-(U10E-A5)
- SW8 pad 6: VDD -> VDD-STBY
- SW9 pad 1: Net-(U7B-A2) -> Net-(U10C-A3)
- SW9 pad 2: Net-(U7B-A2) -> Net-(U10C-A3)
- SW9 pad 6: VDD -> VDD-STBY
- TP3 pad 1: VCC-USB -> VCC-STBY
- TP4 pad 1: +12V -> VDD-SYS
- U1 pad 1: /MB-SPI-CIPO -> /ENC-SW-IN
- U1 pad 2: GND -> /ENC-B
- U1 pad 3: GND -> /ENC-A-IN
- U1 pad 4: /MB-FP-RESET -> GND
- U1 pad 5: /MB-SPI-BTN-CS -> /ENC-A
- U1 pad 6: unconnected-(U1-NC-Pad6) -> /ENC-B-IN
- U1 pad 7: /MB-BTN1-INT -> /ENC-SW
- U1 pad 8: unconnected-(U1-NC-Pad8) -> VDD-STBY
- U2 pad 10: GND -> Net-(SW2C-LED-RK)
- U2 pad 11: /TEST-STEP-SW -> Net-(SW7B-LED-K)
- U2 pad 12: Net-(U2D-4A) -> Net-(SW9B-LED-K)
- U2 pad 13: GND -> Net-(SW12B-LED-K)
- U2 pad 14: VDD -> Net-(SW3B-LED-K)
- U2 pad 15: GND -> Net-(SW4B-LED-K)
- U2 pad 2: Net-(U2A-1A) -> /MB-SPI-COPI
- U2 pad 3: /TEST-START-SW -> /MB-SPI-SCLK
- U2 pad 4: GND -> /MB-SPI-IND-CS
- U2 pad 5: Net-(U2B-2A) -> Net-(SW1B-LED-K)
- U2 pad 6: /TEST-PAUSE-SW -> Net-(SW6B-LED-K)
- U2 pad 7: GND -> Net-(SW11B-LED-K)
- U2 pad 8: /TEST-STOP-SW -> Net-(SW13B-LED-K)
- U2 pad 9: Net-(U2C-3A) -> Net-(SW2B-LED-GK)
- U3 pad 10: /NAV-LEFT-SW-RAW -> Net-(D23-K)
- U3 pad 11: /NAV-RIGHT-SW -> Net-(D6-K)
- U3 pad 12: /NAV-RIGHT-SW-RAW -> Net-(D10-K)
- U3 pad 13: /NAV-BACK-SW -> Net-(D14-K)
- U3 pad 14: /NAV-BACK-SW-IN -> Net-(D17-K)
- U3 pad 15: GND -> Net-(D7-K)
- U3 pad 16: VDD -> Net-(D11-K)
- U3 pad 2: /NAV-UP-SW-RAW -> /MB-SPI-SDO
- U3 pad 3: /NAV-UP-SW -> /MB-SPI-SCLK
- U3 pad 4: /NAV-DOWN-SW-RAW -> /MB-SPI-IND-CS
- U3 pad 5: /NAV-DOWN-SW -> Net-(D5-K)
- U3 pad 6: /NAV-PUSH-SW-RAW -> Net-(D9-K)
- U3 pad 7: /NAV-PUSH-SW -> Net-(D13-K)
- U3 pad 8: GND -> Net-(D16-K)
- U3 pad 9: /NAV-LEFT-SW -> Net-(D21-K)
- U4 pad 10: /NAV-DOWN-SW -> /TEST-PAUSE-SW
- U4 pad 11: /NAV-PUSH-SW -> /TEST-STOP-SW
- U4 pad 12: /NAV-LEFT-SW -> /TEST-STEP-SW
- U4 pad 13: /NAV-RIGHT-SW -> /MENU-HOME-SW
- U4 pad 14: /NAV-BACK-SW -> /MENU-POWER-SW
- U4 pad 15: /MENU-LCR-SW -> /MENU-VOLTMETER-SW
- U4 pad 16: /MENU-LIGHTING-SW -> /MENU-ELOAD-SW
- U4 pad 18: VDD -> VDD-STBY
- U4 pad 2: VDD -> GND
- U4 pad 7: /MB-BTN2-INT -> /MB-BTN1-INT
- U4 pad 9: /NAV-UP-SW -> /TEST-START-SW
- U5 pad 1: unconnected-(U5-NC-Pad1) -> /MB-SPI-CIPO
- U5 pad 2: /FP-SOC-PWR-SW-IN -> VDD
- U5 pad 4: /MB-SOC-PWR-SW -> /MB-FP-RESET
- U5 pad 5: VDD-STBY -> /MB-SPI-BTN-CS
- U6 pad 1: GND -> /MB-SOC-PWR-SW-IN
- U6 pad 2: /MB-SPI-COPI -> GND
- U6 pad 3: /MB-SPI-SCLK -> /MB-SYS-PWR-SW-IN
- U6 pad 4: /MB-SPI-IND-CS -> /MB-SYS-PWR-SW
- U6 pad 5: Net-(U6-OUT0) -> VDD-STBY
- U6 pad 6: Net-(U6-OUT1) -> /MB-SOC-PWR-SW
- U7 pad 1: GND -> /MB-SOC-RST-SW-IN
- U7 pad 2: Net-(U7A-A1) -> GND
- U7 pad 3: /MENU-HOME-SW -> /MB-SOC-SLP-SW-IN
- U7 pad 4: Net-(U7B-A2) -> /MB-SOC-SLEEP-SW
- U7 pad 5: /MENU-POWER-SW -> VDD-STBY
- U7 pad 6: Net-(U7C-A3) -> /MB-SOC-RESET-SW
Other:
- board size 400 x 50 mm -> 400 x 65 mm
- board text added: "1"
- board text added: "12V"
- board text added: "2"
- board text added: "3"
- board text added: "4"
- board text added: "5"
- board text added: "6"
- board text added: "AUTOMATED TEST CONTROL"
- board text added: "BACK"
- board text added: "CONFIGURABLE"
- board text added: "CONN"
- board text added: "ELOAD"
- board text added: "ERR"
- board text added: "ETH"
- board text added: "FULL SYSTEM RESET"
- board text added: "HOME"
- board text added: "LCR"
- board text added: "LIGHTING"
- board text added: "LINK"
- board text added: "MAIN"
- board text added: "MENU NAV"
- board text added: "MENU SELECT"
- board text added: "PAUSE"
- board text added: "PORT 1"
- board text added: "PORT 2"
- board text added: "PORT 3"
- board text added: "PORT 4"
- board text added: "PORT 5"
- board text added: "POWER"
- board text added: "SLEEP"
- board text added: "SOC"
- board text added: "SOC RESET"
- board text added: "START"
- board text added: "STEP"
- board text added: "STOP"
- board text added: "TX/RX"
- board text added: "USB 3.0 HUB"
- board text added: "VCC STBY"
- board text added: "VCC USB"
- board text added: "VDD"
- board text added: "VDD SYS"
- board text added: "VOLT"
