File: FrontPanel/BenchyFrontPanel/BenchyFrontPanel.kicad_sch (KiCad schematic)
At the start: 117 parts, among them J2 MOTHERBOARD CONN, SW1 TL3215AF160GQ, SW10 TL3215AF160BQ, SW11 TL3215AF160BQ, SW12 TL3215AF160BQ, SW13 TL3365AF180QG, SW14 TL3215AF160BQ, SW2 TL3215AF160YQ, SW3 TL3215AF160RQ, SW4 228CMVARGBFR, SW5 TL3215AF160GQ, SW6 TL3215AF160BQ, SW7 B3W-9000-RG2N, SW8 TL3215AF160BQ, SW9 TL3215AF160BQ, U1 MCP23S08-E/ML, U2 SN74HCS125BQAR, U3 SN74HCS365PWR, U4 MCP23S08-E/ML, U5 TC7PZ17FU,LJ(CT, U6 STP16CP05MTR, U7 SN74HCS365PWR, U8 TC7PZ17FU,LJ(CT, U9 STP16CP05MTR

Commit message: Schematic capture mostly complete. Starting PCB layout
Parts:
- removed J2: MOTHERBOARD CONN, Connector_PinHeader_2.54mm:PinHeader_2x13_P2.54mm_Vertical_SMD, symbol Connector_Generic:Conn_02x13_Odd_Even
- removed S1: B3F-4050, Daxxn_Controls_Buttons:B3F-4050, symbol DX_Control_Button:B3F-4050
- added C1, C10, C16, C17, C18, C21, C41, C42, C6, C7, C9: 100n, Daxxn_Standard_Capacitors:CAP_0402, symbol DX_Capacitor_Ceramic:CL05A104KA5NNNC
- added C2, C3: 10n, Daxxn_Standard_Capacitors:CAP_0402, symbol DX_Capacitor_Ceramic:CL05B103KB5NNNC
- added D11, D15, D18, D19, D22, D24, D3, D7, D8: CZ1-0603-BLUE, Daxxn_LEDs:LED_0603_1608Metric, symbol DX_LED:CZ1-0603-BLUE
- added D27, D29: CZ8-0603-YLW-GREEN, Daxxn_LEDs:LED_0603_1608Metric, symbol DX_LED:CZ8-0603-YLW-GREEN
- added D28, D30: CZ2-0603-GREEN, Daxxn_LEDs:LED_0603_1608Metric, symbol DX_LED:CZ2-0603-GREEN
- added EN1: PEC11R-4220F-S0024, Daxxn_Controls_Encoders:PEC11R, symbol DX_Control_RotaryEncoder:PEC11R-4220F-S0024
- added H10, H11, H9: M2.5, MountingHole:MountingHole_2.7mm_M2.5_ISO7380_Pad, symbol Mechanical:MountingHole_Pad
- added J1: RIGOL-LA-PROBE, Daxxn_Connectors_PCI:10018784-10200TLF, symbol DX_Connector_CardEdge:RIGOL_LA_PROBE
- added J2: 046841045100846+, Daxxn_Connectors_FFC:046841045100846+, symbol DX_Connector_FFC:046841045100846+
- added R1, R2, R5, R6: 10K, Daxxn_Standard_Resistors:RES_0402, symbol DX_Resistor:RC0402JR-0710KL
- added R11, R14, R16, R23, R27, R31, R48, R9: 100K, Daxxn_Standard_Resistors:RES_0402, symbol DX_Resistor:RMCF0402FT100K
- added R22, R24, R25, R26: 1K3, Daxxn_Standard_Resistors:RES_0402, symbol DX_Resistor:RC0402FR-071K3L
- added S1: BOJACK-BTN-6X6X5-2, Daxxn_Controls_Buttons:BOJACK-BTN-6x6x5, symbol DX_Control_Button:BOJACK-BTN-6X6X5-2
- added SW14, SW15, SW18, SW19, SW20, SW21, SW5: TL3365AF180QG, Daxxn_Controls_Buttons:TL3365AF180QG, symbol DX_Control_Button:TL3365AF180QG
- added U1: 74LVC3G17GS,115, Daxxn_Packages:X2SON-8_1.4x1mm_P0.35mm, symbol DX_IC_Logic_Buffer:74LVC3G17GS,115
- added U11: SN74HCS365PWR, Daxxn_Packages:TSSOP-16_4.4x5mm_P0.65mm, symbol DX_IC_Logic_Buffer:SN74HCS365PWR
- added U8: MCP23S08-E/ML, Daxxn_Packages:QFN-20-1EP_4x4mm_P0.5mm_EP2.7x2.7mm, symbol DX_IC_Interface_IOExpander:MCP23S08-E/ML
- renumbered C9 to C11, C29 to C12, C14 to C13, C26 to C14, C27 to C15, C30 to C19, C31 to C20, C3 to C22, C20 to C23, C22 to C24, C4 to C25, C10 to C26, C5 to C27, C24 to C28, C6 to C29, C7 to C30, C23 to C31, C17 to C32, C2 to C33, C8 to C34, C11 to C35, C13 to C36, C16 to C37, C18 to C38, C19 to C39, C15 to C4, C21 to C40, C28 to C5, C1 to C8, D9 to D1, D15 to D10, D2 to D12, D10 to D13, D16 to D14, D11 to D16, D8 to D2, D3 to D20, D12 to D21, D13 to D23, D4 to D25, D5 to D26, D1 to D4, D6 to D5, D14 to D6, D7 to D9, R22 to R10, R23 to R12, R24 to R13, R25 to R15, R28 to R17, R32 to R18, R11 to R19, R26 to R20, R27 to R21, R12 to R28, R13 to R29, R30 to R3, R14 to R30, R2 to R32, R8 to R33, R19 to R34, R21 to R35, R3 to R36, R4 to R37, R5 to R38, R6 to R39, R31 to R4, R1 to R40, R7 to R41, R9 to R42, R10 to R43, R15 to R44, R16 to R45, R18 to R46, R20 to R47, R17 to R7, R29 to R8, SW3 to SW1, SW14 to SW10, SW2 to SW11, SW10 to SW12, SW5 to SW13, SW4 to SW16, SW13 to SW17, SW7 to SW2, SW6 to SW3, SW11 to SW4, SW1 to SW6, SW8 to SW7, SW12 to SW8, TP1 to TP3, TP2 to TP4, TP3 to TP5, TP4 to TP6, TP5 to TP7, U7 to U10, U2 to U12, U6 to U2, U9 to U3, U1 to U4, U4 to U5, U5 to U6, U8 to U7, U3 to U9
Connections:
- net +12V: now also J2.33 (Pin_33)
- net GND: now also SW16.1 (SWA), SW16.2 (SWA), C1.2, C10.2, C16.2, C17.2, C18.2, C2.1, C21.2, C3.2, C41.2, C42.2, C6.2, C7.2, C9.2, EN1.C, EN1.MP, EN1.S2, H10.1, H11.1, H9.1, J1.A1 (GND), J1.A11 (GND), J1.A13 (GND), J1.A15 (GND), J1.A17 (GND), J1.A18 (GND), J1.A3 (GND), J1.A5 (GND), J1.A7 (GND), J1.A9 (GND), J1.B1 (GND), J1.B11 (GND), J1.B13 (GND), J1.B15 (GND), J1.B17 (GND), J1.B18 (GND), J1.B3 (GND), J1.B5 (GND), J1.B7 (GND), J1.B9 (GND), J2.32 (Pin_32), J2.34 (Pin_34), J2.35 (Pin_35), J2.44 (Pin_44), J2.45 (Pin_45), R22.2, R24.2, R25.2, R26.2, S1.2, SW14.2, SW15.2, SW18.2, SW19.2, SW20.2, SW21.2, SW5.2, U1.4 (GND), U11.1 (~{OE1}), U11.15 (~{OE2}), U11.8 (GND), U8.17 (GND), U8.2 (A1), U8.21 (GND); no longer SW16.3 (SWB), SW16.4 (SWB)
- net MB-BTN1-INT: now also J2.19 (Pin_19), U8.7 (INT)
- net MB-BTN2-INT: now also J2.20 (Pin_20)
- net MB-FP-RESET: now also J2.28 (Pin_28), U8.4 (~{RESET})
- net MB-IND-BRIGHT: now also J2.16 (Pin_16)
- net MB-IND-ERROR: now also J2.18 (Pin_18)
- net MB-IND-STATUS: now also J2.17 (Pin_17)
- net MB-SOC-PWR-IND: now also J2.24 (Pin_24)
- net MB-SOC-PWR-SW: now also J2.21 (Pin_21)
- net MB-SOC-PWR-SW-IN: now also SW16.3 (SWB), SW16.4 (SWB); no longer SW16.1 (SWA), SW16.2 (SWA)
- net MB-SOC-RESET-SW: now also J2.26 (Pin_26)
- net MB-SOC-SLEEP-SW: now also J2.9 (Pin_9)
- net MB-SOC-USB-HS-IND: now also J2.11 (Pin_11)
- net MB-SOC-USB-SUSP-IND: now also J2.10 (Pin_10)
- net MB-SPI-BTN-CS: now also J2.7 (Pin_7), U8.5 (~{CS})
- net MB-SPI-CIPO: now also J2.5 (Pin_5), U8.1 (SO)
- net MB-SPI-COPI: now also J2.6 (Pin_6), U8.20 (SI)
- net MB-SPI-IND-CS: now also J2.8 (Pin_8)
- net MB-SPI-SCLK: now also J2.4 (Pin_4), U8.19 (SCK)
- net MB-SYS-PWR-SW: now also J2.25 (Pin_25)
- net NAV-BACK-SW-IN: now also S1.1
- net VCC-STBY: now also J2.23 (Pin_23)
- net VCC-USB: now also J2.29 (Pin_29)
- net VDD: now also J2.3 (Pin_3), R5.1, R6.2, R9.1, U8.3 (A0)
- net VDD-STBY: now also C1.1, C18.1, C41.1, D11.2 (A), D15.2 (A), D18.2 (A), D19.2 (A), D22.2 (A), D24.2 (A), D3.2 (A), D7.2 (A), D8.2 (A), R11.1, R14.1, R16.1, R23.1, R27.1, R31.1, R48.1, U1.8 (VCC), U11.16 (VCC), U8.18 (VDD)
- net VDD-SYS: now also J2.1 (Pin_1), J2.2 (Pin_2), J2.22 (Pin_22)
- net at U3.15 (OUT10): now also D7.1 (K)
- net at U3.16 (OUT11): now also D11.1 (K)
- net at U3.17 (OUT12): now also D15.1 (K)
- net at U3.18 (OUT13): now also D18.1 (K)
- net at U3.19 (OUT14): now also D22.1 (K)
- net at U3.20 (OUT15): now also D24.1 (K)
- net at U2.18 (OUT13): now also D19.1 (K)
- net at U2.19 (OUT14): now also D3.1 (K)
- net at U2.20 (OUT15): now also D8.1 (K)
- new net: D27.1 (K), R22.1
- new net: C2.2, EN1.A, R1.2, R5.2
- new net: C3.1, EN1.B, R2.2, R6.1
- new net: D28.1 (K), R24.1
- new net: D30.1 (K), R26.1
- new net: D29.1 (K), R25.1
- new net: U8.6 (NC), U8.8 (NC)
- new net ENC-A: J2.30 (Pin_30), U1.5 (2Y)
- new net ENC-A-IN: R1.1, U1.3 (2A)
- new net ENC-B: J2.31 (Pin_31), U1.2 (3Y)
- new net ENC-B-IN: R2.1, U1.6 (3A)
- new net ENC-SW: U1.7 (1Y), U8.9 (GP0)
- new net ENC-SW-IN: C6.1, EN1.S1, R9.2, U1.1 (1A)
- new net MB-CFG-SW1: U11.3 (Y1), U8.10 (GP1)
- new net MB-CFG-SW1-IN: C7.1, R11.2, SW5.1, U11.2 (A1)
- new net MB-CFG-SW2: U11.5 (Y2), U8.11 (GP2)
- new net MB-CFG-SW2-IN: C9.1, R14.2, SW14.1, U11.4 (A2)
- new net MB-CFG-SW3: U11.7 (Y3), U8.12 (GP3)
- new net MB-CFG-SW3-IN: C10.1, R16.2, SW15.1, U11.6 (A3)
- new net MB-CFG-SW4: U11.9 (Y4), U8.13 (GP4)
- new net MB-CFG-SW4-IN: C16.1, R23.2, SW18.1, U11.10 (A4)
- new net MB-CFG-SW5: U11.11 (Y5), U8.14 (GP5)
- new net MB-CFG-SW5-IN: C17.1, R27.2, SW19.1, U11.12 (A5)
- new net MB-CFG-SW6: U11.13 (Y6), U8.15 (GP6)
- new net MB-CFG-SW6-IN: C21.1, R31.2, SW20.1, U11.14 (A6)
- new net MB-ETH1-LED1: D28.2 (A), J2.12 (Pin_12)
- new net MB-ETH1-LED2: D27.2 (A), J2.13 (Pin_13)
- new net MB-ETH2-LED1: D30.2 (A), J2.14 (Pin_14)
- new net MB-ETH2-LED2: D29.2 (A), J2.15 (Pin_15)
- new net MB-SYS-RESET: C42.1, J2.27 (Pin_27), R48.2, SW21.1
- new net VIN1: J1.A2 (CH0), J1.B2 (CH8), J2.36 (Pin_36)
- new net VIN2: J1.A4 (CH1), J1.B4 (CH9), J2.37 (Pin_37)
- new net VIN3: J1.A6 (CH2), J1.B6 (CH10), J2.38 (Pin_38)
- new net VIN4: J1.A8 (CH3), J1.B8 (CH11), J2.39 (Pin_39)
- new net VIN5: J1.A10 (CH4), J1.B10 (CH12), J2.40 (Pin_40)
- new net VIN6: J1.A12 (CH5), J1.B12 (CH13), J2.41 (Pin_41)
- new net VIN7: J1.A14 (CH6), J1.B14 (CH14), J2.42 (Pin_42)
- new net VIN8: J1.A16 (CH7), J1.B16 (CH15), J2.43 (Pin_43)
Other:
- note added: "ADDRESS = 0x42"
- note added: "ETHERNET INDICATORS"
- note added: "MENU CONTROLS"
- note added: "MOTHERBOARD CONNECTOR"
- note added: "MOUNTING"
- note added: "NAVIGATION CONTROLS"
- note added: "SWITCH IO-EXPANDERS"
- note added: "SYSTEM SWITCHES"
- note added: "TEST SEQUENCE CONTROLS"
- note added: "USB PORT1"
- note added: "USB PORT2"
- note added: "USB PORT3"
- note added: "USB PORT4"
- note added: "USB PORT5"
- note removed: "MATCH CONNECTOR ON MB"
- note removed: "MENU CONTROL"
- note removed: "TEST SEQUENCE CONTROL"
- moved on the sheet: C11, C12, C13, C14, C15, C19, C20, C22, C23, C24, C25, C26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
Changed lines of the file:
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@@
 	(generator "eeschema")
 	(generator_version "9.0")
-	(paper "A3")
+	(paper "User" 470 340)
 	(title_block
 		(title "Benchy Front Panel")
