File: MotherBoard/BenchyMotherBoard-AM625/BenchyMotherBoard-AM625.kicad_sch (KiCad schematic)
At the start: 16 parts

Commit message: Schematic capture mostly complete. Starting PCB layout
Parts:
- added HS1: 960-19-12-S-AB-0, Daxxn_Thermal_Heatsink:960-19-12-S-AB-0, symbol DX_Thermal_HeatSink:960-19-12-S-AB-0
- H1, H10, H11, H12, H13, H14, H15, H16, H2, H3, H4, H5, H6, H7, H8, H9: symbol Mechanical:MountingHole_Pad_MP -> Mechanical:MountingHole_Pad
Connections:
- net GND: now also H1.1, H10.1, H11.1, H12.1, H13.1, H14.1, H15.1, H16.1, H2.1, H3.1, H4.1, H5.1, H6.1, H7.1, H8.1, H9.1; no longer H1.MP, H10.MP, H11.MP, H12.MP, H13.MP, H14.MP, H15.MP, H16.MP, H2.MP, H3.MP, H4.MP, H5.MP, H6.MP, H7.MP, H8.MP, H9.MP
