File: MotherBoard/BenchyMotherBoard-AM625/BenchyMotherboard-AM625_Display.kicad_sch (KiCad schematic)
At the start: 30 parts, among them J10 HD04-19-TH-TR, J18 B2B-XH-A-M, U1 AM6254ATCGGAALW, U13 SII9022ACNU, U24 TPD12S016RKTR, U51 74LVC1G08GW,125, U54 74LVC1G08GW,125, U72 NCR321UX

Commit message: Schematic capture mostly complete. Starting PCB layout
Parts:
- renumbered C279 to C361, C280 to C362, C277 to C363, C281 to C364, C263 to C365, C262 to C366, C382 to C367, C383 to C368, C257 to C369, C381 to C370, J10 to J14, J18 to J15, R23 to R225, R363 to R226, R365 to R227, R364 to R228, R132 to R229, R57 to R230, R56 to R231, R209 to R232, R217 to R233, U1 to U2, U13 to U5, U24 to U50, U72 to U51, U51 to U52, U54 to U53
Connections:
- net LVDS0-CH0+ is gone; now on net LVDS-CH0+: DS1.9 (LVDS-CH0+)
- net LVDS0-CH0- is gone; now on net LVDS-CH0-: DS1.8 (LVDS-CH0-)
- net LVDS0-CH1+ is gone; now on net LVDS-CH1+: DS1.12 (LVDS-CH1+)
- net LVDS0-CH1- is gone; now on net LVDS-CH1-: DS1.11 (LVDS-CH1-)
- net LVDS0-CH2+ is gone; now on net LVDS-CH2+: DS1.15 (LVDS-CH2+)
- net LVDS0-CH2- is gone; now on net LVDS-CH2-: DS1.14 (LVDS-CH2-)
- net LVDS0-CH3+ is gone; now on net LVDS-CH3+: DS1.21 (LVDS-CH3+)
- net LVDS0-CH3- is gone; now on net LVDS-CH3-: DS1.20 (LVDS-CH3-)
- net LVDS0-CLK+ is gone; now on net LVDS-CLK+: DS1.18 (LVDS-CLK+)
- net LVDS0-CLK- is gone; now on net LVDS-CLK-: DS1.17 (LVDS-CLK-)
