File: MotherBoard/BenchyMotherBoard-AM625/BenchyMotherboard-AM625_LightingCtrl.kicad_sch (KiCad schematic)
At the start: 34 parts, among them J36 B2B-XH-A-M, J38 B2B-XH-A-M, J39 B2B-XH-A-M, SW2 TL3365AF180QG, U66 STM32F042G6U6TR, U67 74LVC1G08GW,125, U68 IS31FL3235A-QFLS2-TR, U70 74LVC3G17GS,115, Y3 16MHz

Commit message: Schematic capture mostly complete. Starting PCB layout
Parts:
- removed U66: STM32F042G6U6TR, Daxxn_Packages:QFN-28_4x4mm_P0.5mm, symbol DX_IC_MCU_ST:STM32F042G6U6TR
- added U68: STM32F042G6U6TR, Daxxn_Packages:QFN-28_4x4mm_P0.5mm, symbol DX_IC_MCU_ST:STM32F042G6U6TR
- JP7: renamed from JP3; footprint (none) -> Daxxn_Other:BOOT_SolderJumper-3_P1.3mm_Open
- renumbered C413 to C425, C415 to C426, C411 to C427, C410 to C428, C409 to C429, C408 to C430, C412 to C431, C414 to C432, C419 to C433, C417 to C434, C420 to C435, C418 to C436, C438 to C437, C421 to C438, J36 to J26, J38 to J27, J39 to J28, R303 to R316, R301 to R317, R302 to R318, R304 to R319, R306 to R320, R305 to R321, R307 to R322, R308 to R323, TP21 to TP47, U68 to U69, U67 to U71
Connections:
- net GND: now also U68.16 (GND)
- net LGT-MCU-BOOT: now also U68.1 (BOOT0)
- net LGT-RGB-I2C-SCL: now also U68.27 (PB6)
- net LGT-RGB-I2C-SDA: now also U68.28 (PB7)
- net LGT-RGB-RESET: now also U68.26 (PB5)
- net LGT-SW-1: now also U68.6 (PA0)
- net LGT-SW-2: now also U68.7 (PA1)
- net LGT-SW-3: now also U68.8 (PA2)
- net LGT-SW-4: now also U68.9 (PA3)
- net LGT-SWCLK: now also U68.22 (PA14)
- net LGT-SWDIO: now also U68.21 (PA13)
- net RESET-LGT-MCU: now also U68.4 (RESET)
- net SOC-LGT-INT: now also U68.14 (PB0)
- net SOC-PWR-EN: now also U68.15 (PB1)
- net SOC-SPI-LGT-CS: now also U68.10 (PA4)
- net SOC-SPI-SCLK: now also U68.11 (PA5)
- net SOC-SPI-SDI: now also U68.12 (PA6)
- net SOC-SPI-SDO: now also U68.13 (PA7)
- net VCC-STBY: now also U68.17 (VDD), U68.18 (VDDIO2), U68.5 (VDDA)
- net at Y3.1: now also U68.2 (OSC-IN)
- net at Y3.3: now also U68.3 (OSC-OUT)
