File: MotherBoard/BenchyMotherBoard-AM625/BenchyMotherboard-AM625_LightingCtrl_RGB1.kicad_sch (KiCad schematic)
At the start: 10 parts, among them J22 B4B-XH-AM, Q13 PMXB43UNEZ, Q14 PMXB43UNEZ, Q15 PMXB43UNEZ

Commit message: Schematic capture mostly complete. Starting PCB layout
Parts:
- renumbered J22 to J33, Q13 to Q17, Q14 to Q18, Q15 to Q19, R321 to R356, R323 to R357, R325 to R358, R320 to R359, R322 to R360, R324 to R361
Changed lines of the file:
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@@
 		(on_board yes)
 		(dnp no)
-		(property "Reference" "#PWR0489"
+		(property "Reference" "#PWR0560"
 			(at 41.91 50.8 0)
 			(effects
@@
 			(project "BenchyMotherBoard-AM625"
 				(path "/7184a1e6-58da-49c8-8a6c-ea31385ec956/8494b7c1-cb3d-49c1-ba37-1630d97ce06f/3fe17120-705d-40ef-9e19-837f254f8ef5"
-					(reference "#PWR0489")
+					(reference "#PWR0560")
 					(unit 1)
 				)
@@
 		(on_board yes)
 		(dnp no)
-		(property "Reference" "R320"
+		(property "Reference" "R359"
 			(at 30.48 40.132 90)
 			(effects
@@
 			(project "BenchyMotherBoard-AM625"
 				(path "/7184a1e6-58da-49c8-8a6c-ea31385ec956/8494b7c1-cb3d-49c1-ba37-1630d97ce06f/3fe17120-705d-40ef-9e19-837f254f8ef5"
-					(reference "R320")
+					(reference "R359")
 					(unit 1)
 				)
@@
 		(on_board yes)
 		(dnp no)
-		(property "Reference" "Q14"
+		(property "Reference" "Q18"
 			(at 72.898 40.386 0)
 			(effects
@@
 			(project "BenchyMotherBoard-AM625"
 				(path "/7184a1e6-58da-49c8-8a6c-ea31385ec956/8494b7c1-cb3d-49c1-ba37-1630d97ce06f/3fe17120-705d-40ef-9e19-837f254f8ef5"
-					(reference "Q14")
+					(reference "Q18")
 					(unit 1)
 				)
@@
 		(on_board yes)
 		(dnp no)
-		(property "Reference" "#PWR0518"
+		(property "Reference" "#PWR0559"
 			(at 96.52 34.29 0)
 			(effects
@@
 			(project "BenchyMotherBoard-AM625"
 				(path "/7184a1e6-58da-49c8-8a6c-ea31385ec956/8494b7c1-cb3d-49c1-ba37-1630d97ce06f/3fe17120-705d-40ef-9e19-837f254f8ef5"
-					(reference "#PWR0518")
+					(reference "#PWR0559")
 					(unit 1)
 				)
@@
 		(on_board yes)
 		(dnp no)
-		(property "Reference" "Q15"
+		(property "Reference" "Q19"
 			(at 103.378 40.386 0)
 			(effects
@@
 			(project "BenchyMotherBoard-AM625"
 				(path "/7184a1e6-58da-49c8-8a6c-ea31385ec956/8494b7c1-cb3d-49c1-ba37-1630d97ce06f/3fe17120-705d-40ef-9e19-837f254f8ef5"
-					(reference "Q15")
+					(reference "Q19")
 					(unit 1)
 				)
@@
 		(on_board yes)
 		(dnp no)
-		(property "Reference" "#PWR0517"
+		(property "Reference" "#PWR0558"
 			(at 66.04 34.29 0)
 			(effects
@@
 			(project "BenchyMotherBoard-AM625"
 				(path "/7184a1e6-58da-49c8-8a6c-ea31385ec956/8494b7c1-cb3d-49c1-ba37-1630d97ce06f/3fe17120-705d-40ef-9e19-837f254f8ef5"
-					(reference "#PWR0517")
+					(reference "#PWR0558")
 					(unit 1)
 				)
@@
 		(on_board yes)
 		(dnp no)
-		(property "Reference" "J22"
+		(property "Reference" "J33"
 			(at 114.808 19.812 0)
 			(effects
@@
 				)
 				(path "/7184a1e6-58da-49c8-8a6c-ea31385ec956/8494b7c1-cb3d-49c1-ba37-1630d97ce06f/3fe17120-705d-40ef-9e19-837f254f8ef5"
-					(reference "J22")
+					(reference "J33")
 					(unit 1)
 				)
@@
 		(on_board yes)
 		(dnp no)
-		(property "Reference" "R324"
+		(property "Reference" "R361"
 			(at 91.44 40.132 90)
 			(effects
@@
 			(project "BenchyMotherBoard-AM625"
 				(path "/7184a1e6-58da-49c8-8a6c-ea31385ec956/8494b7c1-cb3d-49c1-ba37-1630d97ce06f/3fe17120-705d-40ef-9e19-837f254f8ef5"
-					(reference "R324")
+					(reference "R361")
 					(unit 1)
 				)
@@
 		(on_board yes)
 		(dnp no)
-		(property "Reference" "R322"
+		(property "Reference" "R360"
 			(at 60.96 40.132 90)
 			(effects
@@
 			(project "BenchyMotherBoard-AM625"
 				(path "/7184a1e6-58da-49c8-8a6c-ea31385ec956/8494b7c1-cb3d-49c1-ba37-1630d97ce06f/3fe17120-705d-40ef-9e19-837f254f8ef5"
-					(reference "R322")
+					(reference "R360")
 					(unit 1)
 				)
@@
 		(on_board yes)
 		(dnp no)
-		(property "Reference" "#PWR0483"
+		(property "Reference" "#PWR0556"
 			(at 105.41 21.59 0)
 			(effects
@@
 			(project "BenchyMotherBoard-AM625"
 				(path "/7184a1e6-58da-49c8-8a6c-ea31385ec956/8494b7c1-cb3d-49c1-ba37-1630d97ce06f/3fe17120-705d-40ef-9e19-837f254f8ef5"
-					(reference "#PWR0483")
+					(reference "#PWR0556")
 					(unit 1)
 				)
@@
 		(on_board yes)
 		(dnp no)
-		(property "Reference" "R325"
+		(property "Reference" "R358"
 			(at 95.504 32.385 0)
 			(effects
@@
 			(project "BenchyMotherBoard-AM625"
 				(path "/7184a1e6-58da-49c8-8a6c-ea31385ec956/8494b7c1-cb3d-49c1-ba37-1630d97ce06f/3fe17120-705d-40ef-9e19-837f254f8ef5"
-					(reference "R325")
+					(reference "R358")
 					(unit 1)
 				)
@@
 		(on_board yes)
 		(dnp no)
-		(property "Reference" "#PWR0490"
+		(property "Reference" "#PWR0561"
 			(at 72.39 50.8 0)
 			(effects
@@
 			(project "BenchyMotherBoard-AM625"
 				(path "/7184a1e6-58da-49c8-8a6c-ea31385ec956/8494b7c1-cb3d-49c1-ba37-1630d97ce06f/3fe17120-705d-40ef-9e19-837f254f8ef5"
-					(reference "#PWR0490")
+					(reference "#PWR0561")
 					(unit 1)
 				)
@@
 		(on_board yes)
 		(dnp no)
-		(property "Reference" "Q13"
+		(property "Reference" "Q17"
 			(at 42.418 40.386 0)
 			(effects
@@
 			(project "BenchyMotherBoard-AM625"
 				(path "/7184a1e6-58da-49c8-8a6c-ea31385ec956/8494b7c1-cb3d-49c1-ba37-1630d97ce06f/3fe17120-705d-40ef-9e19-837f254f8ef5"
-					(reference "Q13")
+					(reference "Q17")
 					(unit 1)
 				)
@@
 		(on_board yes)
 		(dnp no)
-		(property "Reference" "#PWR0516"
+		(property "Reference" "#PWR0557"
 			(at 35.56 34.29 0)
 			(effects
@@
 			(project ""
 				(path "/7184a1e6-58da-49c8-8a6c-ea31385ec956/8494b7c1-cb3d-49c1-ba37-1630d97ce06f/3fe17120-705d-40ef-9e19-837f254f8ef5"
-					(reference "#PWR0516")
+					(reference "#PWR0557")
 					(unit 1)
 				)
@@
 		(on_board yes)
 		(dnp no)
-		(property "Reference" "#PWR0491"
+		(property "Reference" "#PWR0562"
 			(at 102.87 50.8 0)
 			(effects
@@
 			(project "BenchyMotherBoard-AM625"
 				(path "/7184a1e6-58da-49c8-8a6c-ea31385ec956/8494b7c1-cb3d-49c1-ba37-1630d97ce06f/3fe17120-705d-40ef-9e19-837f254f8ef5"
-					(reference "#PWR0491")
+					(reference "#PWR0562")
 					(unit 1)
 				)
@@
 		(on_board yes)
 		(dnp no)
-		(property "Reference" "R323"
+		(property "Reference" "R357"
 			(at 65.024 32.385 0)
 			(effects
@@
 			(project "BenchyMotherBoard-AM625"
 				(path "/7184a1e6-58da-49c8-8a6c-ea31385ec956/8494b7c1-cb3d-49c1-ba37-1630d97ce06f/3fe17120-705d-40ef-9e19-837f254f8ef5"
-					(reference "R323")
+					(reference "R357")
 					(unit 1)
 				)
@@
 		(on_board yes)
 		(dnp no)
-		(property "Reference" "R321"
+		(property "Reference" "R356"
 			(at 34.544 32.385 0)
 			(effects
@@
 			(project "BenchyMotherBoard-AM625"
 				(path "/7184a1e6-58da-49c8-8a6c-ea31385ec956/8494b7c1-cb3d-49c1-ba37-1630d97ce06f/3fe17120-705d-40ef-9e19-837f254f8ef5"
-					(reference "R321")
-					(unit 1)
-				)
+					(reference "R356")
+					(unit 1)
+				)
