File: MotherBoard/BenchyMotherBoard-AM625/BenchyMotherboard-AM625_LightingCtrl_RGBW1.kicad_sch (KiCad schematic)
At the start: 13 parts, among them J21 B5B-XH-A, Q10 PMXB43UNEZ, Q11 PMXB43UNEZ, Q12 PMXB43UNEZ, Q9 PMXB43UNEZ

Commit message: Schematic capture mostly complete. Starting PCB layout
Parts:
- removed J21: B5B-XH-A, Daxxn_Connectors_JST:B5B-XH-A, symbol DX_Connector_JST:B5B-XH-A
- removed Q10, Q11, Q12, Q9: PMXB43UNEZ, Daxxn_Packages:DFN1010D-3, symbol DX_Transistor_MOSFET:PMXB43UNEZ
- removed R312, R314, R316, R318: 100, Daxxn_Standard_Resistors:RES_0402, symbol DX_Resistor:RC0402JR-07100RL
- removed R313, R315, R317, R319: 10K, Daxxn_Standard_Resistors:RES_0402, symbol DX_Resistor:RC0402JR-0710KL
- added J29: B5B-XH-A, Daxxn_Connectors_JST:B5B-XH-A, symbol DX_Connector_JST:B5B-XH-A
- added Q1, Q2, Q3, Q4: PMXB43UNEZ, Daxxn_Packages:DFN1010D-3, symbol DX_Transistor_MOSFET:PMXB43UNEZ
- added R324, R325, R326, R327: 10K, Daxxn_Standard_Resistors:RES_0402, symbol DX_Resistor:RC0402JR-0710KL
- added R328, R329, R330, R331: 100, Daxxn_Standard_Resistors:RES_0402, symbol DX_Resistor:RC0402JR-07100RL
Connections:
- net ${PREFIX}-BLUE: now also R330.1
- net ${PREFIX}-GREEN: now also R328.1
- net ${PREFIX}-RED: now also R329.1
- net ${PREFIX}-WHITE: now also R331.1
- net +12V: now also J29.1 (Pin_1)
- net GND: now also Q1.2 (S), Q2.2 (S), Q3.2 (S), Q4.2 (S)
- net VDD: now also R324.1, R325.1, R326.1, R327.1
- new net: J29.2 (Pin_2), Q1.3 (D)
- new net: J29.3 (Pin_3), Q2.3 (D)
- new net: J29.4 (Pin_4), Q3.3 (D)
- new net: J29.5 (Pin_5), Q4.3 (D)
- new net: Q4.1 (G), R327.2, R331.2
- new net: Q3.1 (G), R326.2, R330.2
- new net: Q1.1 (G), R324.2, R328.2
- new net: Q2.1 (G), R325.2, R329.2
