File: MotherBoard/BenchyMotherBoard-AM625/BenchyMotherboard-AM625_LightingCtrl_RGBW3.kicad_sch (KiCad schematic)
At the start: 13 parts, among them J21 B5B-XH-A, Q10 PMXB43UNEZ, Q11 PMXB43UNEZ, Q12 PMXB43UNEZ, Q9 PMXB43UNEZ

Commit message: Schematic capture mostly complete. Starting PCB layout
Parts:
- removed J21: B5B-XH-A, Daxxn_Connectors_JST:B5B-XH-A, symbol DX_Connector_JST:B5B-XH-A
- removed R312, R314, R316, R318: 100, Daxxn_Standard_Resistors:RES_0402, symbol DX_Resistor:RC0402JR-07100RL
- removed R313, R315, R317, R319: 10K, Daxxn_Standard_Resistors:RES_0402, symbol DX_Resistor:RC0402JR-0710KL
- added J31: B5B-XH-A, Daxxn_Connectors_JST:B5B-XH-A, symbol DX_Connector_JST:B5B-XH-A
- added R340, R341, R342, R343: 10K, Daxxn_Standard_Resistors:RES_0402, symbol DX_Resistor:RC0402JR-0710KL
- added R344, R345, R346, R347: 100, Daxxn_Standard_Resistors:RES_0402, symbol DX_Resistor:RC0402JR-07100RL
Connections:
- net ${PREFIX}-BLUE: now also R346.1
- net ${PREFIX}-GREEN: now also R344.1
- net ${PREFIX}-RED: now also R345.1
- net ${PREFIX}-WHITE: now also R347.1
- net +12V: now also J31.1 (Pin_1)
- net VDD: now also R340.1, R341.1, R342.1, R343.1
- net at Q9.1 (G): now also R340.2, R344.2
- net at Q11.1 (G): now also R342.2, R346.2
- net at Q10.1 (G): now also R341.2, R345.2
- net at Q10.3 (D): now also J31.3 (Pin_3)
- net at Q12.1 (G): now also R343.2, R347.2
- net at Q11.3 (D): now also J31.4 (Pin_4)
- net at Q12.3 (D): now also J31.5 (Pin_5)
- net at Q9.3 (D): now also J31.2 (Pin_2)
