File: MotherBoard/BenchyMotherBoard-AM625/BenchyMotherboard-AM625_LightingCtrl_RGBW4.kicad_sch (KiCad schematic)
At the start: 13 parts, among them J21 B5B-XH-A, Q10 PMXB43UNEZ, Q11 PMXB43UNEZ, Q12 PMXB43UNEZ, Q9 PMXB43UNEZ

Commit message: Schematic capture mostly complete. Starting PCB layout
Parts:
- renumbered J21 to J32, Q11 to Q13, Q12 to Q14, Q10 to Q15, Q9 to Q16, R317 to R348, R319 to R349, R315 to R350, R313 to R351, R316 to R352, R318 to R353, R314 to R354, R312 to R355
Changed lines of the file:
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@@
 		(on_board yes)
 		(dnp no)
-		(property "Reference" "R312"
+		(property "Reference" "R355"
 			(at 127 43.942 90)
 			(effects
@@
 			(project "BenchyMotherBoard-AM625"
 				(path "/7184a1e6-58da-49c8-8a6c-ea31385ec956/8494b7c1-cb3d-49c1-ba37-1630d97ce06f/2264adf4-5034-4152-a85d-181c7e95aca4"
-					(reference "R312")
+					(reference "R355")
 					(unit 1)
 				)
@@
 		(on_board yes)
 		(dnp no)
-		(property "Reference" "R316"
+		(property "Reference" "R352"
 			(at 31.75 43.942 90)
 			(effects
@@
 			(project "BenchyMotherBoard-AM625"
 				(path "/7184a1e6-58da-49c8-8a6c-ea31385ec956/8494b7c1-cb3d-49c1-ba37-1630d97ce06f/2264adf4-5034-4152-a85d-181c7e95aca4"
-					(reference "R316")
+					(reference "R352")
 					(unit 1)
 				)
@@
 		(on_board yes)
 		(dnp no)
-		(property "Reference" "Q10"
+		(property "Reference" "Q15"
 			(at 107.188 44.196 0)
 			(effects
@@
 			(project "BenchyMotherBoard-AM625"
 				(path "/7184a1e6-58da-49c8-8a6c-ea31385ec956/8494b7c1-cb3d-49c1-ba37-1630d97ce06f/2264adf4-5034-4152-a85d-181c7e95aca4"
-					(reference "Q10")
+					(reference "Q15")
 					(unit 1)
 				)
@@
 		(on_board yes)
 		(dnp no)
-		(property "Reference" "#PWR0522"
+		(property "Reference" "#PWR0551"
 			(at 132.08 38.1 0)
 			(effects
@@
 			(project "BenchyMotherBoard-AM625"
 				(path "/7184a1e6-58da-49c8-8a6c-ea31385ec956/8494b7c1-cb3d-49c1-ba37-1630d97ce06f/2264adf4-5034-4152-a85d-181c7e95aca4"
-					(reference "#PWR0522")
+					(reference "#PWR0551")
 					(unit 1)
 				)
@@
 		(on_board yes)
 		(dnp no)
-		(property "Reference" "#PWR0488"
+		(property "Reference" "#PWR0553"
 			(at 74.93 54.61 0)
 			(effects
@@
 			(project "BenchyMotherBoard-AM625"
 				(path "/7184a1e6-58da-49c8-8a6c-ea31385ec956/8494b7c1-cb3d-49c1-ba37-1630d97ce06f/2264adf4-5034-4152-a85d-181c7e95aca4"
-					(reference "#PWR0488")
+					(reference "#PWR0553")
 					(unit 1)
 				)
@@
 		(on_board yes)
 		(dnp no)
-		(property "Reference" "R318"
+		(property "Reference" "R353"
 			(at 63.5 43.942 90)
 			(effects
@@
 			(project "BenchyMotherBoard-AM625"
 				(path "/7184a1e6-58da-49c8-8a6c-ea31385ec956/8494b7c1-cb3d-49c1-ba37-1630d97ce06f/2264adf4-5034-4152-a85d-181c7e95aca4"
-					(reference "R318")
+					(reference "R353")
 					(unit 1)
 				)
@@
 		(on_board yes)
 		(dnp no)
-		(property "Reference" "Q11"
+		(property "Reference" "Q13"
 			(at 43.688 44.196 0)
 			(effects
@@
 			(project "BenchyMotherBoard-AM625"
 				(path "/7184a1e6-58da-49c8-8a6c-ea31385ec956/8494b7c1-cb3d-49c1-ba37-1630d97ce06f/2264adf4-5034-4152-a85d-181c7e95aca4"
-					(reference "Q11")
+					(reference "Q13")
 					(unit 1)
 				)
@@
 		(on_board yes)
 		(dnp no)
-		(property "Reference" "#PWR0519"
+		(property "Reference" "#PWR0548"
 			(at 36.83 38.1 0)
 			(effects
@@
 			(project ""
 				(path "/7184a1e6-58da-49c8-8a6c-ea31385ec956/8494b7c1-cb3d-49c1-ba37-1630d97ce06f/2264adf4-5034-4152-a85d-181c7e95aca4"
-					(reference "#PWR0519")
+					(reference "#PWR0548")
 					(unit 1)
 				)
@@
 		(on_board yes)
 		(dnp no)
-		(property "Reference" "R313"
+		(property "Reference" "R351"
 			(at 131.064 36.195 0)
 			(effects
@@
 			(project "BenchyMotherBoard-AM625"
 				(path "/7184a1e6-58da-49c8-8a6c-ea31385ec956/8494b7c1-cb3d-49c1-ba37-1630d97ce06f/2264adf4-5034-4152-a85d-181c7e95aca4"
-					(reference "R313")
+					(reference "R351")
 					(unit 1)
 				)
@@
 		(on_board yes)
 		(dnp no)
-		(property "Reference" "R317"
+		(property "Reference" "R348"
 			(at 35.814 36.195 0)
 			(effects
@@
 			(project "BenchyMotherBoard-AM625"
 				(path "/7184a1e6-58da-49c8-8a6c-ea31385ec956/8494b7c1-cb3d-49c1-ba37-1630d97ce06f/2264adf4-5034-4152-a85d-181c7e95aca4"
-					(reference "R317")
+					(reference "R348")
 					(unit 1)
 				)
@@
 		(on_board yes)
 		(dnp no)
-		(property "Reference" "R319"
+		(property "Reference" "R349"
 			(at 67.564 36.195 0)
 			(effects
@@
 			(project "BenchyMotherBoard-AM625"
 				(path "/7184a1e6-58da-49c8-8a6c-ea31385ec956/8494b7c1-cb3d-49c1-ba37-1630d97ce06f/2264adf4-5034-4152-a85d-181c7e95aca4"
-					(reference "R319")
+					(reference "R349")
 					(unit 1)
 				)
@@
 		(on_board yes)
 		(dnp no)
-		(property "Reference" "Q12"
+		(property "Reference" "Q14"
 			(at 75.438 44.196 0)
 			(effects
@@
 			(project "BenchyMotherBoard-AM625"
 				(path "/7184a1e6-58da-49c8-8a6c-ea31385ec956/8494b7c1-cb3d-49c1-ba37-1630d97ce06f/2264adf4-5034-4152-a85d-181c7e95aca4"
-					(reference "Q12")
+					(reference "Q14")
 					(unit 1)
 				)
@@
 		(on_board yes)
 		(dnp no)
-		(property "Reference" "J21"
+		(property "Reference" "J32"
 			(at 149.098 19.812 0)
 			(effects
@@
 				)
 				(path "/7184a1e6-58da-49c8-8a6c-ea31385ec956/8494b7c1-cb3d-49c1-ba37-1630d97ce06f/2264adf4-5034-4152-a85d-181c7e95aca4"
-					(reference "J21")
+					(reference "J32")
 					(unit 1)
 				)
@@
 		(on_board yes)
 		(dnp no)
-		(property "Reference" "#PWR0482"
+		(property "Reference" "#PWR0547"
 			(at 139.7 21.59 0)
 			(effects
@@
 				)
 				(path "/7184a1e6-58da-49c8-8a6c-ea31385ec956/8494b7c1-cb3d-49c1-ba37-1630d97ce06f/2264adf4-5034-4152-a85d-181c7e95aca4"
-					(reference "#PWR0482")
+					(reference "#PWR0547")
 					(unit 1)
 				)
@@
 		(on_board yes)
 		(dnp no)
-		(property "Reference" "#PWR0487"
+		(property "Reference" "#PWR0552"
 			(at 43.18 54.61 0)
 			(effects
@@
 			(project "BenchyMotherBoard-AM625"
 				(path "/7184a1e6-58da-49c8-8a6c-ea31385ec956/8494b7c1-cb3d-49c1-ba37-1630d97ce06f/2264adf4-5034-4152-a85d-181c7e95aca4"
-					(reference "#PWR0487")
+					(reference "#PWR0552")
 					(unit 1)
 				)
@@
 		(on_board yes)
 		(dnp no)
-		(property "Reference" "R315"
+		(property "Reference" "R350"
 			(at 99.314 36.195 0)
 			(effects
@@
 			(project "BenchyMotherBoard-AM625"
 				(path "/7184a1e6-58da-49c8-8a6c-ea31385ec956/8494b7c1-cb3d-49c1-ba37-1630d97ce06f/2264adf4-5034-4152-a85d-181c7e95aca4"
-					(reference "R315")
+					(reference "R350")
 					(unit 1)
 				)
@@
 		(on_board yes)
 		(dnp no)
-		(property "Reference" "#PWR0486"
+		(property "Reference" "#PWR0554"
 			(at 106.68 54.61 0)
 			(effects
@@
 			(project "BenchyMotherBoard-AM625"
 				(path "/7184a1e6-58da-49c8-8a6c-ea31385ec956/8494b7c1-cb3d-49c1-ba37-1630d97ce06f/2264adf4-5034-4152-a85d-181c7e95aca4"
-					(reference "#PWR0486")
+					(reference "#PWR0554")
 					(unit 1)
 				)
@@
 		(on_board yes)
 		(dnp no)
-		(property "Reference" "#PWR0520"
+		(property "Reference" "#PWR0549"
 			(at 68.58 38.1 0)
 			(effects
@@
 			(project "BenchyMotherBoard-AM625"
 				(path "/7184a1e6-58da-49c8-8a6c-ea31385ec956/8494b7c1-cb3d-49c1-ba37-1630d97ce06f/2264adf4-5034-4152-a85d-181c7e95aca4"
-					(reference "#PWR0520")
+					(reference "#PWR0549")
 					(unit 1)
 				)
@@
 		(on_board yes)
 		(dnp no)
-		(property "Reference" "R314"
+		(property "Reference" "R354"
 			(at 95.25 43.942 90)
 			(effects
@@
 			(project "BenchyMotherBoard-AM625"
 				(path "/7184a1e6-58da-49c8-8a6c-ea31385ec956/8494b7c1-cb3d-49c1-ba37-1630d97ce06f/2264adf4-5034-4152-a85d-181c7e95aca4"
-					(reference "R314")
+					(reference "R354")
 					(unit 1)
 				)
@@
 		(on_board yes)
 		(dnp no)
-		(property "Reference" "#PWR0485"
+		(property "Reference" "#PWR0555"
 			(at 138.43 54.61 0)
 			(effects
@@
 			(project "BenchyMotherBoard-AM625"
 				(path "/7184a1e6-58da-49c8-8a6c-ea31385ec956/8494b7c1-cb3d-49c1-ba37-1630d97ce06f/2264adf4-5034-4152-a85d-181c7e95aca4"
-					(reference "#PWR0485")
+					(reference "#PWR0555")
 					(unit 1)
 				)
@@
 		(on_board yes)
 		(dnp no)
-		(property "Reference" "#PWR0521"
+		(property "Reference" "#PWR0550"
 			(at 100.33 38.1 0)
 			(effects
@@
 			(project "BenchyMotherBoard-AM625"
 				(path "/7184a1e6-58da-49c8-8a6c-ea31385ec956/8494b7c1-cb3d-49c1-ba37-1630d97ce06f/2264adf4-5034-4152-a85d-181c7e95aca4"
-					(reference "#PWR0521")
+					(reference "#PWR0550")
 					(unit 1)
 				)
@@
 		(on_board yes)
 		(dnp no)
-		(property "Reference" "Q9"
+		(property "Reference" "Q16"
 			(at 138.938 44.196 0)
 			(effects
@@
 			(project "BenchyMotherBoard-AM625"
 				(path "/7184a1e6-58da-49c8-8a6c-ea31385ec956/8494b7c1-cb3d-49c1-ba37-1630d97ce06f/2264adf4-5034-4152-a85d-181c7e95aca4"
-					(reference "Q9")
-					(unit 1)
-				)
+					(reference "Q16")
+					(unit 1)
+				)
