File: MotherBoard/BenchyMotherBoard-AM625/BenchyMotherboard-AM625_LightingCtrl_SwitchedChannels.kicad_sch (KiCad schematic)
At the start: 16 parts, among them J33 B2B-XH-A-M, J34 B2B-XH-A-M, J35 B2B-XH-A-M, J37 B2B-XH-A-M, Q22 PMXB43UNEZ, Q23 PMXB43UNEZ, Q24 PMXB43UNEZ, Q26 PMXB43UNEZ

Commit message: Schematic capture mostly complete. Starting PCB layout
Parts:
- renumbered J33 to J41, J35 to J42, J37 to J43, J34 to J44, Q22 to Q29, Q24 to Q30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
