File: MotherBoard/BenchyMotherBoard-AM625/BenchyMotherboard-AM625_Power.kicad_sch (KiCad schematic)
At the start: 319 parts, among them J13 B4B-XH-AM, U1 AM6254ATCGGAALW, U10 KSZ9021RN, U12 KSZ9021RN, U13 SII9022ACNU, U2 TPS65400RGZT, U20 TLV75901PDRVR, U23 TLV75901PDRVR, U26 AZ1117IH-5.0TRG1, U4 AP3401DNTR-G1, U5 TLV75518PDRVR, U52 74LVC1G08GW,125, U53 74LVC1G08GW,125, U6 MAX16043TG+T, U69 ADM1085AKSZ-REEL7, U7 TPS7A0225PDBVR, U9 USB7206C/KDX

Commit message: Schematic capture mostly complete. Starting PCB layout
Parts:
- removed C422, C424: 10n, Daxxn_Standard_Capacitors:CAP_0402, symbol DX_Capacitor_Ceramic:CL05B103KB5NNNC
- removed C423: 100n, Daxxn_Standard_Capacitors:CAP_0402, symbol DX_Capacitor_Ceramic:CL05B104KA5NNNC
- removed D3: APHCM2012SURCK-F01, Daxxn_Standard_LEDs:LED_0805, symbol DX_LED:APHCM2012SURCK-F01
- removed R165: 2K2, Daxxn_Standard_Resistors:RES_0402, symbol DX_Resistor:RC0402JR-072K2L
- removed R309, R310: R, Daxxn_Standard_Resistors:RES_0402, symbol DX_Device:R
- removed R311: 10K, Daxxn_Standard_Resistors:RES_0402, symbol DX_Resistor:RC0402JR-0710KL
- removed U69: ADM1085AKSZ-REEL7, Daxxn_Packages:SOT-363_SC-70-6, symbol DX_IC_PMIC_Supervisor:ADM1085AKSZ-REEL7
- U13: renamed from U6; footprint Daxxn_Packages:TQFN-24-1EP_4x4mm_P0.5mm_EP2.1x2.1mm -> Daxxn_Packages:QFN50P400X400X80-25N
- renumbered C16 to C1, C63 to C10, C177 to C100, C178 to C101, C79 to C102, C73 to C103, C21 to C104, C80 to C105, C179 to C106, C180 to C107, C181 to C108, C182 to C109, C64 to C11, C183 to C110, C81 to C111, C22 to C112, C9 to C113, C5 to C114, C6 to C115, C7 to C116, C8 to C117, C4 to C118, C3 to C119, C65 to C12, C2 to C120, C1 to C121, C112 to C122, C113 to C123, C111 to C124, C114 to C125, C158 to C126, C131 to C127, C132 to C128, C148 to C129, C66 to C13, C147 to C130, C133 to C131, C134 to C132, C135 to C133, C233 to C134, C231 to C135, C232 to C136, C222 to C137, C223 to C138, C224 to C139, C67 to C14, C225 to C140, C226 to C141, C227 to C142, C228 to C143, C229 to C144, C230 to C145, C130 to C146, C129 to C147, C127 to C148, C128 to C149, C68 to C15, C149 to C150, C157 to C151, C155 to C152, C156 to C153, C150 to C154, C151 to C155, C152 to C156, C153 to C157, C154 to C158, C139 to C159, C69 to C16, C140 to C160, C141 to C161, C142 to C162, C143 to C163, C144 to C164, C145 to C165, C146 to C166, C138 to C167, C137 to C168, C136 to C169, C50 to C17, C126 to C170, C125 to C171, C124 to C172, C123 to C173, C122 to C174, C115 to C175, C189 to C176, C190 to C177, C191 to C178, C184 to C179, C51 to C18, C185 to C180, C186 to C181, C187 to C182, C188 to C183, C259 to C184, C260 to C185, C258 to C186, C261 to C187, C204 to C188, C205 to C189, C52 to C19, C206 to C190, C198 to C191, C199 to C192, C200 to C193, C201 to C194, C202 to C195, C203 to C196, C192 to C197, C193 to C198, C194 to C199, C15 to C2, C53 to C20, C195 to C200, C196 to C201, C197 to C202, C87 to C203, C313 to C204, C207 to C205, C208 to C206, C209 to C207, C210 to C208, C211 to C209, C54 to C21, C212 to C210, C213 to C211, C214 to C212, C215 to C213, C216 to C214, C217 to C215, C218 to C216, C219 to C217, C220 to C218, C221 to C219, C161 to C22, C319 to C220, C86 to C221, C85 to C222, C84 to C223, C320 to C224, C318 to C225, C160 to C23, C159 to C24, C17 to C25, C70 to C26, C18 to C27, C75 to C28, C162 to C29, C56 to C3, C165 to C30, C167 to C31, C163 to C32, C164 to C33, C74 to C34, C102 to C35, C103 to C36, C104 to C37, C105 to C38, C106 to C39, C57 to C4, C91 to C40, C92 to C41, C93 to C42, C94 to C43, C95 to C44, C96 to C45, C97 to C46, C98 to C47, C45 to C48, C46 to C49, C58 to C5, C47 to C50, C48 to C51, C49 to C52, C40 to C53, C41 to C54, C42 to C55, C43 to C56, C44 to C57, C35 to C58, C36 to C59, C59 to C6, C37 to C60, C38 to C61, C39 to C62, C71 to C63, C19 to C64, C76 to C65, C171 to C66, C173 to C67, C172 to C68, C168 to C69, C60 to C7, C169 to C70, C170 to C71, C174 to C72, C77 to C73, C72 to C74, C20 to C75, C78 to C76, C108 to C77, C109 to C78, C55 to C79, C61 to C8, C99 to C80, C100 to C81, C101 to C82, C107 to C83, C27 to C84, C28 to C85, C29 to C86, C30 to C87, C31 to C88, C14 to C89, C62 to C9, C13 to C90, C12 to C91, C11 to C92, C10 to C93, C32 to C94, C33 to C95, C34 to C96, C175 to C97, C176 to C98, C166 to C99, J13 to J1, L3 to L1, L6 to L2, L1 to L3, L2 to L4, R7 to R10, R12 to R11, R11 to R12, R20 to R13, R8 to R14, R9 to R17, R10 to R18, R45 to R19, R17 to R2, R49 to R20, R55 to R21, R54 to R22, R51 to R23, R52 to R24, R50 to R25, R53 to R26, R212 to R27, R214 to R28, R184 to R29, R2 to R3, R185 to R30, R186 to R31, R187 to R32, R343 to R33, R21 to R34, R215 to R35, R216 to R36, R182 to R37, R164 to R38, R3 to R4, R183 to R40, R18 to R5, R4 to R6, R5 to R7, R19 to R8, R6 to R9, TP28 to TP1, TP35 to TP10, TP38 to TP11, TP39 to TP12, TP40 to TP13, TP41 to TP14, TP42 to TP15, TP9 to TP16, TP14 to TP17, TP15 to TP18, TP16 to TP19, TP29 to TP2, TP17 to TP20, TP18 to TP21, TP10 to TP22, TP11 to TP23, TP12 to TP24, TP13 to TP25, TP30 to TP3, TP31 to TP4, TP36 to TP5, TP37 to TP6, TP32 to TP7, TP33 to TP8, TP34 to TP9, U2 to U1, U26 to U11, U52 to U14, U53 to U15, U1 to U2, U7 to U3, U20 to U4, U13 to U5, U5 to U6, U4 to U7, U9 to U8, U23 to U9
Connections:
- net VDD-DDR-EN is gone; now on net PSEQ-EN2: U7.1 (EN)
- net PSEQ-EN1: no longer U1.48 (ENSW1/ENSEQ)
- net SOC-PWR-EN: now also U1.48 (ENSW1/ENSEQ)
Other:
- note added: "DDR4 VPP SUPPLY (2V5)"
- note added: "EFUSE PROGRAMMING SUPPLY (1V8)"
- note added: "HDMI CONNECTOR SUPPLY (5V)"
- note added: "MAIN SOC SUPPLY"
- moved on the sheet: C146, C147, C148, C149, C150, C151, C152, C153, C154, C155, C156, C157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
