File: MotherBoard/BenchyMotherBoard-AM625/BenchyMotherboard-AM625_PowerDistribution.kicad_sch (KiCad schematic)
At the start: 72 parts, among them J1 S4B-XA-SK, J15 ATX-0039299243, J16 ATX-0039293046, J19 0039293046, J24 B4B-XH-AM, J25 B4B-XH-AM, J26 B4B-XH-AM, J27 B4B-XH-AM, J41 FRONT PANEL CONN, SW1 TL3365AF180QG, U14 74LVC1G17GV,125, U3 LM317-JCET, U36 74AVC4T245BQ,115, U37 74LVC1G17GV,125, U59 STM32F412RGT6, U71 74AVC4T245BQ,115, Y2 16MHz

Commit message: Schematic capture mostly complete. Starting PCB layout
Parts:
- removed C314, C315, C384, C385: 100n, Daxxn_Standard_Capacitors:CAP_0402, symbol DX_Capacitor_Ceramic:CL05A104KA5NNNC
- removed J41: FRONT PANEL CONN, Connector_PinHeader_2.54mm:PinHeader_2x17_P2.54mm_Horizontal, symbol Connector_Generic:Conn_02x17_Odd_Even
- removed R218, R219, R26, R35: 10K, Daxxn_Standard_Resistors:RES_0402, symbol DX_Resistor:RC0402JR-0710KL
- removed S6: PS-5850A-6PL, Daxxn_Controls_Switches:PS-5850A-6PL, symbol DX_Control_Button:PS-5850A-6PL
- removed TP44: TP-FP-EXTRA1, TestPoint:TestPoint_Pad_D2.5mm, symbol DX_Device:TEST-POINT
- removed TP45: TP-FP-EXTRA2, TestPoint:TestPoint_Pad_D2.5mm, symbol DX_Device:TEST-POINT
- removed TP46: TP-FP-EXTRA3, TestPoint:TestPoint_Pad_D2.5mm, symbol DX_Device:TEST-POINT
- removed TP47: TP-FP-EXTRA4, TestPoint:TestPoint_Pad_D2.5mm, symbol DX_Device:TEST-POINT
- removed U14, U37: 74LVC1G17GV,125, Daxxn_Packages:SOT-23-5, symbol DX_IC_Logic_Buffer:74LVC1G17GV,125
- added C439: 100n, Daxxn_Standard_Capacitors:CAP_0402, symbol DX_Capacitor_Ceramic:CL05A104KA5NNNC
- added J24: 62684-451100ALF, Daxxn_Connectors_FFC:62684-451100ALF, symbol DX_Connector_FFC:62684-451100ALF
- added U72: 74LVC1G08GW,125, Daxxn_Packages:SOT-353_SC-70-5, symbol DX_IC_Logic_AND:74LVC1G08GW,125
- renumbered C367 to C371, C368 to C372, C369 to C373, C370 to C374, C371 to C377, C372 to C378, C373 to C379, C374 to C380, C23 to C381, C26 to C382, C24 to C383, C25 to C384, C356 to C385, C357 to C386, C358 to C387, C359 to C388, C360 to C389, C361 to C390, C362 to C391, C363 to C392, C364 to C393, C386 to C394, C365 to C395, C366 to C396, C427 to C397, C428 to C398, J15 to J16, J16 to J17, J19 to J18, J25 to J19, J26 to J20, J24 to J21, J27 to J22, J1 to J23, JP1 to JP6, JPR1 to JPR2, L4 to L6, R126 to R234, R125 to R235, R13 to R236, R14 to R237, R129 to R238, R130 to R239, R127 to R240, R211 to R241, R210 to R242, R213 to R243, TP22 to TP42, U59 to U54, U3 to U55, U36 to U56, U71 to U57
Connections:
- net SOC-PWR-SW is gone; now on net FP-SOC-PWR-SW: U54.24 (PC4)
- net +12V: now also J24.33 (Pin_33)
- net 3V3: now also J24.1 (Pin_1), J24.2 (Pin_2), J24.22 (Pin_22)
- net 5V: now also J24.29 (Pin_29)
- net ETH1-LED1: now also J24.12 (Pin_12)
- net ETH1-LED2: now also J24.13 (Pin_13)
- net ETH2-LED1: now also J24.14 (Pin_14)
- net ETH2-LED2: now also J24.15 (Pin_15)
- net FP-BTN1-INT: now also J24.19 (Pin_19)
- net FP-BTN2-INT: now also J24.20 (Pin_20)
- net FP-IND-BRIGHT: now also J24.16 (Pin_16)
- net FP-IND-ERROR: now also J24.18 (Pin_18)
- net FP-IND-STATUS: now also J24.17 (Pin_17)
- net FP-RESET: now also J24.28 (Pin_28)
- net FP-SOC-PWR-IND: now also J24.24 (Pin_24)
- net FP-SOC-PWR-SW: now also J24.21 (Pin_21)
- net FP-SOC-RESET-SW: now also J24.26 (Pin_26)
- net FP-SOC-SLEEP-SW: now also J24.9 (Pin_9)
- net FP-SPI-BTN-CS: now also J24.7 (Pin_7)
- net FP-SPI-CIPO: now also J24.5 (Pin_5)
- net FP-SPI-COPI: now also J24.6 (Pin_6)
- net FP-SPI-IND-CS: now also J24.8 (Pin_8)
- net FP-SPI-SCLK: now also J24.4 (Pin_4)
- net FP-SYS-PWR-SW: now also J24.25 (Pin_25)
- net GND: now also C439.1, J24.32 (Pin_32), J24.34 (Pin_34), J24.35 (Pin_35), J24.44 (Pin_44), J24.45 (Pin_45), J24.MP (MountPin), U72.3 (GND)
- net PMCU-RESET: now also U72.4 (Y); no longer R234.2, SW1.1
- net USB-SOC-HS-IND: now also J24.11 (Pin_11)
- net USB-SOC-SUSP-IND: now also J24.10 (Pin_10)
- net VCC-STBY: now also J24.23 (Pin_23)
- net VDD: now also C439.2, J24.3 (Pin_3), U72.5 (VCC)
- net BOOT renamed PMCU-BOOT
- new net ENC-A: J24.30 (Pin_30)
- new net ENC-B: J24.31 (Pin_31)
- new net PMCU-RESET-SW: R234.2, SW1.1, U72.2 (A)
- new net SYS-RESET: J24.27 (Pin_27), U72.1 (B)
- new net VIN1: J24.36 (Pin_36)
- new net VIN2: J24.37 (Pin_37)
- new net VIN3: J24.38 (Pin_38)
- new net VIN4: J24.39 (Pin_39)
- new net VIN5: J24.40 (Pin_40)
- new net VIN6: J24.41 (Pin_41)
- new net VIN7: J24.42 (Pin_42)
- new net VIN8: J24.43 (Pin_43)
- no-connect marks 2 -> 0
Other:
- note added: "NEED TO REFACTOR THE RESET BLOCK DIAGRAM."
- note removed: "MAIN POWER SWITCH"
- moved on the sheet: C371, C372, C373, C374, C375, C376, C377, C378, C379, C380, C381, C382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
