File: MotherBoard/BenchyMotherBoard-AM625/BenchyMotherboard-AM625_SOC-Control.kicad_sch (KiCad schematic)
At the start: 53 parts, among them U1 AM6254ATCGGAALW, U15 LMK1C1104DQFR, U34 TMP100NA/3K, U35 TMP100NA/3K, U42 SN74HCS541DGSR, U48 74LVC1G08GW,125, U49 74LVC1G08GW,125, X1 32.768KHz, X2 25MHz, Y1 25MHz

Commit message: Schematic capture mostly complete. Starting PCB layout
Parts:
- R52: renamed from R347; footprint Daxxn_Standard_Resistors:RES_0402 -> Daxxn_Standard_Resistors:RES_0201
- R54: renamed from R349; footprint Daxxn_Standard_Resistors:RES_0402 -> Daxxn_Standard_Resistors:RES_0201
- renumbered C110 to C226, C426 to C227, C425 to C228, C308 to C229, C440 to C230, C441 to C231, C316 to C232, C303 to C233, C304 to C234, C88 to C235, C90 to C236, JPR2 to JPR1, R139 to R41, R136 to R42, R140 to R43, R142 to R44, R137 to R45, R138 to R46, R131 to R47, R39 to R48, R41 to R49, R40 to R50, R350 to R51, R345 to R53, R143 to R55, R141 to R56, R146 to R57, R144 to R58, R33 to R59, R32 to R60, R69 to R61, R31 to R62, R30 to R63, TP2 to TP26, TP4 to TP27, TP1 to TP28, TP5 to TP29, TP3 to TP30, TP6 to TP31, TP8 to TP32, TP7 to TP33, U42 to U16, U48 to U17, U49 to U18, U34 to U19, U1 to U2, U35 to U20, U15 to U21, X2 to X1, X1 to X2
