File: MotherBoard/BenchyMotherBoard-AM625/BenchyMotherboard-AM625_SPI-Flash.kicad_sch (KiCad schematic)
At the start: 19 parts, among them U1 AM6254ATCGGAALW, U21 S28HS512TGABHI010, U31 74LVC1G08GW,125

Commit message: Schematic capture mostly complete. Starting PCB layout
Parts:
- renumbered C278 to C301, C276 to C302, C275 to C303, C274 to C304, C273 to C305, C272 to C306, R62 to R161, R63 to R162, R67 to R163, R68 to R164, R66 to R165, R60 to R166, R64 to R167, R61 to R168, R65 to R169, R59 to R170, U1 to U2, U21 to U37, U31 to U38
Changed lines of the file:
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@@
 		(on_board yes)
 		(dnp no)
-		(property "Reference" "R63"
+		(property "Reference" "R162"
 			(at 98.806 31.115 0)
 			(effects
@@
 			(project ""
 				(path "/7184a1e6-58da-49c8-8a6c-ea31385ec956/aad981fb-9d0f-43cf-87cf-306d8b58c3f7"
-					(reference "R63")
+					(reference "R162")
 					(unit 1)
 				)
@@
 		(on_board yes)
 		(dnp no)
-		(property "Reference" "R61"
+		(property "Reference" "R168"
 			(at 153.416 99.695 0)
 			(effects
@@
 			(project "BenchyMotherBoard-AM625"
 				(path "/7184a1e6-58da-49c8-8a6c-ea31385ec956/aad981fb-9d0f-43cf-87cf-306d8b58c3f7"
-					(reference "R61")
+					(reference "R168")
 					(unit 1)
 				)
@@
 		(on_board yes)
 		(dnp no)
-		(property "Reference" "R59"
+		(property "Reference" "R170"
 			(at 107.95 112.395 0)
 			(effects
@@
 			(project "BenchyMotherBoard-AM625"
 				(path "/7184a1e6-58da-49c8-8a6c-ea31385ec956/aad981fb-9d0f-43cf-87cf-306d8b58c3f7"
-					(reference "R59")
+					(reference "R170")
 					(unit 1)
 				)
@@
 		(on_board yes)
 		(dnp no)
-		(property "Reference" "U1"
+		(property "Reference" "U2"
 			(at 165.1 19.812 0)
 			(effects
@@
 			(project "BenchyMotherBoard-AM625"
 				(path "/7184a1e6-58da-49c8-8a6c-ea31385ec956/aad981fb-9d0f-43cf-87cf-306d8b58c3f7"
-					(reference "U1")
+					(reference "U2")
 					(unit 9)
 				)
@@
 		(on_board yes)
 		(dnp yes)
-		(property "Reference" "R65"
+		(property "Reference" "R169"
 			(at 164.592 100.838 90)
 			(effects
@@
 			(project "BenchyMotherBoard-AM625"
 				(path "/7184a1e6-58da-49c8-8a6c-ea31385ec956/aad981fb-9d0f-43cf-87cf-306d8b58c3f7"
-					(reference "R65")
+					(reference "R169")
 					(unit 1)
 				)
@@
 		(on_board yes)
 		(dnp no)
-		(property "Reference" "C276"
+		(property "Reference" "C302"
 			(at 44.958 42.926 0)
 			(effects
@@
 			(project "BenchyMotherBoard-AM625"
 				(path "/7184a1e6-58da-49c8-8a6c-ea31385ec956/aad981fb-9d0f-43cf-87cf-306d8b58c3f7"
-					(reference "C276")
+					(reference "C302")
 					(unit 1)
 				)
@@
 		(on_board yes)
 		(dnp no)
-		(property "Reference" "C273"
+		(property "Reference" "C305"
 			(at 64.008 42.926 0)
 			(effects
@@
 			(project "BenchyMotherBoard-AM625"
 				(path "/7184a1e6-58da-49c8-8a6c-ea31385ec956/aad981fb-9d0f-43cf-87cf-306d8b58c3f7"
-					(reference "C273")
+					(reference "C305")
 					(unit 1)
 				)
@@
 		(on_board yes)
 		(dnp no)
-		(property "Reference" "U31"
+		(property "Reference" "U38"
 			(at 95.25 124.206 0)
 			(effects
@@
 			(project ""
 				(path "/7184a1e6-58da-49c8-8a6c-ea31385ec956/aad981fb-9d0f-43cf-87cf-306d8b58c3f7"
-					(reference "U31")
+					(reference "U38")
 					(unit 1)
 				)
@@
 		(on_board yes)
 		(dnp no)
-		(property "Reference" "C272"
+		(property "Reference" "C306"
 			(at 86.36 109.22 90)
 			(effects
@@
 			(project "BenchyMotherBoard-AM625"
 				(path "/7184a1e6-58da-49c8-8a6c-ea31385ec956/aad981fb-9d0f-43cf-87cf-306d8b58c3f7"
-					(reference "C272")
+					(reference "C306")
 					(unit 1)
 				)
@@
 		(on_board yes)
 		(dnp yes)
-		(property "Reference" "R60"
+		(property "Reference" "R166"
 			(at 153.416 92.075 0)
 			(effects
@@
 			(project ""
 				(path "/7184a1e6-58da-49c8-8a6c-ea31385ec956/aad981fb-9d0f-43cf-87cf-306d8b58c3f7"
-					(reference "R60")
+					(reference "R166")
 					(unit 1)
 				)
@@
 		(on_board yes)
 		(dnp no)
-		(property "Reference" "C275"
+		(property "Reference" "C303"
 			(at 51.308 42.926 0)
 			(effects
@@
 			(project "BenchyMotherBoard-AM625"
 				(path "/7184a1e6-58da-49c8-8a6c-ea31385ec956/aad981fb-9d0f-43cf-87cf-306d8b58c3f7"
-					(reference "C275")
+					(reference "C303")
 					(unit 1)
 				)
@@
 		(on_board no)
 		(dnp no)
-		(property "Reference" "#PWR0162"
+		(property "Reference" "#PWR0237"
 			(at 96.52 104.14 0)
 			(effects
@@
 			(project "BenchyMotherBoard-AM625"
 				(path "/7184a1e6-58da-49c8-8a6c-ea31385ec956/aad981fb-9d0f-43cf-87cf-306d8b58c3f7"
-					(reference "#PWR0162")
+					(reference "#PWR0237")
 					(unit 1)
 				)
@@
 		(on_board yes)
 		(dnp no)
-		(property "Reference" "U21"
+		(property "Reference" "U37"
 			(at 91.44 32.766 0)
 			(effects
@@
 			(project ""
 				(path "/7184a1e6-58da-49c8-8a6c-ea31385ec956/aad981fb-9d0f-43cf-87cf-306d8b58c3f7"
-					(reference "U21")
+					(reference "U37")
 					(unit 1)
 				)
@@
 		(on_board yes)
 		(dnp no)
-		(property "Reference" "C274"
+		(property "Reference" "C304"
 			(at 57.658 42.926 0)
 			(effects
@@
 			(project "BenchyMotherBoard-AM625"
 				(path "/7184a1e6-58da-49c8-8a6c-ea31385ec956/aad981fb-9d0f-43cf-87cf-306d8b58c3f7"
-					(reference "C274")
+					(reference "C304")
 					(unit 1)
 				)
@@
 		(on_board yes)
 		(dnp no)
-		(property "Reference" "R62"
+		(property "Reference" "R161"
 			(at 154.432 28.448 90)
 			(effects
@@
 			(project ""
 				(path "/7184a1e6-58da-49c8-8a6c-ea31385ec956/aad981fb-9d0f-43cf-87cf-306d8b58c3f7"
-					(reference "R62")
+					(reference "R161")
 					(unit 1)
 				)
@@
 		(on_board yes)
 		(dnp no)
-		(property "Reference" "#PWR0161"
+		(property "Reference" "#PWR0236"
 			(at 152.4 109.22 0)
 			(effects
@@
 			(project "BenchyMotherBoard-AM625"
 				(path "/7184a1e6-58da-49c8-8a6c-ea31385ec956/aad981fb-9d0f-43cf-87cf-306d8b58c3f7"
-					(reference "#PWR0161")
+					(reference "#PWR0236")
 					(unit 1)
 				)
@@
 		(on_board yes)
 		(dnp no)
-		(property "Reference" "R64"
+		(property "Reference" "R167"
 			(at 164.592 95.758 90)
 			(effects
@@
 			(project "BenchyMotherBoard-AM625"
 				(path "/7184a1e6-58da-49c8-8a6c-ea31385ec956/aad981fb-9d0f-43cf-87cf-306d8b58c3f7"
-					(reference "R64")
+					(reference "R167")
 					(unit 1)
 				)
@@
 		(on_board yes)
 		(dnp no)
-		(property "Reference" "#PWR0158"
+		(property "Reference" "#PWR0233"
 			(at 38.1 82.55 0)
 			(effects
@@
 			(project "BenchyMotherBoard-AM625"
 				(path "/7184a1e6-58da-49c8-8a6c-ea31385ec956/aad981fb-9d0f-43cf-87cf-306d8b58c3f7"
-					(reference "#PWR0158")
+					(reference "#PWR0233")
 					(unit 1)
 				)
@@
 		(on_board no)
 		(dnp no)
-		(property "Reference" "#PWR0156"
+		(property "Reference" "#PWR0232"
 			(at 41.91 36.83 0)
 			(effects
@@
 			(project "BenchyMotherBoard-AM625"
 				(path "/7184a1e6-58da-49c8-8a6c-ea31385ec956/aad981fb-9d0f-43cf-87cf-306d8b58c3f7"
-					(reference "#PWR0156")
+					(reference "#PWR0232")
 					(unit 1)
 				)
@@
 		(on_board yes)
 		(dnp no)
-		(property "Reference" "#PWR0163"
+		(property "Reference" "#PWR0234"
 			(at 97.79 86.36 0)
 			(effects
@@
 			(project "BenchyMotherBoard-AM625"
 				(path "/7184a1e6-58da-49c8-8a6c-ea31385ec956/aad981fb-9d0f-43cf-87cf-306d8b58c3f7"
-					(reference "#PWR0163")
+					(reference "#PWR0234")
 					(unit 1)
 				)
@@
 		(on_board yes)
 		(dnp no)
-		(property "Reference" "R66"
+		(property "Reference" "R165"
 			(at 98.806 76.835 0)
 			(effects
@@
 			(project ""
 				(path "/7184a1e6-58da-49c8-8a6c-ea31385ec956/aad981fb-9d0f-43cf-87cf-306d8b58c3f7"
-					(reference "R66")
+					(reference "R165")
 					(unit 1)
 				)
@@
 		(on_board yes)
 		(dnp no)
-		(property "Reference" "C278"
+		(property "Reference" "C301"
 			(at 38.608 42.926 0)
 			(effects
@@
 			(project ""
 				(path "/7184a1e6-58da-49c8-8a6c-ea31385ec956/aad981fb-9d0f-43cf-87cf-306d8b58c3f7"
-					(reference "C278")
+					(reference "C301")
 					(unit 1)
 				)
@@
 		(on_board yes)
 		(dnp no)
-		(property "Reference" "#PWR0157"
+		(property "Reference" "#PWR0238"
 			(at 77.47 106.68 0)
 			(effects
@@
 			(project "BenchyMotherBoard-AM625"
 				(path "/7184a1e6-58da-49c8-8a6c-ea31385ec956/aad981fb-9d0f-43cf-87cf-306d8b58c3f7"
-					(reference "#PWR0157")
+					(reference "#PWR0238")
 					(unit 1)
 				)
@@
 		(on_board no)
 		(dnp no)
-		(property "Reference" "#PWR0160"
+		(property "Reference" "#PWR0235"
 			(at 156.21 90.17 0)
 			(effects
@@
 			(project "BenchyMotherBoard-AM625"
 				(path "/7184a1e6-58da-49c8-8a6c-ea31385ec956/aad981fb-9d0f-43cf-87cf-306d8b58c3f7"
-					(reference "#PWR0160")
+					(reference "#PWR0235")
 					(unit 1)
 				)
@@
 		(on_board yes)
 		(dnp no)
-		(property "Reference" "R67"
+		(property "Reference" "R163"
 			(at 105.156 31.115 0)
 			(effects
@@
 			(project "BenchyMotherBoard-AM625"
 				(path "/7184a1e6-58da-49c8-8a6c-ea31385ec956/aad981fb-9d0f-43cf-87cf-306d8b58c3f7"
-					(reference "R67")
+					(reference "R163")
 					(unit 1)
 				)
@@
 		(on_board no)
 		(dnp no)
-		(property "Reference" "#PWR0159"
+		(property "Reference" "#PWR0231"
 			(at 101.6 24.13 0)
 			(effects
@@
 			(project "BenchyMotherBoard-AM625"
 				(path "/7184a1e6-58da-49c8-8a6c-ea31385ec956/aad981fb-9d0f-43cf-87cf-306d8b58c3f7"
-					(reference "#PWR0159")
+					(reference "#PWR0231")
 					(unit 1)
 				)
@@
 		(on_board yes)
 		(dnp no)
-		(property "Reference" "#PWR0154"
+		(property "Reference" "#PWR0239"
 			(at 92.71 132.08 0)
 			(effects
@@
 			(project ""
 				(path "/7184a1e6-58da-49c8-8a6c-ea31385ec956/aad981fb-9d0f-43cf-87cf-306d8b58c3f7"
-					(reference "#PWR0154")
+					(reference "#PWR0239")
 					(unit 1)
 				)
@@
 		(on_board yes)
 		(dnp no)
-		(property "Reference" "R68"
+		(property "Reference" "R164"
 			(at 149.352 30.988 90)
 			(effects
@@
 			(project "BenchyMotherBoard-AM625"
 				(path "/7184a1e6-58da-49c8-8a6c-ea31385ec956/aad981fb-9d0f-43cf-87cf-306d8b58c3f7"
-					(reference "R68")
+					(reference "R164")
 					(unit 1)
 				)
