File: MotherBoard/BenchyMotherBoard-AM625/BenchyMotherboard-AM625_USB.kicad_sch (KiCad schematic)
At the start: 46 parts, among them J3 5787745-2, J9 GSB3211311WEU, U1 AM6254ATCGGAALW, U25 AP2156SG-13, U55 W25Q16JVUXIQ TR, U56 74HC2G08DP,125, U8 USB2412-DZK-TR, U9 USB7206C/KDX

Commit message: Schematic capture mostly complete. Starting PCB layout
Parts:
- renumbered C345 to C307, C344 to C308, C355 to C309, C342 to C310, C343 to C311, C348 to C312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
